File: eagle/Frontboard.sch (EAGLE design)
At the start: 24 parts, among them IC1 LM35DM_NOPB

Commit message: updates
Parts:
- LEDS: value (none) -> LEDS
Changed lines of the file:
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@@
 <part name="LED1" library="SparkFun-LED" deviceset="LED" device="1206-BOTTOM" value="WHITE"/>
 <part name="LED5" library="SparkFun-LED" deviceset="LED" device="1206-BOTTOM" value="WHITE"/>
-<part name="LEDS" library="pinhead" deviceset="PINHD-1X4" device="_2.54-SMD"/>
+<part name="LEDS" library="pinhead" deviceset="PINHD-1X4" device="_2.54-SMD" value="LEDS"/>
 <part name="IC_SENSE" library="CY8CMBR3116-LQXIT" deviceset="CY8CMBR3116-LQXIT" device=""/>
 <part name="R1" library="resistor" library_urn="urn:adsk.eagle:library:348" deviceset="R-EU_" device="R0805" package3d_urn="urn:adsk.eagle:package:26059/1" value="560E"/>

Commit message: updates
Parts:
- removed C1, C5: 0.1uf, rcl:C-EUC0805
- removed C2: 1uf, rcl:C-EUC0805
- removed C6: 2.2nf, rcl:C-EUC0805
- removed IC1: LM35DM_NOPB, LM35DM_NOPB:LM35DM_NOPB
- removed IC_SENSE: CY8CMBR3116-LQXIT, CY8CMBR3116-LQXIT:CY8CMBR3116-LQXIT
- removed JP_I2C: I2C, pinhead:PINHD-1X6_2.54-SMD
- removed LED1, LED2, LED4, LED5: WHITE, SparkFun-LED:LED1206-BOTTOM
- removed LEDS: LEDS, pinhead:PINHD-1X4_2.54-SMD
- removed R1, R2, R5, R6, RS1, RS3: 560E, resistor:R-EU_R0805
- removed R3, R4, RL1, RL2, RL4, RL5: 330E, resistor:R-EU_R0805
- added 3V3_REGULATOR: MCP1703T-3302E_MB, MCP1703T-3302E_MB:MCP1703T-3302E_MB
- added BCU: BCU, pinhead:PINHD-2X5_2.54-SMD
- added BRAIN: STM32L072CBT, STM32L072CBT:STM32L072CBT
- added CB1, CB2, CB3, CB4: 100nf, rcl:C-EUC0603
- added CLO1: 7pF, rcl:C-EUC0603
- added CLO2: 7pf, rcl:C-EUC0603
- added CLO3, CLO4: 18pf, rcl:C-EUC0603
- added CR1, CR2: 1uF, rcl:C-EUC0603
- added CRST: 0.1uF, rcl:C-EUC0603
- added F1: PPTC_6V500MA, SparkFun-Fuses:PPTC_6V500MA
- added RUSBVCC: 220, resistor:R-EU_R0603
- added USBCONNECTOR: (no value), tag-connect:TC2030-MCP-NL
- added Y1: ABS07-32.768KHZ-7-T, ABS07-32.768KHZ-7-T:ABS07-32.768KHZ-7-T
- added Y2: ABM3B-8.000MHZ-B2-T, ABM3B-8.000MHZ-B2-T:ABM3B-8.000MHZ-B2-T
Connections:
- removed net HOST_INT: IC_SENSE.!HI!/BUZ/GPO7, JP_I2C.3
- removed net I2C_SCL: JP_I2C.4, R3.2
- removed net I2C_SDA: JP_I2C.5, R4.2
- removed net LED1: LEDS.1, RL1.1
- removed net LED2: LEDS.3, RL2.1
- removed net LED4: LEDS.2, RL4.1
- removed net LED5: LEDS.4, RL5.1
- removed net N$14: LED5.A, RL5.2
- removed net N$15: LED4.A, RL4.2
- removed net N$16: LED2.A, RL2.2
- removed net N$17: LED1.A, RL1.2
- removed net N$19: C5.1, IC_SENSE.VCC
- removed net N$20: C6.1, IC_SENSE.CMOD
- removed net N$4: IC_SENSE.CS11/GPO3, RS3.2
- removed net N$5: IC_SENSE.CS0/PS0, R1.2
- removed net N$6: IC_SENSE.CS1/PS1, R2.2
- removed net N$7: IC_SENSE.CS3, R6.2
- removed net N$8: IC_SENSE.CS2/GUARD, R5.2
- removed net SENS_1: RS1.1
- removed net SENS_2: R5.1
- removed net SENS_3: RS3.1
- removed net SENS_4: R6.1
- removed net SENS_PROX_1: R1.1
- removed net SENS_PROX_2: R2.1
- removed net TEMP: IC1.VOUT, JP_I2C.6
- removed net VCC: C1.1, C2.1, IC1.+VS, IC_SENSE.VDD, JP_I2C.2
- new net +3V3: 3V3_REGULATOR.VOUT, BRAIN.VDD, BRAIN.VDDA, BRAIN.VDD_2, BRAIN.VDD_3, CB1.1, CB2.1, CB3.1, CB4.1, CR2.1
- new net +5V: 3V3_REGULATOR.VIN1, 3V3_REGULATOR.VIN2, BCU.1, CR1.2
- new net OSC32_IN: BRAIN.PC14-OSC32_IN, CLO1.2, Y1.1
- new net OSC32_OUT: BRAIN.PC15-OSC32_OUT, CLO2.2, Y1.2
- new net OSC_IN: BRAIN.PH0-OSC_IN, CLO3.2, Y2.NC1
- new net OSC_OUT: BRAIN.PH1-OSC_OUT, CLO4.2, Y2.NC2
- new net RXD: BCU.7
- new net TXD: BCU.3
- new net USB_DM: BRAIN.PA11, USBCONNECTOR.ICSP_CLK/PGC
- new net USB_DP: BRAIN.PA12, USBCONNECTOR.ICSP_DAT/PGD
- new net USB_VCC: BRAIN.VDD_UBS, RUSBVCC.1
- net GND: now also 3V3_REGULATOR.GND, BCU.9, BRAIN.VSS, BRAIN.VSSA, BRAIN.VSS_2, BRAIN.VSS_3, CB1.2, CB2.2, CB3.2, CB4.2, CLO1.1, CLO2.1, CLO3.1, CLO4.1, CR1.1, CR2.2, CRST.2, USBCONNECTOR.VSS(GND), Y2.GND1, Y2.GND2; no longer C1.2, C2.2, C5.2, C6.2, IC1.GND, IC_SENSE.CS15/SH/!HI, IC_SENSE.CS4, IC_SENSE.CS5, IC_SENSE.CS6, IC_SENSE.CS7, IC_SENSE.VSS, JP_I2C.1, LED1.C, LED2.C, LED4.C, LED5.C
- net N$1: now also BRAIN.NRST, CRST.1; no longer IC_SENSE.I2C_SCL, R3.1
- net N$2: now also F1.2, USBCONNECTOR.VDD; no longer IC_SENSE.I2C_SDA, R4.1
- net N$3: now also F1.1, RUSBVCC.2; no longer IC_SENSE.CS10/GPO2, RS1.2
Other:
- note removed: "Use MC Pins to control the LED'S. It would be better to use an I2C LED Driver"

Commit message: updates
Parts:
- removed CLO3, CLO4: 18pf, rcl:C-EUC0603
- removed CRST: 0.1uF, rcl:C-EUC0603
- removed F1: PPTC_6V500MA, SparkFun-Fuses:PPTC_6V500MA
- removed RUSBVCC: 220, resistor:R-EU_R0603
- removed USBCONNECTOR: (no value), tag-connect:TC2030-MCP-NL
- removed Y2: ABM3B-8.000MHZ-B2-T, ABM3B-8.000MHZ-B2-T:ABM3B-8.000MHZ-B2-T
- added C7: 0.1uF, rcl:C-EUC0603
- added CS1, CS2, CS3: 47nF, rcl:C-EUC0603
- added LED1, LED2, LED3, LED4: WL-SMRW156120BS75300-B_RVS-MOUNT, Wurth_Elektronik_Optoelectronics_rev15b (1):WL-SMRW156120BS75300-B_RVS-MOUNT
- added R1: CSTCE8M00G55-R0, CSTCE8M00G55-R0:CSTCE8M00G55-R0
- added RL1, RL2, RL3, RL4, RP1, RP2, RS1, RS2, RS3, RS4: 330E, rcl:R-EU_R0603
- added RST1, RST2: 0, wirepad:SMD5
- added SWD: SWD, tag-connect:TC2030-MCP-NL
- BRAIN: value STM32L072CBT -> STM32L152RET6; device STM32L072CBT:STM32L072CBT -> STM32L152RET6:STM32L152RET6
- renumbered CB1 to C3, CB2 to C4, CB3 to C5, CB4 to C6, CR1 to C1, CR2 to C2
Connections:
- removed net USB_DM: BRAIN.PA11, USBCONNECTOR.ICSP_CLK/PGC
- removed net USB_DP: BRAIN.PA12, USBCONNECTOR.ICSP_DAT/PGD
- removed net USB_VCC: BRAIN.VDD_UBS, RUSBVCC.1
- new net G10_IO1: BRAIN.PC6
- new net G10_IO2: BRAIN.PC7, RS3.2
- new net G10_IO3: BRAIN.PC8, RS1.2
- new net G10_IO4: BRAIN.PC9, CS1.1
- new net G1_IO1: BRAIN.PA0-WKUP1
- new net G1_IO2: BRAIN.PA1, RP1.2
- new net G1_IO3: BRAIN.PA2, RP2.2
- new net G1_IO4: BRAIN.PA3, CS2.1
- new net G7_IO1: BRAIN.PB12
- new net G7_IO2: BRAIN.PB13
- new net G7_IO3: BRAIN.PB14
- new net G7_IO4: BRAIN.PB15
- new net G8_IO1: BRAIN.PC0
- new net G8_IO2: BRAIN.PC1, RS2.2
- new net G8_IO3: BRAIN.PC2, RS4.2
- new net G8_IO4: BRAIN.PC3, CS3.1
- new net I2C1_SCL: BRAIN.PB6
- new net I2C1_SDA: BRAIN.PB7
- new net LED1: RL1.1
- new net LED2: RL2.1
- new net LED4: RL3.1
- new net LED5: RL4.1
- new net N$10: BRAIN.PA12
- new net N$19: LED1.A, RL1.2
- new net N$20: LED2.A, RL2.2
- new net N$21: LED3.A, RL3.2
- new net N$22: LED4.A, RL4.2
- new net N$7: BRAIN.PA9
- new net N$8: BRAIN.PA10
- new net N$9: BRAIN.PA11
- new net NRST: BRAIN.NRST, C7.1, RST1.P, SWD.VPP/MCLR
- new net SENS_1: RS1.1
- new net SENS_2: RS2.1
- new net SENS_3: RS3.1
- new net SENS_4: RS4.1
- new net SENS_PROX_1: RP1.1
- new net SENS_PROX_2: RP2.1
- new net SWCLK: BRAIN.PA14, SWD.ICSP_CLK/PGC
- new net SWDIO: BRAIN.PA13, SWD.ICSP_DAT/PGD
- net +3V3: now also BRAIN.VDD1, BRAIN.VDD2, BRAIN.VDD3, BRAIN.VDD4; no longer BRAIN.VDD, BRAIN.VDD_2, BRAIN.VDD_3
- net GND: now also BRAIN.BOOT0, BRAIN.PB2, BRAIN.VSS1, BRAIN.VSS2, BRAIN.VSS3, BRAIN.VSS4, C7.2, CS1.2, CS2.2, CS3.2, LED1.K, LED2.K, LED3.K, LED4.K, R1.2, RST2.P, SWD.VSS(GND); no longer BRAIN.VSS, BRAIN.VSS_2, BRAIN.VSS_3, CLO3.1, CLO4.1, CRST.2, USBCONNECTOR.VSS(GND), Y2.GND1, Y2.GND2
- net N$1: now also BRAIN.PB3; no longer BRAIN.NRST, CRST.1
- net N$2: now also BRAIN.PB4; no longer F1.2, USBCONNECTOR.VDD
- net N$3: now also BRAIN.PA8; no longer F1.1, RUSBVCC.2
- net OSC_IN: now also R1.1; no longer CLO3.2, Y2.NC1
- net OSC_OUT: now also R1.3; no longer CLO4.2, Y2.NC2

Commit message: updates
Parts:
- added IC1: NCT75DR2G, NCT75DR2G:NCT75DR2G
- added RST3, RST4: 0, wirepad:SMD5
- added RT1: 100K, rcl:R-EU_R0603
Connections:
- removed net G7_IO1: BRAIN.PB12
- removed net LED5: RL4.1
- removed net N$10: BRAIN.PA12
- new net I2C2_SCL: BRAIN.PB10, IC1.SCL
- new net I2C2_SDA: BRAIN.PB11, IC1.SDA
- new net LED3: BRAIN.PB12, RL3.1
- new net PRG: BRAIN.PA12, RST3.P, RT1.2
- net +3V3: now also IC1.A0, IC1.A1, IC1.A2, IC1.VDD, RT1.1
- net GND: now also IC1.GND, RST4.P
- net LED1: now also BRAIN.PC10
- net LED2: now also BRAIN.PC13-WKUP2
- net LED4: now also BRAIN.PB1, RL4.1; no longer RL3.1
Other:
- note added: "I²C Adr.: 0x4F"
