File: eagle/Frontboard2.brd (EAGLE design)
At the start: 69.8 x 69.8 mm, 43 parts, among them Y1 ABS07-32.768KHZ-7-T

Commit message: updates
Parts:
- removed BRAIN: STM32L152RET6, STM32L152RET6:QFP50P1200X1200X160-64N
- removed C6: 100nf, rcl:C0603
- removed CS1, CS2, CS3: 47nF, rcl:C0603
- removed R1: CSTCE8M00G55-R0, CSTCE8M00G55-R0:CSTCE12M0G55-R0
- removed R2, R3: 4.7k, rcl:R0603
- removed SWD: SWD, tag-connect:TC2030-MCP-NL
- added C10, C9: 100nf, rcl:C0603
- added IC1: CY8CMBR3116-LQXI, CY8CMBR3116-LQXI:QFN50P400X400X60-25N
- added U1: STM32L432KX, STM32L432KC:UFQFPN32-5X5MM
- added Y2: DSC1001CC1-008.0000, DSC1001BE5-016.0000T:DSC1001BE50160000T
- C3: value 100nf -> 2.2nF
- C4: value 100nf -> 0.1uF
- RP1, RP2, RS1, RS2, RS3, RS4: value 330E -> 560E
- moved RST1 53.3 mm to (61.6, 39.4)
- moved RST3 53.3 mm to (8.26, 39.4)
- moved RT1 53.3 mm to (8.26, 44.5)
- moved C7 29.6 mm to (61.6, 44.5), turned to 90 degrees
- moved TEMP 28.5 mm to (34.9, 7.75), turned to 0 degrees
- moved C8 23.6 mm to (34.9, 10.2), turned to 180 degrees
- moved CLO2 23.3 mm to (32.4, 62.2), turned to 270 degrees
- moved CLO1 22.4 mm to (34.9, 62.2), turned to 270 degrees
- moved C4 20.8 mm to (29.8, 32.4), turned to 270 degrees
- moved Y1 18.1 mm to (36.8, 56.5), turned to 180 degrees
- moved C3 15.5 mm to (27.3, 32.4), turned to 270 degrees
- moved C5 14.7 mm to (33.0, 44.5), turned to 0 degrees
- moved RS1 5.08 mm to (48.9, 41.3)
- moved RS2 5.08 mm to (21.0, 41.3)
- moved RS3 5.08 mm to (48.9, 28.6)
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Connections:
- removed net G10_IO1: BRAIN.37
- removed net G10_IO2: BRAIN.38, RS3.2
- removed net G10_IO3: BRAIN.39, RS1.2
- removed net G10_IO4: BRAIN.40, CS1.1
- removed net G1_IO1: BRAIN.14
- removed net G1_IO2: BRAIN.15, RP1.2
- removed net G1_IO3: BRAIN.16, RP2.2
- removed net G1_IO4: BRAIN.17, CS2.1
- removed net G7_IO2: BRAIN.34
- removed net G7_IO3: BRAIN.35
- removed net G7_IO4: BRAIN.36
- removed net G8_IO1: BRAIN.8
- removed net G8_IO2: BRAIN.9, RS2.2
- removed net G8_IO3: BRAIN.10, RS4.2
- removed net G8_IO4: BRAIN.11, CS3.1
- removed net I2C1_SCL: BRAIN.58
- removed net I2C1_SDA: BRAIN.59
- removed net I2C2_SCL: BRAIN.29, R3.2, TEMP.2
- removed net I2C2_SDA: BRAIN.30, R2.2, TEMP.4
- removed net N$1: BRAIN.55
- removed net N$2: BRAIN.56
- removed net N$3: BRAIN.41
- removed net N$7: BRAIN.42
- removed net N$8: BRAIN.43
- removed net N$9: BRAIN.44
- removed net OSC_IN: BRAIN.5, R1.1
- removed net OSC_OUT: BRAIN.6, R1.3
- removed net VLCD: BRAIN.1
- new net CMOD: C3.1, IC1.5
- new net EP_GND: IC1.25
- new net EXT_CLK: U1.6, Y2.3
- new net HOST_INT: IC1.23, U1.18
- new net I2C_SCL: IC1.22, TEMP.2, U1.19
- new net I2C_SDA: IC1.21, TEMP.4, U1.20
- new net IC_SENS_1: IC1.18, RS1.2
- new net IC_SENS_2: IC1.3, RS2.2
- new net IC_SENS_3: IC1.17, RS3.2
- new net IC_SENS_4: IC1.4, RS4.2
- new net IC_SENS_PROX_1: IC1.1, RP1.2
- new net IC_SENS_PROX_2: IC1.2, RP2.2
- new net VCC: C4.1, IC1.6
- net +3V3: now also C10.1, C5.2, C9.2, IC1.7, U1.1, U1.17, U1.5, Y2.4; no longer BRAIN.13, BRAIN.19, BRAIN.32, BRAIN.48, BRAIN.64, C3.1, C4.1, C5.1, C6.1, R2.1, R3.1
- net GND: now also C10.2, C5.1, C9.1, IC1.10, IC1.11, IC1.12, IC1.13, IC1.14, IC1.15, IC1.16, IC1.19, IC1.20, IC1.8, IC1.9, U1.16, U1.31, U1.32, Y2.2; no longer BRAIN.12, BRAIN.18, BRAIN.28, BRAIN.31, BRAIN.47, BRAIN.60, BRAIN.63, C5.2, C6.2, CS1.2, CS2.2, CS3.2, R1.2, SWD.3
- net LED1: now also U1.29; no longer BRAIN.51
- net LED2: now also U1.10; no longer BRAIN.2
- net LED3: now also U1.27; no longer BRAIN.33
- net LED4: now also U1.12; no longer BRAIN.27
- net NRST: now also U1.4; no longer BRAIN.7, SWD.1, SWD.2
- net OSC32_IN: now also U1.2; no longer BRAIN.3
- net OSC32_OUT: now also U1.3; no longer BRAIN.4
- net PRG: now also U1.11; no longer BRAIN.45
- net SWCLK: now also U1.24; no longer BRAIN.49, SWD.5
- net SWDIO: now also U1.23; no longer BRAIN.46, SWD.4
Routing:
- net GND: track 417.1 -> 462.2 mm, vias 0 -> 5
- net SENS_PROX_2: track 185.8 -> 230.9 mm
- net I2C_SCL: track 0.00 -> 44.8 mm, vias 0 -> 4
- net I2C_SDA: track 0.00 -> 44.7 mm, vias 0 -> 4
- net I2C2_SCL: track 33.7 -> 0.00 mm, vias 4 -> 0
- net I2C2_SDA: track 33.2 -> 0.00 mm, vias 4 -> 0
- net IC_SENS_1: track 0.00 -> 23.8 mm
- net G8_IO3: track 20.0 -> 0.00 mm, vias 2 -> 0
- net G10_IO2: track 19.1 -> 0.00 mm, vias 2 -> 0
- net NRST: track 40.0 -> 56.8 mm, vias 4 -> 5
- net IC_SENS_3: track 0.00 -> 16.5 mm
- net IC_SENS_2: track 0.00 -> 16.3 mm, vias 0 -> 2
- net LED3: track 22.2 -> 38.1 mm
- net G10_IO3: track 15.4 -> 0.00 mm, vias 2 -> 0
- net G8_IO2: track 15.1 -> 0.00 mm, vias 2 -> 0
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
Commit message: updates
Parts:
- removed Y2: DSC1001CC1-008.0000, DSC1001BE5-016.0000T:DSC1001BE50160000T
Connections:
- net +3V3: no longer Y2.4
- net EXT_CLK: no longer Y2.3
- net GND: no longer Y2.2
Routing:
- net GND: track 462.2 -> 449.7 mm
- net +3V3: track 120.0 -> 117.8 mm
- net EXT_CLK: track 3.42 -> 2.91 mm
Changed lines of the file:
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@@
 <setting verticaltext="up"/>
 </settings>
-<grid distance="50" unitdist="mil" unit="inch" style="lines" multiple="1" display="yes" altdistance="5" altunitdist="mil" altunit="inch"/>
+<grid distance="50" unitdist="mil" unit="inch" style="lines" multiple="1" display="yes" altdistance="0.025" altunitdist="inch" altunit="inch"/>
 <layers>
 <layer number="1" name="Top" color="4" fill="1" visible="yes" active="yes"/>
@@
 <layer number="43" name="vRestrict" color="2" fill="10" visible="yes" active="yes"/>
 <layer number="44" name="Drills" color="7" fill="1" visible="no" active="yes"/>
-<layer number="45" name="Holes" color="7" fill="1" visible="no" active="yes"/>
+<layer number="45" name="Holes" color="7" fill="1" visible="yes" active="yes"/>
 <layer number="46" name="Milling" color="3" fill="1" visible="no" active="yes"/>
 <layer number="47" name="Measures" color="7" fill="1" visible="no" active="yes"/>
@@
 <attribute name="SPICEPREFIX" value="C" x="29.845" y="32.385" size="1.778" layer="27" rot="R270" display="off"/>
 </element>
-<element name="Y2" library="DSC1001BE5-016.0000T" package="DSC1001BE50160000T" value="DSC1001CC1-008.0000" x="31.115" y="56.515">
-<attribute name="ARROW_PART_NUMBER" value="DSC1001BE5-016.0000T" x="31.115" y="56.515" size="1.778" layer="27" display="off"/>
-<attribute name="ARROW_PRICE/STOCK" value="https://www.arrow.com/en/products/dsc1001be5-016.0000t/microchip-technology" x="31.115" y="56.515" size="1.778" layer="27" display="off"/>
-<attribute name="DESCRIPTION" value="Standard Clock Oscillators MEMS Oscillator Low PWR LVCMOS -20C-70C" x="31.115" y="56.515" size="1.778" layer="27" display="off"/>
-<attribute name="HEIGHT" value="0mm" x="31.115" y="56.515" size="1.778" layer="27" display="off"/>
-<attribute name="MANUFACTURER_NAME" value="Microchip" x="31.115" y="56.515" size="1.778" layer="27" display="off"/>
-<attribute name="MANUFACTURER_PART_NUMBER" value="DSC1001BE5-016.0000T" x="31.115" y="56.515" size="1.778" layer="27" display="off"/>
-<attribute name="RS_PART_NUMBER" value="" x="31.115" y="56.515" size="1.778" layer="27" display="off"/>
-<attribute name="RS_PRICE/STOCK" value="" x="31.115" y="56.515" size="1.778" layer="27" display="off"/>
-</element>
 </elements>
 <signals>
@@
 <wire x1="36.925" y1="34.302" x2="36.925" y2="34.802" width="0.1524" layer="1"/>
 <wire x1="36.925" y1="34.802" x2="36.925" y2="35.302" width="0.1524" layer="1"/>
-<contactref element="Y2" pad="2"/>
 <contactref element="U1" pad="31"/>
 <wire x1="37.275" y1="51.915440625" x2="37.275" y2="51.415315625" width="0.3048" layer="1"/>
@@
 <wire x1="37.465" y1="63.08" x2="32.385" y2="63.08" width="0.3048" layer="1"/>
 <wire x1="34.925" y1="63.08" x2="34.925" y2="66.04" width="0.3048" layer="1"/>
-<wire x1="30.315" y1="55.245" x2="17.78" y2="55.245" width="0.3048" layer="1"/>
 <wire x1="34.925" y1="63.08" x2="37.465" y2="63.08" width="0.3048" layer="1"/>
 <wire x1="32.17" y1="38.52" x2="31.496" y2="37.846" width="0.3048" layer="1"/>
@@
 <wire x1="33.44" y1="32.639" x2="33.44" y2="32.817" width="0.3048" layer="1"/>
 <wire x1="33.44" y1="32.817" x2="33.675" y2="33.052" width="0.3048" layer="1"/>
-<contactref element="Y2" pad="4"/>
 <wire x1="33.87" y1="39.204" x2="33.87" y2="41.91" width="0.3048" layer="1"/>
 <wire x1="33.87" y1="41.91" x2="33.87" y2="44.45" width="0.3048" layer="1"/>
@@
 <wire x1="39.37" y1="55.499" x2="39.37" y2="59.475" width="0.3048" layer="1"/>
 <wire x1="34.671" y1="53.721" x2="34.036" y2="54.356" width="0.3048" layer="1"/>
-<wire x1="34.036" y1="56.264" x2="32.515" y2="57.785" width="0.3048" layer="1"/>
 <wire x1="34.036" y1="54.356" x2="34.036" y2="56.264" width="0.3048" layer="1"/>
 <wire x1="33.87" y1="39.204" x2="32.512" y2="37.846" width="0.3048" layer="1"/>
@@
 <signal name="EXT_CLK">
 <contactref element="U1" pad="6"/>
-<contactref element="Y2" pad="3"/>
 <wire x1="34.1748125" y1="52.515" x2="34.1748125" y2="53.0741875" width="0.1524" layer="1"/>
-<wire x1="32.515" y1="54.734" x2="32.515" y2="55.245" width="0.1524" layer="1"/>
 <wire x1="34.1748125" y1="53.0741875" x2="32.515" y2="54.734" width="0.1524" layer="1"/>
 </signal>
