File: eagle/Frontboard2.sch (EAGLE design)
At the start: 39 parts, among them IC1 NCT75DR2G, IC2 HTS221TR, Y1 ABS07-32.768KHZ-7-T

Commit message: updates
Parts:
- removed BRAIN: STM32L152RET6, STM32L152RET6:STM32L152RET6
- removed C6: 100nf, rcl:C-EUC0603
- removed CS1, CS2, CS3: 47nF, rcl:C-EUC0603
- removed IC2: HTS221TR, HTS221TR:HTS221TR
- removed R1: CSTCE8M00G55-R0, CSTCE8M00G55-R0:CSTCE8M00G55-R0
- removed SWD: SWD, tag-connect:TC2030-MCP-NL
- added C10, C8, C9: 100nf, rcl:C-EUC0603
- added TEMP: HTS221TR, HTS221TR:HTS221TR
- added U1: STM32L432KX, STM32L432KC:STM32L432KX
- added Y2: DSC1001CC1-008.0000, DSC1001BE5-016.0000T:DSC1001BE5-016.0000T
- C3: value 100nf -> 2.2nF
- C4: value 100nf -> 0.1uF
- IC1: value NCT75DR2G -> CY8CMBR3116-LQXI; device NCT75DR2G:NCT75DR2G -> CY8CMBR3116-LQXI:CY8CMBR3116-LQXI
- RP1, RP2, RS1, RS2, RS3, RS4: value 330E -> 560E
Connections:
- removed net G10_IO1: BRAIN.PC6
- removed net G10_IO2: BRAIN.PC7, RS3.2
- removed net G10_IO3: BRAIN.PC8, RS1.2
- removed net G10_IO4: BRAIN.PC9, CS1.1
- removed net G1_IO1: BRAIN.PA0-WKUP1
- removed net G1_IO2: BRAIN.PA1, RP1.2
- removed net G1_IO3: BRAIN.PA2, RP2.2
- removed net G1_IO4: BRAIN.PA3, CS2.1
- removed net G7_IO2: BRAIN.PB13
- removed net G7_IO3: BRAIN.PB14
- removed net G7_IO4: BRAIN.PB15
- removed net G8_IO1: BRAIN.PC0
- removed net G8_IO2: BRAIN.PC1, RS2.2
- removed net G8_IO3: BRAIN.PC2, RS4.2
- removed net G8_IO4: BRAIN.PC3, CS3.1
- removed net I2C1_SCL: BRAIN.PB6
- removed net I2C1_SDA: BRAIN.PB7
- removed net I2C2_SCL: BRAIN.PB10, IC1.SCL, IC2.SCL/SPC
- removed net I2C2_SDA: BRAIN.PB11, IC1.SDA, IC2.SDA/SDI/SDO
- removed net N$1: BRAIN.PB3
- removed net N$10: IC2.SPI_ENABLE
- removed net N$2: BRAIN.PB4
- removed net N$3: BRAIN.PA8
- removed net N$7: BRAIN.PA9
- removed net N$8: BRAIN.PA10
- removed net N$9: BRAIN.PA11
- removed net OSC_IN: BRAIN.PH0-OSC_IN, R1.1
- removed net OSC_OUT: BRAIN.PH1-OSC_OUT, R1.3
- new net CMOD: C3.1, IC1.CMOD
- new net EXT_CLK: U1.PA0-CK_IN, Y2.OUT
- new net HOST_INT: IC1.HI/BUZ/GPO7, U1.PA8
- new net I2C_SCL: IC1.I2C_SCL, TEMP.SCL/SPC, U1.PA9
- new net I2C_SDA: IC1.I2C_SDA, TEMP.SDA/SDI/SDO, U1.PA10
- new net IC_SENS_1: IC1.CS6, RS1.2
- new net IC_SENS_2: IC1.CS2/GUARD, RS2.2
- new net IC_SENS_3: IC1.CS7, RS3.2
- new net IC_SENS_4: IC1.CS3, RS4.2
- new net IC_SENS_PROX_1: IC1.CS0/PS0, RP1.2
- new net IC_SENS_PROX_2: IC1.CS1/PS1, RP2.2
- new net VCC: C4.1, IC1.VCC
- net +3V3: now also C10.1, C5.2, C8.2, C9.2, TEMP.SPI_ENABLE, TEMP.VDD, U1.VDD, U1.VDDA/VREF+, U1.VDD_2, Y2.VDD; no longer BRAIN.VDD1, BRAIN.VDD2, BRAIN.VDD3, BRAIN.VDD4, BRAIN.VDDA, C3.1, C4.1, C5.1, C6.1, IC1.A0, IC1.A1, IC1.A2, IC2.VDD
- net GND: now also C10.2, C5.1, C8.1, C9.1, IC1.CS10/GPO2, IC1.CS11/GPO3, IC1.CS12/GP14, IC1.CS13/GPO5, IC1.CS14/GPO6, IC1.CS15/SH/!HI, IC1.CS4, IC1.CS5, IC1.CS8/GPO0, IC1.CS9/GPO1, IC1.VSS, TEMP.GND, U1.PH3-BOOT0, U1.VSS, U1.VSS_2, Y2.GND; no longer BRAIN.BOOT0, BRAIN.PB2, BRAIN.VSS1, BRAIN.VSS2, BRAIN.VSS3, BRAIN.VSS4, BRAIN.VSSA, C5.2, C6.2, CS1.2, CS2.2, CS3.2, IC1.GND, IC2.GND, R1.2, SWD.VSS(GND)
- net LED1: now also U1.PB6; no longer BRAIN.PC10
- net LED2: now also U1.PA4; no longer BRAIN.PC13-WKUP2
- net LED3: now also U1.PB4; no longer BRAIN.PB12
- net LED4: now also U1.PA6; no longer BRAIN.PB1
- net NRST: now also U1.NRST; no longer BRAIN.NRST, SWD.VPP/MCLR
- net OSC32_IN: now also U1.PC14-OSC32_IN; no longer BRAIN.PC14-OSC32_IN
- net OSC32_OUT: now also U1.PC15-OSC32_OUT; no longer BRAIN.PC15-OSC32_OUT
- net PRG: now also U1.PA5; no longer BRAIN.PA12
- net SWCLK: now also U1.PA14; no longer BRAIN.PA14, SWD.ICSP_CLK/PGC
- net SWDIO: now also U1.PA13; no longer BRAIN.PA13, SWD.ICSP_DAT/PGD
Other:
- note added: "I2C READ: 0xBF I2C WRITE: 0xBE"
- note removed: "I²C Adr.: 0x4F"
- moved on the sheet: C3, C4, C5, C7, RST1, RST2, RST3, RST4, RT1

Commit message: updates
Parts:
- removed Y2: DSC1001CC1-008.0000, DSC1001BE5-016.0000T:DSC1001BE5-016.0000T
Connections:
- net +3V3: no longer Y2.VDD
- net EXT_CLK: no longer Y2.OUT
- net GND: no longer Y2.GND
Changed lines of the file:
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@@
 <part name="C3" library="rcl" library_urn="urn:adsk.eagle:library:334" deviceset="C-EU" device="C0603" package3d_urn="urn:adsk.eagle:package:23616/2" value="2.2nF"/>
 <part name="C4" library="rcl" library_urn="urn:adsk.eagle:library:334" deviceset="C-EU" device="C0603" package3d_urn="urn:adsk.eagle:package:23616/2" value="0.1uF"/>
-<part name="Y2" library="DSC1001BE5-016.0000T" deviceset="DSC1001BE5-016.0000T" device="" value="DSC1001CC1-008.0000"/>
 </parts>
 <sheets>
@@
 <instance part="C3" gate="G$1" x="238.76" y="5.08"/>
 <instance part="C4" gate="G$1" x="243.84" y="5.08"/>
-<instance part="Y2" gate="G$1" x="25.4" y="-58.42"/>
 </instances>
 <busses>
@@
 </segment>
 <segment>
-<pinref part="Y2" gate="G$1" pin="GND"/>
-<wire x1="25.4" y1="-60.96" x2="17.78" y2="-60.96" width="0.1524" layer="91"/>
-<label x="17.78" y="-60.96" size="1.016" layer="95" rot="R180" xref="yes"/>
-</segment>
-<segment>
 <pinref part="U1" gate="A" pin="PH3-BOOT0"/>
 <wire x1="213.36" y1="-53.34" x2="228.6" y2="-53.34" width="0.1524" layer="91"/>
@@
 <junction x="269.24" y="-17.78"/>
 <label x="269.24" y="-22.86" size="1.016" layer="95" rot="R270" xref="yes"/>
-</segment>
-<segment>
-<pinref part="Y2" gate="G$1" pin="VDD"/>
-<wire x1="58.42" y1="-60.96" x2="68.58" y2="-60.96" width="0.1524" layer="91"/>
-<label x="68.58" y="-60.96" size="1.016" layer="95" xref="yes"/>
 </segment>
 </net>
@@
 <label x="132.08" y="-60.96" size="1.016" layer="95" rot="R180" xref="yes"/>
 </segment>
-<segment>
-<pinref part="Y2" gate="G$1" pin="OUT"/>
-<wire x1="58.42" y1="-58.42" x2="68.58" y2="-58.42" width="0.1524" layer="91"/>
-<label x="68.58" y="-58.42" size="1.016" layer="95" xref="yes"/>
-</segment>
-</net>
+</net>
