File: eagle/4ButtonSwitch.Rev1.brd (EAGLE design)
At the start: 69.8 x 69.8 mm, 41 parts, among them IC1 CY8CMBR3116-LQXI, U1 STM32L432KX, Y1 ABS07-32.768KHZ-7-T

Commit message: updates
Parts:
- moved RST1 39.4 mm to (22.2, 39.4)
- moved RST4 39.4 mm to (22.2, 30.5)
- moved C7 33.2 mm to (31.8, 59.1)
- moved TEMP 23.7 mm to (47.9, 28.4), turned to 180 degrees
- moved C8 19.0 mm to (47.9, 26.0), turned to 0 degrees
- moved RI2C2 5.85 mm to (35.6, 45.1)
- moved RT1 5.43 mm to (29.8, 49.5), turned to 90 degrees
- moved RL1 5.10 mm to (48.3, 50.8), turned to 0 degrees
- moved RL2 5.10 mm to (21.6, 50.8), turned to 180 degrees
- moved RI2C1 3.42 mm to (35.6, 43.8)
- moved C6 2.54 mm to (31.1, 24.8)
- moved C9 2.54 mm to (36.2, 29.8)
- moved C10 1.27 mm to (38.1, 59.1)
- moved C4 1.27 mm to (33.7, 29.8)
- moved CLO1 1.27 mm to (36.2, 59.1)
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Connections:
- net LED1: now also U1.28; no longer U1.29
- net RXD: now also U1.29
- net TXD: now also U1.30
Routing:
- net GND: track 0.00 -> 124.9 mm, vias 0 -> 13
- net +3V3: track 0.00 -> 59.7 mm, vias 0 -> 6
- net NRST: track 0.00 -> 56.5 mm, vias 0 -> 4
- net TXD: track 0.00 -> 39.5 mm, vias 0 -> 2
- net RXD: track 0.00 -> 38.0 mm, vias 0 -> 2
- net LED4: track 0.00 -> 37.6 mm
- net LED3: track 0.00 -> 37.0 mm
- net PRG: track 0.00 -> 28.5 mm
- net +5V: track 0.00 -> 18.8 mm
- net SWCLK: track 0.00 -> 16.4 mm, vias 0 -> 1
- net SWDIO: track 0.00 -> 15.6 mm, vias 0 -> 1
- net I2C_SDA: track 0.00 -> 12.6 mm
- net I2C_SCL: track 0.00 -> 12.4 mm
- net HOST_INT: track 0.00 -> 11.0 mm
- net SENS_3: track 0.00 -> 10.8 mm, vias 0 -> 2
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
Commit message: updates
Parts:
- removed Y1: ABS07-32.768KHZ-7-T, ABS07-32.768KHZ-7-T:ABS-07
- added C11: 0.01uF, rcl:C0402
- added OSC32: ABS07-32.768KHZ-7-T, ABS07-32.768KHZ-7-T:ABS-07
- added OSC8M: ASF1, crystal:ASF
- moved C10 0.63 mm to (38.1, 59.7)
- moved C7 0.63 mm to (31.8, 59.7)
- moved CLO1 0.63 mm to (36.2, 59.7)
- moved CLO2 0.63 mm to (33.7, 59.7)
- renumbered IC1 to SENSBRAIN, U1 to BRAIN
Connections:
- new net SHIELD: SENSBRAIN.9
- net +3V3: now also C11.1, OSC8M.4
- net EXT_CLK: now also OSC8M.3
- net GND: now also C11.2, OSC8M.2; no longer SENSBRAIN.9
- net OSC32_IN: now also OSC32.1; no longer Y1.1
- net OSC32_OUT: now also OSC32.2; no longer Y1.2
Routing:
- net +3V3: track 59.7 -> 91.5 mm, vias 6 -> 7
- net I2C_SCL: track 12.4 -> 35.3 mm, vias 0 -> 2
- net I2C_SDA: track 12.6 -> 32.2 mm
- net GND: track 124.9 -> 135.6 mm, vias 13 -> 14
- net SHIELD: track 0.00 -> 5.92 mm, vias 0 -> 9
- net EXT_CLK: track 0.00 -> 5.64 mm
- net NRST: track 56.5 -> 60.9 mm
- net OSC32_IN: track 5.90 -> 8.73 mm
- net OSC32_OUT: track 6.73 -> 8.34 mm
- added copper zone on layer 1, net SHIELD
Other:
- board text added: "GND"
- board text added: "NRST"
- board text added: "SWCLK"
- board text added: "SWDIO"

Commit message: updates
Parts:
- SIEMENS-BCU: value BCU -> SIEMENS BCU
- renumbered BCU to SIEMENS-BCU
Other:
- board text added: "+5V"
- board text added: "0XCDDC"
- board text added: "4xTouch Button Rev 1.0"
- board text added: "RXD"
- board text added: "TXD"
Changed lines of the file:
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@@
 <drawing>
 <settings>
-<setting alwaysvectorfont="no"/>
+<setting alwaysvectorfont="yes"/>
 <setting verticaltext="up"/>
 </settings>
@@
 <layers>
 <layer number="1" name="Top" color="4" fill="1" visible="yes" active="yes"/>
-<layer number="2" name="Route2" color="1" fill="3" visible="no" active="yes"/>
+<layer number="2" name="Route2" color="1" fill="3" visible="yes" active="yes"/>
 <layer number="3" name="Route3" color="4" fill="3" visible="no" active="no"/>
 <layer number="4" name="Route4" color="1" fill="4" visible="no" active="no"/>
@@
 <layer number="13" name="Route13" color="4" fill="5" visible="no" active="no"/>
 <layer number="14" name="Route14" color="1" fill="6" visible="no" active="no"/>
-<layer number="15" name="Route15" color="4" fill="6" visible="no" active="yes"/>
-<layer number="16" name="Bottom" color="1" fill="1" visible="no" active="yes"/>
+<layer number="15" name="Route15" color="4" fill="6" visible="yes" active="yes"/>
+<layer number="16" name="Bottom" color="1" fill="1" visible="yes" active="yes"/>
 <layer number="17" name="Pads" color="2" fill="1" visible="yes" active="yes"/>
 <layer number="18" name="Vias" color="2" fill="1" visible="yes" active="yes"/>
@@
 <layer number="24" name="bOrigins" color="15" fill="1" visible="yes" active="yes"/>
 <layer number="25" name="tNames" color="7" fill="1" visible="yes" active="yes"/>
-<layer number="26" name="bNames" color="7" fill="1" visible="no" active="yes"/>
+<layer number="26" name="bNames" color="7" fill="1" visible="yes" active="yes"/>
 <layer number="27" name="tValues" color="7" fill="1" visible="no" active="yes"/>
 <layer number="28" name="bValues" color="7" fill="1" visible="no" active="yes"/>
@@
 <text x="46.228" y="28.575" size="1.016" layer="25" rot="R90">NRST</text>
 <text x="48.768" y="29.21" size="1.016" layer="25" rot="R90">GND</text>
+<text x="48.514" y="7.62" size="1.778" layer="26" rot="MR0">4xTouch Button Rev 1.0</text>
+<text x="37.465" y="5.715" size="1.016" layer="26" rot="MR0">0XCDDC</text>
+<text x="30.353" y="10.033" size="1.016" layer="25" rot="R90">+5V</text>
+<text x="40.513" y="9.652" size="1.016" layer="25" rot="R90">GND</text>
+<text x="32.893" y="9.906" size="1.016" layer="25" rot="R90">TXD</text>
+<text x="37.973" y="9.779" size="1.016" layer="25" rot="R90">RXD</text>
 </plain>
 <attributes>
@@
 </autorouter>
 <elements>
-<element name="BCU" library="pinhead" package="2X05SMD" value="BCU" x="31.115" y="18.415" smashed="yes">
-<attribute name="NAME" x="33.1978" y="12.2428" size="1.016" layer="25" ratio="10"/>
+<element name="SIEMENS-BCU" library="pinhead" package="2X05SMD" value="SIEMENS BCU" x="31.115" y="18.415" smashed="yes">
+<attribute name="NAME" x="30.0228" y="16.8148" size="1.016" layer="25" ratio="10"/>
 <attribute name="VALUE" x="28.575" y="12.7" size="1.27" layer="27"/>
 </element>
@@
 <signals>
 <signal name="+5V">
-<contactref element="BCU" pad="1"/>
+<contactref element="SIEMENS-BCU" pad="1"/>
 <contactref element="3V3_REGULATOR" pad="2"/>
 <contactref element="C1" pad="2"/>
@@
 </signal>
 <signal name="TXD">
-<contactref element="BCU" pad="3"/>
+<contactref element="SIEMENS-BCU" pad="3"/>
 <contactref element="BRAIN" pad="30"/>
 <wire x1="37.275" y1="50.9151875" x2="38.069525" y2="50.9151875" width="0.1524" layer="1"/>
 <wire x1="38.069525" y1="50.9151875" x2="38.1" y2="50.9456625" width="0.1524" layer="1"/>
 <via x="38.1" y="50.9456625" extent="1-16" drill="0.35"/>
-<wire x1="38.1" y1="50.9456625" x2="38.1" y2="21.59" width="0.3048" layer="2"/>
+<wire x1="38.1" y1="50.9456625" x2="38.1" y2="21.59" width="0.1524" layer="2"/>
 <wire x1="38.1" y1="21.59" x2="33.655" y2="17.145" width="0.1524" layer="2"/>
 <via x="33.655" y="17.145" extent="1-16" drill="0.35"/>
@@
 </signal>
 <signal name="RXD">
-<contactref element="BCU" pad="7"/>
+<contactref element="SIEMENS-BCU" pad="7"/>
 <contactref element="BRAIN" pad="29"/>
 <wire x1="37.275" y1="50.4150625" x2="38.831525" y2="50.4150625" width="0.1524" layer="1"/>
@@
 </signal>
 <signal name="GND">
-<contactref element="BCU" pad="9"/>
+<contactref element="SIEMENS-BCU" pad="9"/>
 <contactref element="C1" pad="1"/>
 <contactref element="C2" pad="2"/>
@@
 <wire x1="34.675" y1="32.5179" x2="34.675" y2="33.052" width="0.1524" layer="1"/>
 <wire x1="34.675" y1="32.5179" x2="35.1889" y2="32.004" width="0.1524" layer="1"/>
-<polygon width="0.1778" layer="1" spacing="1.778" pour="hatch" isolate="0.889" thermals="no" rank="6">
-<vertex x="1.27" y="1.27"/>
-<vertex x="63.5" y="2.54"/>
-<vertex x="67.31" y="6.35"/>
-<vertex x="67.31" y="63.5"/>
-<vertex x="63.5" y="67.31"/>
-<vertex x="0.635" y="67.31"/>
-</polygon>
 <wire x1="35.1889" y1="32.004" x2="36.068" y2="32.004" width="0.1524" layer="1"/>
 <wire x1="36.068" y1="32.004" x2="36.576" y2="32.004" width="0.1524" layer="1"/>

Commit message: updates
Other:
- board text added: "Konnekting | 0XCDDC | 2018 by ChriD"
- board text removed: "0XCDDC"
Changed lines of the file:
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@@
 <text x="48.768" y="29.21" size="1.016" layer="25" rot="R90">GND</text>
 <text x="48.514" y="7.62" size="1.778" layer="26" rot="MR0">4xTouch Button Rev 1.0</text>
-<text x="37.465" y="5.715" size="1.016" layer="26" rot="MR0">0XCDDC</text>
+<text x="47.498" y="5.207" size="1.016" layer="26" rot="MR0">Konnekting | 0XCDDC | 2018 by ChriD</text>
 <text x="30.353" y="10.033" size="1.016" layer="25" rot="R90">+5V</text>
 <text x="40.513" y="9.652" size="1.016" layer="25" rot="R90">GND</text>
@@
 <via x="55.118" y="28.448" extent="1-16" drill="0.35"/>
 <via x="55.118" y="42.672" extent="1-16" drill="0.35"/>
-<via x="27.432" y="27.432" extent="1-16" drill="0.35"/>
+<via x="27.432" y="28.321" extent="1-16" drill="0.35"/>
 <via x="43.434" y="42.672" extent="1-16" drill="0.35"/>
 <polygon width="0.1778" layer="1" spacing="1.778" pour="hatch" isolate="0.889" thermals="no" rank="6">

Commit message: updates
Connections:
- net RXD renamed USART1_TX
- net TXD renamed USART1_RX
- new net USART2_RX: BRAIN.9
- new net USART2_TX: BRAIN.8
- new net USB_DM: BRAIN.21
- new net USB_DP: BRAIN.22
Routing:
- net USB_DM: track 0.00 -> 16.6 mm, vias 0 -> 2
- net USART2_RX: track 0.00 -> 16.1 mm, vias 0 -> 2
- net USB_DP: track 0.00 -> 14.7 mm, vias 0 -> 2
- net USART2_TX: track 0.00 -> 14.2 mm, vias 0 -> 2
- net SWDIO: track 15.6 -> 21.6 mm
- net SWCLK: track 16.4 -> 20.5 mm
- net GND: track 135.6 -> 137.2 mm, vias 14 -> 15
Other:
- board text added: "4xTouch Button Rev 1.1"
- board text added: "USB_DM"
- board text added: "USB_DP"
- board text removed: "4xTouch Button Rev 1.0"
