File: eagle/4ButtonSwitch.Rev1.sch (EAGLE design)
At the start: 39 parts, among them IC1 CY8CMBR3116-LQXI, U1 STM32L432KX, Y1 ABS07-32.768KHZ-7-T

Commit message: updates
Connections:
- net LED1: now also U1.PB5; no longer U1.PB6
- net RXD: now also U1.PB6
- net TXD: now also U1.PB7
Changed lines of the file:
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@@
 <label x="50.8" y="43.18" size="1.016" layer="95" rot="R270" xref="yes"/>
+</segment>
+<segment>
+<pinref part="U1" gate="A" pin="PB7"/>
+<wire x1="213.36" y1="-55.88" x2="228.6" y2="-55.88" width="0.1524" layer="91"/>
+<label x="228.6" y="-55.88" size="1.016" layer="95" xref="yes"/>
 </segment>
 </net>
@@
 <wire x1="55.88" y1="53.34" x2="55.88" y2="43.18" width="0.1524" layer="91"/>
 <label x="55.88" y="43.18" size="1.016" layer="95" rot="R270" xref="yes"/>
+</segment>
+<segment>
+<pinref part="U1" gate="A" pin="PB6"/>
+<wire x1="213.36" y1="-58.42" x2="228.6" y2="-58.42" width="0.1524" layer="91"/>
+<label x="228.6" y="-58.42" size="1.016" layer="95" xref="yes"/>
 </segment>
 </net>
@@
 </segment>
 <segment>
-<pinref part="IC1" gate="G$1" pin="CS15/SH/!HI"/>
-<wire x1="274.32" y1="-12.7" x2="274.32" y2="-17.78" width="0.1524" layer="91"/>
-<wire x1="274.32" y1="-17.78" x2="276.86" y2="-17.78" width="0.1524" layer="91"/>
 <pinref part="IC1" gate="G$1" pin="CS12/GP14"/>
 <wire x1="276.86" y1="-17.78" x2="279.4" y2="-17.78" width="0.1524" layer="91"/>
@@
 <pinref part="IC1" gate="G$1" pin="CS14/GPO6"/>
 <wire x1="276.86" y1="-12.7" x2="276.86" y2="-17.78" width="0.1524" layer="91"/>
-<junction x="276.86" y="-17.78"/>
 <wire x1="281.94" y1="-17.78" x2="287.02" y2="-17.78" width="0.1524" layer="91"/>
 <junction x="281.94" y="-17.78"/>
 <label x="287.02" y="-17.78" size="1.016" layer="95" xref="yes"/>
+<pinref part="IC1" gate="G$1" pin="CS15/SH/!HI"/>
+<wire x1="274.32" y1="-12.7" x2="274.32" y2="-17.78" width="0.1524" layer="91"/>
+<wire x1="274.32" y1="-17.78" x2="276.86" y2="-17.78" width="0.1524" layer="91"/>
+<junction x="276.86" y="-17.78"/>
 </segment>
 <segment>
@@
 </segment>
 <segment>
-<pinref part="U1" gate="A" pin="PB6"/>
-<wire x1="213.36" y1="-58.42" x2="228.6" y2="-58.42" width="0.1524" layer="91"/>
-<label x="228.6" y="-58.42" size="1.016" layer="95" xref="yes"/>
-</segment>
-</net>
+<pinref part="U1" gate="A" pin="PB5"/>
+<wire x1="213.36" y1="-60.96" x2="228.6" y2="-60.96" width="0.1524" layer="91"/>
+<label x="228.6" y="-60.96" size="1.016" layer="95" xref="yes"/>
+</segment>
+</net>

Commit message: updates
Parts:
- added C11: 0.01uF, rcl:C-EUC0402
- added OSC8M: ASF1, crystal:ASF1
- renumbered IC1 to SENSBRAIN, U1 to BRAIN, Y1 to OSC32
Connections:
- new net SHIELD: SENSBRAIN.CS15/SH/!HI
- net +3V3: now also C11.1, OSC8M.VCC
- net EXT_CLK: now also OSC8M.FO
- net GND: now also C11.2, OSC8M.GND; no longer SENSBRAIN.CS15/SH/!HI

Commit message: updates
Parts:
- SIEMENS-BCU: value BCU -> SIEMENS BCU
- renumbered BCU to SIEMENS-BCU
Other:
- note added: "ASFL-1-8.000"
Changed lines of the file:
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@@
 </classes>
 <parts>
-<part name="BCU" library="pinhead" deviceset="PINHD-2X5" device="_2.54-SMD" value="BCU"/>
+<part name="SIEMENS-BCU" library="pinhead" deviceset="PINHD-2X5" device="_2.54-SMD" value="SIEMENS BCU"/>
 <part name="3V3_REGULATOR" library="MCP1703T-3302E_MB" deviceset="MCP1703T-3302E_MB" device=""/>
 <part name="+3V1" library="supply1" library_urn="urn:adsk.eagle:library:371" deviceset="+3V3" device=""/>
@@
 <text x="276.86" y="-60.96" size="1.016" layer="91">I2C READ: 0xBF
 I2C WRITE: 0xBE</text>
+<text x="101.6" y="-132.08" size="1.778" layer="91">ASFL-1-8.000</text>
 </plain>
 <instances>
-<instance part="BCU" gate="A" x="53.34" y="55.88" rot="R90"/>
+<instance part="SIEMENS-BCU" gate="A" x="53.34" y="55.88" rot="R90"/>
 <instance part="3V3_REGULATOR" gate="G$1" x="40.64" y="20.32"/>
 <instance part="+3V1" gate="G$1" x="22.86" y="63.5"/>
@@
 <net name="+5V" class="0">
 <segment>
-<pinref part="BCU" gate="A" pin="1"/>
+<pinref part="SIEMENS-BCU" gate="A" pin="1"/>
 <wire x1="48.26" y1="53.34" x2="48.26" y2="43.18" width="0.1524" layer="91"/>
 <label x="48.26" y="43.18" size="1.016" layer="95" rot="R270" xref="yes"/>
@@
 <net name="TXD" class="0">
 <segment>
-<pinref part="BCU" gate="A" pin="3"/>
+<pinref part="SIEMENS-BCU" gate="A" pin="3"/>
 <wire x1="50.8" y1="53.34" x2="50.8" y2="43.18" width="0.1524" layer="91"/>
 <label x="50.8" y="43.18" size="1.016" layer="95" rot="R270" xref="yes"/>
@@
 <net name="RXD" class="0">
 <segment>
-<pinref part="BCU" gate="A" pin="7"/>
+<pinref part="SIEMENS-BCU" gate="A" pin="7"/>
 <wire x1="55.88" y1="53.34" x2="55.88" y2="43.18" width="0.1524" layer="91"/>
 <label x="55.88" y="43.18" size="1.016" layer="95" rot="R270" xref="yes"/>
@@
 <net name="GND" class="0">
 <segment>
-<pinref part="BCU" gate="A" pin="9"/>
+<pinref part="SIEMENS-BCU" gate="A" pin="9"/>
 <wire x1="58.42" y1="53.34" x2="58.42" y2="43.18" width="0.1524" layer="91"/>
 <label x="58.42" y="43.18" size="1.016" layer="95" rot="R270" xref="yes"/>

Commit message: updates
Other:
- note added: "I2C Adr.: 0x37"
- note added: "WM17451-ND"
Changed lines of the file:
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@@
 I2C WRITE: 0xBE</text>
 <text x="101.6" y="-132.08" size="1.778" layer="91">ASFL-1-8.000</text>
+<text x="243.84" y="43.18" size="1.778" layer="91">I2C Adr.: 0x37</text>
+<text x="243.84" y="43.18" size="1.778" layer="91">I2C Adr.: 0x37</text>
+<text x="45.72" y="63.5" size="1.778" layer="91">WM17451-ND
+</text>
 </plain>
 <instances>

Commit message: updates
Connections:
- net RXD renamed USART1_TX
- net TXD renamed USART1_RX
- new net USART2_RX: BRAIN.PA3
- new net USART2_TX: BRAIN.PA2
- new net USB_DM: BRAIN.PA11
- new net USB_DP: BRAIN.PA12
Other:
- note added: "TODO: * I2C Pins auf VIAS"
Changed lines of the file:
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@@
 <text x="45.72" y="63.5" size="1.778" layer="91">WM17451-ND
+</text>
+<text x="162.56" y="-22.86" size="1.778" layer="91">TODO:
+* I2C Pins auf VIAS
 </text>
 </plain>
@@
 </segment>
 </net>
-<net name="TXD" class="0">
-<segment>
-<pinref part="SIEMENS-BCU" gate="A" pin="3"/>
-<wire x1="50.8" y1="53.34" x2="50.8" y2="43.18" width="0.1524" layer="91"/>
-<label x="50.8" y="43.18" size="1.016" layer="95" rot="R270" xref="yes"/>
-</segment>
-<segment>
-<pinref part="BRAIN" gate="A" pin="PB7"/>
-<wire x1="213.36" y1="-55.88" x2="228.6" y2="-55.88" width="0.1524" layer="91"/>
-<label x="228.6" y="-55.88" size="1.016" layer="95" xref="yes"/>
-</segment>
-</net>
-<net name="RXD" class="0">
-<segment>
-<pinref part="SIEMENS-BCU" gate="A" pin="7"/>
-<wire x1="55.88" y1="53.34" x2="55.88" y2="43.18" width="0.1524" layer="91"/>
-<label x="55.88" y="43.18" size="1.016" layer="95" rot="R270" xref="yes"/>
-</segment>
-<segment>
-<pinref part="BRAIN" gate="A" pin="PB6"/>
-<wire x1="213.36" y1="-58.42" x2="228.6" y2="-58.42" width="0.1524" layer="91"/>
-<label x="228.6" y="-58.42" size="1.016" layer="95" xref="yes"/>
-</segment>
-</net>
 <net name="GND" class="0">
 <segment>
@@
 </segment>
 </net>
+<net name="USB_DP" class="0">
+<segment>
+<pinref part="BRAIN" gate="A" pin="PA12"/>
+<wire x1="213.36" y1="-76.2" x2="228.6" y2="-76.2" width="0.1524" layer="91"/>
+<label x="228.6" y="-76.2" size="1.016" layer="95" xref="yes"/>
+</segment>
+</net>
+<net name="USB_DM" class="0">
+<segment>
+<pinref part="BRAIN" gate="A" pin="PA11"/>
+<wire x1="213.36" y1="-78.74" x2="228.6" y2="-78.74" width="0.1524" layer="91"/>
+<label x="228.6" y="-78.74" size="1.016" layer="95" xref="yes"/>
+</segment>
+</net>
+<net name="USART2_TX" class="0">
+<segment>
+<pinref part="BRAIN" gate="A" pin="PA2"/>
+<wire x1="147.32" y1="-66.04" x2="132.08" y2="-66.04" width="0.1524" layer="91"/>
+<label x="132.08" y="-66.04" size="1.016" layer="95" rot="R180" xref="yes"/>
+</segment>
+</net>
+<net name="USART2_RX" class="0">
+<segment>
+<pinref part="BRAIN" gate="A" pin="PA3"/>
+<wire x1="147.32" y1="-68.58" x2="132.08" y2="-68.58" width="0.1524" layer="91"/>
+<label x="132.08" y="-68.58" size="1.016" layer="95" rot="R180" xref="yes"/>
+</segment>
+</net>
+<net name="USART1_RX" class="0">
+<segment>
+<pinref part="BRAIN" gate="A" pin="PB7"/>
+<wire x1="213.36" y1="-55.88" x2="228.6" y2="-55.88" width="0.1524" layer="91"/>
+<label x="228.6" y="-55.88" size="1.016" layer="95" xref="yes"/>
+</segment>
+<segment>
+<pinref part="SIEMENS-BCU" gate="A" pin="3"/>
+<wire x1="50.8" y1="53.34" x2="50.8" y2="43.18" width="0.1524" layer="91"/>
+<label x="50.8" y="43.18" size="1.016" layer="95" rot="R270" xref="yes"/>
+</segment>
+</net>
+<net name="USART1_TX" class="0">
+<segment>
+<pinref part="BRAIN" gate="A" pin="PB6"/>
+<wire x1="213.36" y1="-58.42" x2="228.6" y2="-58.42" width="0.1524" layer="91"/>
+<label x="228.6" y="-58.42" size="1.016" layer="95" xref="yes"/>
+</segment>
+<segment>
+<pinref part="SIEMENS-BCU" gate="A" pin="7"/>
+<wire x1="55.88" y1="53.34" x2="55.88" y2="43.18" width="0.1524" layer="91"/>
+<label x="55.88" y="43.18" size="1.016" layer="95" rot="R270" xref="yes"/>
+</segment>
+</net>
