File: eagle/4ButtonSwitch.Rev2.sch (EAGLE design)
At the start: 42 parts, among them IC1 STM32F303RET6

Commit message: Rev 2
Parts:
- removed PRG2, RST1: 0, wirepad:SMD5
- added GND_NRST, NRST1: 0, wirepad:SMD5
- renumbered IC1 to MCU, RST4 to GND_PRG, SENSBRAIN to SENSORMCU
Connections:
- net N$18 renamed USART3_RX
- net N$23 renamed USART3_TX
- removed net N$1: MCU.VDD_3
- removed net N$10: MCU.VDDA
- removed net N$11: MCU.VSSA
- removed net N$12: MCU.NRST
- removed net N$13: MCU.BOOT0
- removed net N$14: MCU.PA2
- removed net N$15: MCU.PA3
- removed net N$16: MCU.PC4
- removed net N$17: MCU.PC5
- removed net N$2: MCU.VSS_3
- removed net N$3: MCU.VDD_4
- removed net N$4: MCU.VSS_4
- removed net N$5: MCU.VBAT
- removed net N$6: MCU.VSS_1
- removed net N$7: MCU.VDD_1
- removed net N$8: MCU.VDD_2
- removed net N$9: MCU.VSS_2
- removed net USB_DM: BRAIN.PA11
- removed net USB_DP: BRAIN.PA12
- new net I2C1_SCL: MCU.PB6
- new net I2C1_SDA: MCU.PB7
- new net I2C2_SCL: MCU.PF1-OSC_OUT
- new net I2C2_SDA: MCU.PF0-OSC_IN
- new net I2C3_SCL: MCU.PA8
- new net I2C3_SDA: MCU.PC9
- net +3V3: now also C10.2, C9.1, MCU.VBAT, MCU.VDDA, MCU.VDD_1, MCU.VDD_2, MCU.VDD_3, MCU.VDD_4; no longer BRAIN.VDD, BRAIN.VDDA/VREF+, BRAIN.VDD_2, C10.1, C9.2
- net GND: now also C10.1, C9.2, GND_NRST.P, MCU.BOOT0, MCU.VSSA, MCU.VSS_1, MCU.VSS_2, MCU.VSS_3, MCU.VSS_4; no longer BRAIN.PH3-BOOT0, BRAIN.VSS, BRAIN.VSS_2, C10.2, C9.1, PRG2.P
- net I2C_SCL: no longer BRAIN.PA9
- net I2C_SDA: no longer BRAIN.PA10
- net NRST: now also MCU.NRST, NRST1.P; no longer BRAIN.NRST, RST1.P
- net OSC32_IN: now also MCU.PC14-OSC32_IN; no longer BRAIN.PC14-OSC32_IN
- net OSC32_OUT: now also MCU.PC15-OSC32_OUT; no longer BRAIN.PC15-OSC32_OUT
- net PRG: now also MCU.PA5; no longer BRAIN.PA5
- net SWCLK: now also MCU.PA14; no longer BRAIN.PA14
- net SWDIO: now also MCU.PA13; no longer BRAIN.PA13
- net USART1_RX: now also MCU.PC5; no longer BRAIN.PB7
- net USART1_TX: now also MCU.PC4; no longer BRAIN.PB6
- net USART2_RX: now also MCU.PA3; no longer BRAIN.PA3
- net USART2_TX: now also MCU.PA2; no longer BRAIN.PA2
Other:
- moved on the sheet: C10, C7, C9

Commit message: Rev 2
Parts:
- removed BRAIN: STM32L432KX, STM32L432KC:STM32L432KX
- removed C11: 0.01uF, rcl:C-EUC0402
- removed OSC8M: ASF1, crystal:ASF1
- added C12, C13, C14: 100nf, rcl:C-EUC0402
- C4, C7: value 0.1uF -> 100nF
Connections:
- removed net EXT_CLK: BRAIN.PA0-CK_IN, OSC8M.FO
- net +3V3: now also C12.1, C13.2, C14.1; no longer C11.1, OSC8M.VCC
- net GND: now also C12.2, C13.1, C14.2, SENSORMCU.EP_GND; no longer C11.2, OSC8M.GND
- net HOST_INT: now also MCU.PC3; no longer BRAIN.PA8
- net LED1: now also MCU.PA11; no longer BRAIN.PB5
- net LED2: now also MCU.PB9; no longer BRAIN.PA4
- net LED3: now also MCU.PA10; no longer BRAIN.PB4
- net LED4: now also MCU.PA4; no longer BRAIN.PA6
Other:
- note removed: "ASFL-1-8.000"
- moved on the sheet: C10, C7, C9, GND_NRST, MCU, NRST1, RI2C1, RI2C2, RP1, RP2, RS1, RS2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

Commit message: rev 2
Parts:
- LED1, LED2, LED3, LED4: value WL-SMRW156120BS75300-B_RVS-MOUNT -> LWP4-BOTTOM; device Wurth_Elektronik_Optoelectronics_rev15b (1):WL-SMRW156120BS75300-B_RVS-MOUNT -> led:LWP4-BOTTOM
Connections:
- net GND: now also LED1.C, LED2.C, LED3.C, LED4.C, SENSORMCU.CS7; no longer LED1.K, LED2.K, LED3.K, LED4.K, SENSORMCU.CS9/GPO1
- net IC_SENS_1: now also SENSORMCU.CS2/GUARD; no longer SENSORMCU.CS6
- net IC_SENS_2: now also SENSORMCU.CS3; no longer SENSORMCU.CS2/GUARD
- net IC_SENS_3: now also SENSORMCU.CS6; no longer SENSORMCU.CS7
- net IC_SENS_4: now also SENSORMCU.CS9/GPO1; no longer SENSORMCU.CS3
- net IC_SENS_PROX_1: now also SENSORMCU.CS1/PS1; no longer SENSORMCU.CS0/PS0
- net IC_SENS_PROX_2: now also SENSORMCU.CS0/PS0; no longer SENSORMCU.CS1/PS1
Other:
- note added: "LEDS OSRAM LW P473"
