File: eagle/4ButtonSwitch.Rev2.brd (EAGLE design)
At the start: 69.8 x 69.8 mm, 44 parts, among them IC1 STM32F303RET6

Commit message: Rev 2
Parts:
- moved C10 51.4 mm to (-5.08, 31.8)
- moved RT1 45.5 mm to (-12.1, 31.8)
- moved C9 44.4 mm to (-4.45, 47.6)
- moved C11 18.2 mm to (12.1, 48.9)
- moved C5 14.8 mm to (35.6, 29.8)
- moved C7 6.35 mm to (38.1, 59.7)
- renumbered IC1 to MCU, PRG2 to GND_NRST, RST1 to NRST1, RST4 to GND_PRG, SENSBRAIN to SENSORMCU
Connections:
- net N$18 renamed USART3_RX
- net N$23 renamed USART3_TX
- removed net N$1: MCU.48
- removed net N$10: MCU.13
- removed net N$11: MCU.12
- removed net N$12: MCU.7
- removed net N$13: MCU.60
- removed net N$14: MCU.16
- removed net N$15: MCU.17
- removed net N$16: MCU.24
- removed net N$17: MCU.25
- removed net N$2: MCU.47
- removed net N$3: MCU.64
- removed net N$4: MCU.63
- removed net N$5: MCU.1
- removed net N$6: MCU.18
- removed net N$7: MCU.19
- removed net N$8: MCU.32
- removed net N$9: MCU.31
- removed net USB_DM: BRAIN.21
- removed net USB_DP: BRAIN.22
- new net I2C1_SCL: MCU.58
- new net I2C1_SDA: MCU.59
- new net I2C2_SCL: MCU.6
- new net I2C2_SDA: MCU.5
- new net I2C3_SCL: MCU.41
- new net I2C3_SDA: MCU.40
- new net VDD: BRAIN.17
- new net VDDA/VREF+: BRAIN.5
- new net VDD_2: BRAIN.1
- new net VSS: BRAIN.32
- new net VSS_2: BRAIN.16
- net +3V3: now also C10.2, C9.1, MCU.1, MCU.13, MCU.19, MCU.32, MCU.48, MCU.64; no longer BRAIN.1, BRAIN.17, BRAIN.5, C10.1, C9.2
- net GND: now also C10.1, C9.2, MCU.12, MCU.18, MCU.31, MCU.47, MCU.60, MCU.63; no longer BRAIN.16, BRAIN.31, BRAIN.32, C10.2, C9.1
- net I2C_SCL: no longer BRAIN.19
- net I2C_SDA: no longer BRAIN.20
- net NRST: now also MCU.7; no longer BRAIN.4
- net OSC32_IN: now also MCU.3; no longer BRAIN.2
- net OSC32_OUT: now also MCU.4; no longer BRAIN.3
- net PRG: now also MCU.21; no longer BRAIN.11
- net SWCLK: now also MCU.49; no longer BRAIN.24
- net SWDIO: now also MCU.46; no longer BRAIN.23
- net USART1_RX: now also MCU.25; no longer BRAIN.30
- net USART1_TX: now also MCU.24; no longer BRAIN.29
- net USART2_RX: now also MCU.17; no longer BRAIN.9
- net USART2_TX: now also MCU.16; no longer BRAIN.8
Routing:
- net LED4: track 37.6 -> 0.00 mm
- net LED3: track 37.0 -> 0.23 mm
- net I2C_SCL: track 35.3 -> 0.00 mm, vias 2 -> 0
- net I2C_SDA: track 32.2 -> 0.00 mm
- net SWDIO: track 21.6 -> 0.00 mm
- net NRST: track 21.0 -> 0.01 mm, vias 2 -> 1
- net SWCLK: track 20.5 -> 0.00 mm
- net USART2_RX: track 16.1 -> 0.00 mm, vias 2 -> 1
- net USART2_TX: track 14.2 -> 0.00 mm, vias 2 -> 1
- net GND: track 25.1 -> 12.3 mm, vias 9 -> 5
- net SENS_2: track 11.2 -> 0.00 mm
- net HOST_INT: track 11.0 -> 0.00 mm
- net SENS_3: track 10.8 -> 0.00 mm
- net LED1: track 10.7 -> 0.00 mm
- net LED2: track 10.6 -> 0.00 mm
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Other:
- board text added: "4xTouch Button Rev 2.0"
- board text removed: "4xTouch Button Rev 1.1"

Commit message: Rev 2
Parts:
- removed BRAIN: STM32L432KX, STM32L432KC:UFQFPN32-5X5MM
- removed C11: 0.01uF, rcl:C0402
- removed OSC8M: ASF1, crystal:ASF
- added C12, C13, C14: 100nf, rcl:C0402
- C4, C7: value 0.1uF -> 100nF
- moved RT1 56.1 mm to (43.8, 27.3), turned to 180 degrees
- moved C10 54.7 mm to (49.5, 29.2), turned to 180 degrees
- moved C9 54.4 mm to (49.5, 40.6), turned to 0 degrees
- moved MCU 54.3 mm to (43.8, 34.9)
- moved C7 24.3 mm to (35.6, 35.6), turned to 180 degrees
- moved CLO2 22.9 mm to (33.0, 36.8), turned to 0 degrees
- moved CLO1 20.6 mm to (33.0, 39.4), turned to 0 degrees
- moved OSC32 17.8 mm to (35.6, 38.1), turned to 270 degrees
- moved RS1 11.7 mm to (28.6, 38.7), turned to 270 degrees
- moved RS3 11.3 mm to (29.2, 31.8), turned to 90 degrees
- moved C8 10.2 mm to (58.0, 24.8)
- moved TEMP 10.2 mm to (58.0, 27.2)
- moved C4 8.89 mm to (24.8, 29.8)
- moved C5 8.89 mm to (26.7, 29.8)
- moved RP1 8.89 mm to (21.0, 37.5)
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Connections:
- removed net EP_GND: SENSORMCU.25
- removed net EXT_CLK: BRAIN.6, OSC8M.3
- removed net VDD: BRAIN.17
- removed net VDDA/VREF+: BRAIN.5
- removed net VDD_2: BRAIN.1
- removed net VSS: BRAIN.32
- removed net VSS_2: BRAIN.16
- net +3V3: now also C12.1, C13.2, C14.1; no longer C11.1, OSC8M.4
- net GND: now also C12.2, C13.1, C14.2, SENSORMCU.25; no longer C11.2, OSC8M.2
- net HOST_INT: now also MCU.11; no longer BRAIN.18
- net LED1: now also MCU.44; no longer BRAIN.28
- net LED2: now also MCU.62; no longer BRAIN.10
- net LED3: now also MCU.43; no longer BRAIN.27
- net LED4: now also MCU.20; no longer BRAIN.12
Routing:
- net GND: track 12.3 -> 1.41 mm, vias 5 -> 1
- net +3V3: track 3.14 -> 0.00 mm
- net OSC32_IN: track 0.64 -> 0.00 mm
- net OSC32_OUT: track 0.60 -> 0.00 mm
- net SENS_PROX_2: vias 2 -> 0
- net SENS_PROX_1: vias 2 -> 0

Commit message: rev 2
Parts:
- LED1, LED2, LED3, LED4: value WL-SMRW156120BS75300-B_RVS-MOUNT -> LWP4-BOTTOM; device Wurth_Elektronik_Optoelectronics_rev15b (1):WL-SMRW-1206-CYLDR-REVERSE-MOUNT -> led:P47F-BOTTOM
- moved GND_NRST 54.8 mm to (62.9, 40.0)
- moved PRG1 54.8 mm to (62.9, 29.8)
- moved RT1 20.5 mm to (33.7, 45.1), turned to 270 degrees
- moved RI2C1 14.4 mm to (26.0, 33.0), turned to 270 degrees
- moved RI2C2 13.0 mm to (26.0, 36.2), turned to 90 degrees
- moved C5 12.6 mm to (18.4, 39.4), turned to 270 degrees
- moved C4 10.8 mm to (19.7, 39.4), turned to 90 degrees
- moved C3 9.86 mm to (21.0, 39.4), turned to 90 degrees
- moved C7 9.55 mm to (34.9, 45.1), turned to 90 degrees
- moved RS3 6.63 mm to (22.9, 29.8)
- moved RL1 5.39 mm to (52.1, 47.0), turned to 90 degrees
- moved RL2 5.39 mm to (17.8, 47.0), turned to 90 degrees
- moved RS2 5.24 mm to (22.2, 39.4), turned to 270 degrees
- moved RP2 4.96 mm to (24.8, 39.4), turned to 270 degrees
- moved SENSORMCU 3.86 mm to (22.2, 34.4), turned to 270 degrees
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Connections:
- net GND: now also LED1.C, LED2.C, LED3.C, LED4.C, SENSORMCU.17; no longer LED1.1, LED2.1, LED3.1, LED4.1, SENSORMCU.15
- net IC_SENS_1: now also SENSORMCU.3; no longer SENSORMCU.18
- net IC_SENS_2: now also SENSORMCU.4; no longer SENSORMCU.3
- net IC_SENS_3: now also SENSORMCU.18; no longer SENSORMCU.17
- net IC_SENS_4: now also SENSORMCU.15; no longer SENSORMCU.4
- net IC_SENS_PROX_1: now also SENSORMCU.2; no longer SENSORMCU.1
- net IC_SENS_PROX_2: now also SENSORMCU.1; no longer SENSORMCU.2
- net N$19: now also LED1.A; no longer LED1.2
- net N$20: now also LED2.A; no longer LED2.2
- net N$21: now also LED3.A; no longer LED3.2
- net N$22: now also LED4.A; no longer LED4.2
Routing:
- net SENS_PROX_2: track 117.5 -> 145.6 mm, vias 0 -> 3
- net GND: track 1.41 -> 27.9 mm, vias 1 -> 9
- net +3V3: track 0.00 -> 24.7 mm, vias 0 -> 3
- net SENS_PROX_1: track 117.5 -> 140.1 mm, vias 0 -> 3
- net SENS_3: track 0.00 -> 21.1 mm, vias 1 -> 2
- net SENS_1: track 0.00 -> 18.1 mm, vias 1 -> 2
- net +5V: track 3.55 -> 18.9 mm
- net IC_SENS_1: track 0.00 -> 5.49 mm, vias 0 -> 2
- net SENS_2: track 0.00 -> 4.43 mm, vias 1 -> 2
- net SENS_4: track 0.00 -> 4.06 mm, vias 1 -> 2
- net VCC: track 0.00 -> 3.35 mm
- net IC_SENS_PROX_2: track 0.00 -> 2.84 mm
- net IC_SENS_PROX_1: track 0.00 -> 2.52 mm
- net IC_SENS_2: track 0.00 -> 2.41 mm
- net IC_SENS_3: track 0.00 -> 2.18 mm
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
Commit message: rev 2
Parts:
- moved RT1 22.5 mm to (49.5, 29.2), turned to 0 degrees
- moved C7 9.55 mm to (35.6, 35.6), turned to 270 degrees
- moved RI2C1 6.87 mm to (31.8, 36.8), turned to 90 degrees
- moved OSC32 5.99 mm to (30.5, 40.0), turned to 180 degrees
- moved CLO2 4.02 mm to (34.3, 38.7), turned to 270 degrees
- moved RI2C2 3.24 mm to (29.2, 36.8)
- moved C10 1.27 mm to (49.5, 27.9)
- moved C8 0.81 mm to (55.0, 26.7)
- moved C14 0.63 mm to (35.6, 32.4)
- moved CLO1 0.63 mm to (35.6, 38.7)
Routing:
- net GND: track 27.9 -> 115.0 mm, vias 9 -> 17
- net NRST: track 0.00 -> 32.9 mm, vias 1 -> 2
- net LED4: track 0.00 -> 26.8 mm
- net LED2: track 0.00 -> 26.7 mm
- net USART1_RX: track 0.00 -> 23.4 mm, vias 0 -> 2
- net USART1_TX: track 0.00 -> 18.0 mm
- net HOST_INT: track 0.00 -> 17.4 mm, vias 0 -> 2
- net LED3: track 0.00 -> 14.5 mm, vias 0 -> 2
- net +3V3: track 24.7 -> 10.9 mm, vias 3 -> 0
- net LED1: track 0.00 -> 11.3 mm, vias 0 -> 2
- net I2C_SDA: track 0.00 -> 11.1 mm, vias 0 -> 1
- net SWDIO: track 0.00 -> 10.4 mm
- net OSC32_OUT: track 0.00 -> 10.0 mm
- net SWCLK: track 0.00 -> 9.90 mm
- net USART2_RX: track 0.00 -> 9.78 mm
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- added copper zone on layer 1, net +3V3
