File: eagle/4ButtonSwitch.Rev2.1.brd (EAGLE design)
At the start: 69.8 x 69.8 mm, 44 parts

Commit message: Rev2.1
Parts:
- added C11: 4.7uf, rcl:C0402
- C14: value 100nf -> 10nf
- moved RI2C2 22.8 mm to (51.4, 31.8), turned to 270 degrees
- moved RI2C1 19.1 mm to (50.2, 31.8), turned to 270 degrees
- moved RP2 12.6 mm to (16.5, 29.8), turned to 90 degrees
- moved C5 10.0 mm to (21.6, 29.8), turned to 90 degrees
- moved C3 9.71 mm to (19.1, 29.8), turned to 270 degrees
- moved C4 9.55 mm to (20.3, 29.8), turned to 270 degrees
- moved CLO2 9.09 mm to (27.3, 33.7), turned to 0 degrees
- moved CLO1 7.75 mm to (27.3, 36.2), turned to 0 degrees
- moved RT1 7.10 mm to (50.2, 28.6), turned to 270 degrees
- moved RP1 7.01 mm to (16.5, 40.0)
- moved OSC32 5.08 mm to (30.5, 34.9), turned to 270 degrees
- moved C8 4.03 mm to (51.4, 28.6), turned to 90 degrees
- moved RS4 3.81 mm to (17.8, 29.8)
- moved RS1 2.62 mm to (23.5, 40.0)
- moved C10 1.27 mm to (48.3, 28.6)
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Connections:
- removed net I2C3_SCL: MCU.41
- removed net I2C3_SDA: MCU.40
- net +3V3: now also C11.1
- net GND: now also C11.2, SENSORMCU.3; no longer SENSORMCU.19
- net I2C_SCL: now also MCU.41
- net I2C_SDA: now also MCU.40
- net IC_SENS_1: now also SENSORMCU.18; no longer SENSORMCU.3
- net IC_SENS_2: now also SENSORMCU.19; no longer SENSORMCU.4
- net IC_SENS_3: now also SENSORMCU.15; no longer SENSORMCU.18
- net IC_SENS_4: now also SENSORMCU.4; no longer SENSORMCU.15
- net IC_SENS_PROX_1: now also SENSORMCU.1; no longer SENSORMCU.2
- net IC_SENS_PROX_2: now also SENSORMCU.2; no longer SENSORMCU.1
Routing:
- net GND: track 35.8 -> 89.8 mm, vias 11 -> 16
- net +3V3: track 25.0 -> 55.9 mm
- net SENS_PROX_2: track 147.5 -> 117.5 mm, vias 3 -> 2
- net SENS_PROX_1: track 140.1 -> 117.5 mm, vias 3 -> 2
- net SENS_3: track 21.1 -> 0.00 mm, vias 2 -> 1
- net SENS_1: track 18.1 -> 0.00 mm, vias 2 -> 1
- net +5V: track 2.12 -> 19.8 mm
- net OSC32_OUT: track 0.00 -> 11.5 mm
- net OSC32_IN: track 0.00 -> 9.49 mm
- net I2C_SCL: track 0.00 -> 4.66 mm
- net SENS_2: track 4.43 -> 0.00 mm, vias 2 -> 1
- net SENS_4: track 4.06 -> 0.00 mm, vias 2 -> 1
- net I2C_SDA: track 0.00 -> 3.63 mm
- net VCC: track 0.00 -> 3.61 mm
Other:
- board text added: "4xTouch Button Rev 2.1"
- board text removed: "4xTouch Button Rev 2.0"

Commit message: Rev 2.1
Parts:
- moved RP2 4.58 mm to (19.1, 33.7)
- moved RP1 4.07 mm to (19.1, 36.8)
- moved C3 1.27 mm to (20.3, 29.8)
- moved C4 1.27 mm to (21.6, 29.8)
- moved C5 1.27 mm to (22.9, 29.8)
- moved RS1 1.27 mm to (24.8, 40.0)
- moved RS2 1.27 mm to (23.5, 40.0)
- moved RS3 1.27 mm to (24.8, 29.8)
- moved RS4 1.27 mm to (19.1, 29.8)
- moved SENSORMCU 1.27 mm to (22.9, 35.1)
- moved CLO1 0.90 mm to (27.9, 35.6)
- moved CLO2 0.90 mm to (27.9, 34.3)
- moved OSC32 0.63 mm to (31.1, 34.9)
Connections:
- net GND: now also SENSORMCU.15; no longer SENSORMCU.12
- net IC_SENS_3: now also SENSORMCU.12; no longer SENSORMCU.15
Routing:
- net USART1_RX: track 0.00 -> 24.2 mm
- net USART1_TX: track 0.00 -> 20.7 mm, vias 0 -> 2
- net SENS_PROX_2: track 117.5 -> 136.3 mm, vias 2 -> 3
- net SENS_PROX_1: track 117.5 -> 136.1 mm, vias 2 -> 3
- net SENS_3: track 0.00 -> 17.2 mm, vias 1 -> 2
- net SENS_1: track 0.00 -> 17.2 mm, vias 1 -> 2
- net GND: track 89.8 -> 105.9 mm, vias 16 -> 21
- net SWCLK: track 0.00 -> 12.0 mm
- net SWDIO: track 0.00 -> 11.4 mm
- net USART2_TX: track 0.00 -> 7.36 mm
- net USART2_RX: track 0.00 -> 6.84 mm, vias 1 -> 3
- net IC_SENS_4: track 0.00 -> 5.37 mm
- net CMOD: track 0.00 -> 4.45 mm
- net SENS_4: track 0.00 -> 3.80 mm, vias 1 -> 2
- net SENS_2: track 0.00 -> 3.80 mm, vias 1 -> 2
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
Commit message: Rev 2.1
Parts:
- added S1: PCM12SMTR, PCM12SMTR:PCM12SMTR_1
Connections:
- new net SHIELD_OR_GND: S1.2
- net GND: now also S1.1
- net PRG: now also MCU.28; no longer MCU.21
- net SHIELD: now also S1.3
Routing:
- net I2C_SCL: track 4.66 -> 48.2 mm, vias 1 -> 3
- net I2C_SDA: track 3.63 -> 42.7 mm, vias 1 -> 4
- net LED4: track 0.00 -> 31.8 mm, vias 0 -> 2
- net NRST: track 1.91 -> 32.2 mm, vias 0 -> 2
- net LED2: track 0.00 -> 25.5 mm
- net PRG: track 0.00 -> 22.9 mm
- net HOST_INT: track 0.00 -> 20.5 mm, vias 0 -> 2
- net LED3: track 0.00 -> 15.3 mm, vias 0 -> 2
- net LED1: track 0.00 -> 13.1 mm, vias 0 -> 2
- net +3V3: track 52.8 -> 59.4 mm
- net GND: track 105.9 -> 111.1 mm, vias 21 -> 24
- net OSC32_OUT: track 8.53 -> 11.3 mm
- net OSC32_IN: track 6.83 -> 9.61 mm
- added copper zone on layer 1, net SHIELD_OR_GND
- added copper zone on layer 16, net SHIELD_OR_GND
- removed copper zone on layer 1, net SHIELD
- removed copper zone on layer 16, net SHIELD

Commit message: Rev 2.1
Parts:
- moved GND_NRST 56.8 mm to (6.99, 29.8)
- moved GND_PRG 56.8 mm to (62.9, 40.0)
- moved C13 0.64 mm to (39.4, 27.3)
- renumbered NRST1 to NRST, PRG1 to PRG
Routing:
- net SENS_PROX_2: track 136.3 -> 133.4 mm
- net SENS_PROX_1: track 136.1 -> 133.1 mm
- net SENS_3: track 17.2 -> 18.8 mm
- net SENS_1: track 17.2 -> 18.8 mm
- net SHIELD_OR_GND: track 0.00 -> 1.43 mm, vias 0 -> 1
Other:
- board text added: "SCL"
- board text added: "SDA"
- board text removed: "NRST"
