File: eagle/4ButtonSwitch.Rev2.1.brd (EAGLE design)
At the start: 69.8 x 69.8 mm, 46 parts

Commit message: Rev 2.1
Parts:
- added RS: 560E, resistor:R0402
Connections:
- new net N$1: RS.2, SENSORMCU.9
- net SHIELD: now also RS.1; no longer SENSORMCU.9
Routing:
- net GND: track 110.7 -> 193.8 mm, vias 24 -> 20
- net SHIELD: track 0.00 -> 18.1 mm, vias 0 -> 2
- net N$1: track 0.00 -> 9.63 mm, vias 0 -> 2
- net SHIELD_OR_GND: track 1.43 -> 2.77 mm
- added copper zone on layer 1, net GND
- added copper zone on layer 2, net SHIELD_OR_GND
- removed copper zone on layer 2, net GND
- removed copper zone on layer 1, net SHIELD_OR_GND

Commit message: Rev 2.1
Routing:
- net I2C_SCL: vias 3 -> 2
Other:
- board text added: "SHIELD"
Changed lines of the file:
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@@
 <setting verticaltext="up"/>
 </settings>
-<grid distance="50" unitdist="mil" unit="mil" style="lines" multiple="1" display="yes" altdistance="5" altunitdist="mil" altunit="mil"/>
+<grid distance="50" unitdist="mil" unit="inch" style="lines" multiple="1" display="yes" altdistance="5" altunitdist="mil" altunit="inch"/>
 <layers>
 <layer number="1" name="Top" color="4" fill="1" visible="yes" active="yes"/>
@@
 <text x="31.369" y="27.305" size="0.762" layer="26" rot="MR0">TXD</text>
 <text x="33.909" y="27.305" size="0.762" layer="26" rot="MR0">RXD</text>
+<text x="33.274" y="55.245" size="1.016" layer="25" rot="R90">SHIELD</text>
+<text x="37.592" y="55.245" size="1.016" layer="25" rot="R90">GND</text>
 </plain>
 <attributes>
@@
 <wire x1="22.61" y1="37.052" x2="22.61" y2="37.72431875" width="0.1524" layer="1"/>
 <wire x1="22.61" y1="37.72431875" x2="22.356659375" y2="37.977659375" width="0.1524" layer="1"/>
-<via x="22.356659375" y="37.977659375" extent="1-16" drill="0.2"/>
 <wire x1="30.48" y1="40.64" x2="29.21" y2="39.37" width="0.1524" layer="1"/>
 <wire x1="26.162" y1="40.005" x2="22.987" y2="40.005" width="0.1524" layer="1"/>

Commit message: updates
Parts:
- renumbered SIEMENS-BCU to SAM12235-ND
Connections:
- net HOST_INT: now also MCU.8; no longer MCU.11
- net PRG: now also MCU.27; no longer MCU.28
Routing:
- net HOST_INT: track 20.5 -> 21.2 mm
Changed lines of the file:
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@@
 </autorouter>
 <elements>
-<element name="SIEMENS-BCU" library="pinhead" package="2X05SMD" value="SIEMENS BCU" x="31.115" y="17.526" smashed="yes">
-<attribute name="NAME" x="30.0228" y="6.4008" size="1.016" layer="25" ratio="10"/>
+<element name="SAM12235-ND" library="pinhead" package="2X05SMD" value="SIEMENS BCU" x="31.115" y="17.526" smashed="yes">
 <attribute name="VALUE" x="28.575" y="11.811" size="1.27" layer="27"/>
 </element>
@@
 </element>
 <element name="RL1" library="resistor" library_urn="urn:adsk.eagle:library:348" package="R0402" package3d_urn="urn:adsk.eagle:package:26058/1" value="330E" x="52.07" y="46.99" smashed="yes" rot="R90">
-<attribute name="NAME" x="53.848" y="45.974" size="1.016" layer="25" rot="R90"/>
+<attribute name="NAME" x="51.308" y="45.72" size="1.016" layer="25" rot="R90"/>
 <attribute name="VALUE" x="53.975" y="46.355" size="1.27" layer="27" rot="R90"/>
 </element>
@@
 </element>
 <element name="RL3" library="resistor" library_urn="urn:adsk.eagle:library:348" package="R0402" package3d_urn="urn:adsk.eagle:package:26058/1" value="330E" x="52.07" y="22.86" smashed="yes" rot="R270">
-<attribute name="NAME" x="52.832" y="23.876" size="1.016" layer="25" rot="R270"/>
+<attribute name="NAME" x="50.292" y="24.13" size="1.016" layer="25" rot="R270"/>
 <attribute name="VALUE" x="50.165" y="23.495" size="1.27" layer="27" rot="R270"/>
 </element>
@@
 <signals>
 <signal name="+5V">
-<contactref element="SIEMENS-BCU" pad="1"/>
+<contactref element="SAM12235-ND" pad="1"/>
 <contactref element="3V3_REGULATOR" pad="2"/>
 <contactref element="C1" pad="2"/>
@@
 </signal>
 <signal name="GND">
-<contactref element="SIEMENS-BCU" pad="9"/>
+<contactref element="SAM12235-ND" pad="9"/>
 <contactref element="C1" pad="1"/>
 <contactref element="C2" pad="2"/>
@@
 <contactref element="PRG" pad="1"/>
 <contactref element="RT1" pad="2"/>
-<contactref element="MCU" pad="28"/>
-<wire x1="44.295" y1="29.187" x2="44.295" y2="27.587" width="0.3048" layer="1"/>
-<wire x1="44.295" y1="27.587" x2="45.212" y2="26.67" width="0.3048" layer="1"/>
-<wire x1="45.212" y1="26.67" x2="48.91" y2="26.67" width="0.3048" layer="1"/>
+<wire x1="48.91" y1="26.67" x2="45.212" y2="26.67" width="0.3048" layer="1"/>
 <wire x1="48.91" y1="26.67" x2="50.165" y2="27.925" width="0.3048" layer="1"/>
 <wire x1="51.2556" y1="26.98571875" x2="51.2556" y2="26.9764" width="0.1524" layer="1"/>
@@
 <wire x1="51.2556" y1="26.9764" x2="51.562" y2="26.67" width="0.1524" layer="1"/>
 <wire x1="51.562" y1="26.67" x2="59.69" y2="26.67" width="0.1524" layer="1"/>
+<contactref element="MCU" pad="27"/>
+<wire x1="43.795" y1="28.087" x2="43.795" y2="29.187" width="0.3048" layer="1"/>
+<wire x1="45.212" y1="26.67" x2="43.795" y2="28.087" width="0.3048" layer="1"/>
 </signal>
 <signal name="IC_SENS_PROX_1">
@@
 <signal name="HOST_INT">
 <contactref element="SENSORMCU" pad="23"/>
-<contactref element="MCU" pad="11"/>
-<wire x1="36.807" y1="33.675" x2="33.548" y2="33.675" width="0.1524" layer="1"/>
 <wire x1="25.4" y1="32.512" x2="24.892" y2="33.02" width="0.1524" layer="1"/>
 <via x="24.892" y="33.02" extent="1-16" drill="0.2"/>
-<wire x1="33.548" y1="33.675" x2="32.385" y2="32.512" width="0.1524" layer="1"/>
-<wire x1="32.385" y1="32.512" x2="25.4" y2="32.512" width="0.1524" layer="1"/>
+<wire x1="25.4" y1="32.512" x2="32.385" y2="32.512" width="0.1524" layer="1"/>
 <wire x1="22.11" y1="37.052" x2="22.098" y2="37.064" width="0.1524" layer="1"/>
 <wire x1="22.098" y1="37.064" x2="22.098" y2="37.592" width="0.1524" layer="1"/>
@@
 <wire x1="21.209" y1="37.338" x2="24.892" y2="33.655" width="0.1524" layer="15"/>
 <wire x1="24.892" y1="33.655" x2="24.892" y2="33.02" width="0.1524" layer="15"/>
+<contactref element="MCU" pad="8"/>
+<wire x1="35.81" y1="35.175" x2="36.807" y2="35.175" width="0.1524" layer="1"/>
+<wire x1="32.385" y1="32.512" x2="34.544" y2="34.671" width="0.1524" layer="1"/>
+<wire x1="34.544" y1="34.671" x2="35.306" y2="34.671" width="0.1524" layer="1"/>
+<wire x1="35.306" y1="34.671" x2="35.81" y2="35.175" width="0.1524" layer="1"/>
 </signal>
 <signal name="CMOD">
@@
 </signal>
 <signal name="USART1_RX">
-<contactref element="SIEMENS-BCU" pad="3"/>
+<contactref element="SAM12235-ND" pad="3"/>
 <contactref element="MCU" pad="25"/>
 <wire x1="32.385" y1="13.716" x2="32.639" y2="13.97" width="0.1524" layer="1"/>
@@
 </signal>
 <signal name="USART1_TX">
-<contactref element="SIEMENS-BCU" pad="7"/>
+<contactref element="SAM12235-ND" pad="7"/>
 <contactref element="MCU" pad="24"/>
 <wire x1="42.295" y1="29.187" x2="42.295" y2="28.071" width="0.1524" layer="1"/>
