File: eagle/4ButtonSwitch.Rev2.1.sch (EAGLE design)
At the start: 43 parts

Commit message: Rev 2.1
Connections:
- net GND: now also SENSORMCU.CS9/GPO1; no longer SENSORMCU.CS12/GP14
- net IC_SENS_3: now also SENSORMCU.CS12/GP14; no longer SENSORMCU.CS9/GPO1
Changed lines of the file:
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@@
 <pinref part="SENSORMCU" gate="G$1" pin="CS4"/>
 <wire x1="281.94" y1="50.8" x2="281.94" y2="63.5" width="0.1524" layer="91"/>
-<wire x1="281.94" y1="63.5" x2="289.56" y2="63.5" width="0.1524" layer="91"/>
-<label x="289.56" y="63.5" size="1.016" layer="95" xref="yes"/>
-</segment>
-<segment>
+<label x="281.94" y="63.5" size="1.016" layer="95" rot="R90" xref="yes"/>
+</segment>
+<segment>
+<pinref part="SENSORMCU" gate="G$1" pin="CS9/GPO1"/>
+<wire x1="297.18" y1="17.78" x2="302.26" y2="17.78" width="0.1524" layer="91"/>
+<pinref part="SENSORMCU" gate="G$1" pin="CS8/GPO0"/>
+<wire x1="302.26" y1="20.32" x2="297.18" y2="20.32" width="0.1524" layer="91"/>
+<pinref part="SENSORMCU" gate="G$1" pin="CS7"/>
+<wire x1="297.18" y1="22.86" x2="302.26" y2="22.86" width="0.1524" layer="91"/>
+<wire x1="302.26" y1="22.86" x2="302.26" y2="20.32" width="0.1524" layer="91"/>
+<junction x="302.26" y="20.32"/>
+<wire x1="302.26" y1="17.78" x2="302.26" y2="20.32" width="0.1524" layer="91"/>
+<pinref part="SENSORMCU" gate="G$1" pin="CS10/GPO2"/>
+<wire x1="297.18" y1="15.24" x2="302.26" y2="15.24" width="0.1524" layer="91"/>
+<wire x1="302.26" y1="12.7" x2="302.26" y2="15.24" width="0.1524" layer="91"/>
+<wire x1="302.26" y1="12.7" x2="302.26" y2="10.16" width="0.1524" layer="91"/>
+<junction x="302.26" y="12.7"/>
 <pinref part="SENSORMCU" gate="G$1" pin="CS11/GPO3"/>
 <wire x1="297.18" y1="12.7" x2="302.26" y2="12.7" width="0.1524" layer="91"/>
-<wire x1="302.26" y1="12.7" x2="302.26" y2="15.24" width="0.1524" layer="91"/>
-<pinref part="SENSORMCU" gate="G$1" pin="CS10/GPO2"/>
-<wire x1="297.18" y1="15.24" x2="302.26" y2="15.24" width="0.1524" layer="91"/>
-<wire x1="302.26" y1="12.7" x2="302.26" y2="10.16" width="0.1524" layer="91"/>
-<junction x="302.26" y="12.7"/>
 <label x="302.26" y="10.16" size="1.016" layer="95" xref="yes"/>
-</segment>
-<segment>
-<pinref part="SENSORMCU" gate="G$1" pin="CS12/GP14"/>
+<wire x1="302.26" y1="17.78" x2="302.26" y2="15.24" width="0.1524" layer="91"/>
+<junction x="302.26" y="17.78"/>
+<junction x="302.26" y="15.24"/>
+</segment>
+<segment>
 <wire x1="276.86" y1="-17.78" x2="279.4" y2="-17.78" width="0.1524" layer="91"/>
-<wire x1="279.4" y1="-17.78" x2="281.94" y2="-17.78" width="0.1524" layer="91"/>
-<wire x1="281.94" y1="-17.78" x2="281.94" y2="-12.7" width="0.1524" layer="91"/>
 <pinref part="SENSORMCU" gate="G$1" pin="CS13/GPO5"/>
 <wire x1="279.4" y1="-12.7" x2="279.4" y2="-17.78" width="0.1524" layer="91"/>
-<junction x="279.4" y="-17.78"/>
 <pinref part="SENSORMCU" gate="G$1" pin="CS14/GPO6"/>
 <wire x1="276.86" y1="-12.7" x2="276.86" y2="-17.78" width="0.1524" layer="91"/>
-<wire x1="281.94" y1="-17.78" x2="287.02" y2="-17.78" width="0.1524" layer="91"/>
-<junction x="281.94" y="-17.78"/>
-<label x="287.02" y="-17.78" size="1.016" layer="95" xref="yes"/>
+<wire x1="276.86" y1="-17.78" x2="276.86" y2="-22.86" width="0.1524" layer="91"/>
+<junction x="276.86" y="-17.78"/>
+<label x="276.86" y="-22.86" size="1.27" layer="95" rot="R270" xref="yes"/>
 </segment>
 <segment>
@@
 <wire x1="269.24" y1="50.8" x2="269.24" y2="55.88" width="0.1524" layer="91"/>
 <label x="269.24" y="55.88" size="1.27" layer="95" rot="R90" xref="yes"/>
-</segment>
-<segment>
-<pinref part="SENSORMCU" gate="G$1" pin="CS8/GPO0"/>
-<wire x1="302.26" y1="20.32" x2="297.18" y2="20.32" width="0.1524" layer="91"/>
-<pinref part="SENSORMCU" gate="G$1" pin="CS7"/>
-<wire x1="297.18" y1="22.86" x2="302.26" y2="22.86" width="0.1524" layer="91"/>
-<wire x1="302.26" y1="22.86" x2="302.26" y2="20.32" width="0.1524" layer="91"/>
-<wire x1="302.26" y1="20.32" x2="304.8" y2="20.32" width="0.1524" layer="91"/>
-<junction x="302.26" y="20.32"/>
-<label x="304.8" y="20.32" size="1.27" layer="95" xref="yes"/>
 </segment>
 <segment>
@@
 </segment>
 <segment>
-<pinref part="SENSORMCU" gate="G$1" pin="CS9/GPO1"/>
-<wire x1="297.18" y1="17.78" x2="302.26" y2="17.78" width="0.1524" layer="91"/>
-<label x="302.26" y="17.78" size="1.27" layer="95" xref="yes"/>
-</segment>
-</net>
+<pinref part="SENSORMCU" gate="G$1" pin="CS12/GP14"/>
+<wire x1="281.94" y1="-12.7" x2="281.94" y2="-22.86" width="0.1524" layer="91"/>
+<label x="281.94" y="-22.86" size="1.27" layer="95" rot="R270" xref="yes"/>
+</segment>
+</net>

Commit message: Rev 2.1
Parts:
- added S1: PCM12SMTR, PCM12SMTR:PCM12SMTR
Connections:
- new net SHIELD_OR_GND: S1.2
- net GND: now also S1.1
- net PRG: now also MCU.PB2; no longer MCU.PA5
- net SHIELD: now also S1.3
Changed lines of the file:
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@@
 <part name="LED4" library="led" library_urn="urn:adsk.eagle:library:259" deviceset="*P4" device="-BOTTOM" package3d_urn="urn:adsk.eagle:package:15878/1" technology="LW"/>
 <part name="C11" library="rcl" library_urn="urn:adsk.eagle:library:334" deviceset="C-EU" device="C0402" package3d_urn="urn:adsk.eagle:package:23626/1" value="4.7uf"/>
+<part name="S1" library="PCM12SMTR" deviceset="PCM12SMTR" device=""/>
 </parts>
 <sheets>
@@
 <instance part="LED4" gate="G$1" x="154.94" y="17.78" rot="R270"/>
 <instance part="C11" gate="G$1" x="109.22" y="17.78"/>
+<instance part="S1" gate="G$1" x="345.44" y="-35.56"/>
 </instances>
 <busses>
@@
 <label x="246.38" y="20.32" size="1.27" layer="95" rot="R180" xref="yes"/>
 </segment>
+<segment>
+<pinref part="S1" gate="G$1" pin="1"/>
+<wire x1="345.44" y1="-35.56" x2="335.28" y2="-35.56" width="0.1524" layer="91"/>
+<label x="335.28" y="-35.56" size="1.27" layer="95" rot="R180" xref="yes"/>
+</segment>
 </net>
 <net name="+3V3" class="0">
@@
 </segment>
 <segment>
-<pinref part="MCU" gate="G$1" pin="PA5"/>
-<wire x1="165.1" y1="-129.54" x2="165.1" y2="-137.16" width="0.1524" layer="91"/>
-<label x="165.1" y="-137.16" size="1.27" layer="95" rot="R270" xref="yes"/>
+<pinref part="MCU" gate="G$1" pin="PB2"/>
+<wire x1="182.88" y1="-129.54" x2="182.88" y2="-137.16" width="0.1524" layer="91"/>
+<label x="182.88" y="-137.16" size="1.27" layer="95" rot="R270" xref="yes"/>
 </segment>
 </net>
@@
 <label x="274.32" y="-22.86" size="1.016" layer="95" rot="R270" xref="yes"/>
 </segment>
+<segment>
+<pinref part="S1" gate="G$1" pin="3"/>
+<wire x1="365.76" y1="-35.56" x2="375.92" y2="-35.56" width="0.1524" layer="91"/>
+<label x="375.92" y="-35.56" size="1.27" layer="95" xref="yes"/>
+</segment>
 </net>
 <net name="USART2_TX" class="0">
@@
 </segment>
 </net>
+<net name="SHIELD_OR_GND" class="0">
+<segment>
+<pinref part="S1" gate="G$1" pin="2"/>
+<wire x1="345.44" y1="-38.1" x2="335.28" y2="-38.1" width="0.1524" layer="91"/>
+<label x="335.28" y="-38.1" size="1.27" layer="95" rot="R180" xref="yes"/>
+</segment>
+</net>

Commit message: Rev 2.1
Parts:
- renumbered NRST1 to NRST, PRG1 to PRG
Other:
- moved on the sheet: GND_NRST, GND_PRG
Changed lines of the file:
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@@
 <part name="CLO1" library="rcl" library_urn="urn:adsk.eagle:library:334" deviceset="C-EU" device="C0402" package3d_urn="urn:adsk.eagle:package:23626/1" value="7pF"/>
 <part name="CLO2" library="rcl" library_urn="urn:adsk.eagle:library:334" deviceset="C-EU" device="C0402" package3d_urn="urn:adsk.eagle:package:23626/1" value="7pf"/>
-<part name="NRST1" library="wirepad" library_urn="urn:adsk.eagle:library:412" deviceset="SMD5" device="" package3d_urn="urn:adsk.eagle:package:30841/1" value="0"/>
-<part name="GND_NRST" library="wirepad" library_urn="urn:adsk.eagle:library:412" deviceset="SMD5" device="" package3d_urn="urn:adsk.eagle:package:30841/1" value="0"/>
+<part name="NRST" library="wirepad" library_urn="urn:adsk.eagle:library:412" deviceset="SMD5" device="" package3d_urn="urn:adsk.eagle:package:30841/1" value="0"/>
+<part name="GND_PRG" library="wirepad" library_urn="urn:adsk.eagle:library:412" deviceset="SMD5" device="" package3d_urn="urn:adsk.eagle:package:30841/1" value="0"/>
 <part name="RL2" library="resistor" library_urn="urn:adsk.eagle:library:348" deviceset="R-EU_" device="R0402" package3d_urn="urn:adsk.eagle:package:26058/1" value="330E"/>
 <part name="RL1" library="resistor" library_urn="urn:adsk.eagle:library:348" deviceset="R-EU_" device="R0402" package3d_urn="urn:adsk.eagle:package:26058/1" value="330E"/>
@@
 <part name="RP1" library="resistor" library_urn="urn:adsk.eagle:library:348" deviceset="R-EU_" device="R0402" package3d_urn="urn:adsk.eagle:package:26058/1" value="560E"/>
 <part name="RP2" library="resistor" library_urn="urn:adsk.eagle:library:348" deviceset="R-EU_" device="R0402" package3d_urn="urn:adsk.eagle:package:26058/1" value="560E"/>
-<part name="PRG1" library="wirepad" library_urn="urn:adsk.eagle:library:412" deviceset="SMD5" device="" package3d_urn="urn:adsk.eagle:package:30841/1" value="0"/>
-<part name="GND_PRG" library="wirepad" library_urn="urn:adsk.eagle:library:412" deviceset="SMD5" device="" package3d_urn="urn:adsk.eagle:package:30841/1" value="0"/>
+<part name="PRG" library="wirepad" library_urn="urn:adsk.eagle:library:412" deviceset="SMD5" device="" package3d_urn="urn:adsk.eagle:package:30841/1" value="0"/>
+<part name="GND_NRST" library="wirepad" library_urn="urn:adsk.eagle:library:412" deviceset="SMD5" device="" package3d_urn="urn:adsk.eagle:package:30841/1" value="0"/>
 <part name="RT1" library="resistor" library_urn="urn:adsk.eagle:library:348" deviceset="R-EU_" device="R0402" package3d_urn="urn:adsk.eagle:package:26058/1" value="100K"/>
 <part name="TEMP" library="HTS221TR" deviceset="HTS221TR" device=""/>
@@
 <instance part="CLO1" gate="G$1" x="50.8" y="-15.24" rot="R90"/>
 <instance part="CLO2" gate="G$1" x="50.8" y="-35.56" rot="R90"/>
-<instance part="NRST1" gate="1" x="86.36" y="-92.964" rot="MR90"/>
-<instance part="GND_NRST" gate="1" x="86.36" y="-97.536" rot="MR270"/>
+<instance part="NRST" gate="1" x="86.36" y="-92.964" rot="MR90"/>
+<instance part="GND_PRG" gate="1" x="86.36" y="-97.536" rot="MR270"/>
 <instance part="RL2" gate="G$1" x="177.8" y="43.18" rot="R180"/>
 <instance part="RL1" gate="G$1" x="177.8" y="55.88" rot="R180"/>
@@
 <instance part="RP1" gate="G$1" x="345.44" y="17.78" rot="R90"/>
 <instance part="RP2" gate="G$1" x="337.82" y="17.78" rot="R90"/>
-<instance part="PRG1" gate="1" x="254" y="-106.68" rot="MR90"/>
-<instance part="GND_PRG" gate="1" x="254" y="-111.76" rot="MR270"/>
+<instance part="PRG" gate="1" x="254" y="-106.68" rot="MR90"/>
+<instance part="GND_NRST" gate="1" x="254" y="-111.76" rot="MR270"/>
 <instance part="RT1" gate="G$1" x="269.24" y="-101.6" rot="R180"/>
 <instance part="TEMP" gate="G$1" x="261.62" y="-66.04"/>
@@
 </segment>
 <segment>
-<pinref part="GND_PRG" gate="1" pin="P"/>
+<pinref part="GND_NRST" gate="1" pin="P"/>
 <wire x1="254" y1="-114.3" x2="254" y2="-119.38" width="0.1524" layer="91"/>
 <label x="254" y="-119.38" size="1.016" layer="95" rot="R270" xref="yes"/>
@@
 <wire x1="86.36" y1="-101.6" x2="81.28" y2="-101.6" width="0.1524" layer="91"/>
 <wire x1="93.98" y1="-99.06" x2="93.98" y2="-101.6" width="0.1524" layer="91"/>
-<pinref part="GND_NRST" gate="1" pin="P"/>
+<pinref part="GND_PRG" gate="1" pin="P"/>
 <wire x1="86.36" y1="-100.076" x2="86.36" y2="-101.6" width="0.1524" layer="91"/>
 <junction x="86.36" y="-101.6"/>
@@
 <junction x="93.98" y="-88.9"/>
 <pinref part="MCU" gate="G$1" pin="NRST"/>
-<pinref part="NRST1" gate="1" pin="P"/>
+<pinref part="NRST" gate="1" pin="P"/>
 <wire x1="86.36" y1="-90.424" x2="86.36" y2="-88.9" width="0.1524" layer="91"/>
 <junction x="86.36" y="-88.9"/>
@@
 <net name="PRG" class="0">
 <segment>
-<pinref part="PRG1" gate="1" pin="P"/>
+<pinref part="PRG" gate="1" pin="P"/>
 <wire x1="254" y1="-104.14" x2="254" y2="-101.6" width="0.1524" layer="91"/>
 <label x="254" y="-96.52" size="1.016" layer="95" rot="R90" xref="yes"/>

Commit message: Rev 2.1
Parts:
- added RS: 560E, resistor:R-EU_R0402
Connections:
- new net N$1: RS.2, SENSORMCU.CS15/SH/!HI
- net SHIELD: now also RS.1; no longer SENSORMCU.CS15/SH/!HI
Changed lines of the file:
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@@
 <part name="C11" library="rcl" library_urn="urn:adsk.eagle:library:334" deviceset="C-EU" device="C0402" package3d_urn="urn:adsk.eagle:package:23626/1" value="4.7uf"/>
 <part name="S1" library="PCM12SMTR" deviceset="PCM12SMTR" device=""/>
+<part name="RS" library="resistor" library_urn="urn:adsk.eagle:library:348" deviceset="R-EU_" device="R0402" package3d_urn="urn:adsk.eagle:package:26058/1" value="560E"/>
 </parts>
 <sheets>
@@
 <instance part="C11" gate="G$1" x="109.22" y="17.78"/>
 <instance part="S1" gate="G$1" x="345.44" y="-35.56"/>
+<instance part="RS" gate="G$1" x="274.32" y="-30.48" rot="R90"/>
 </instances>
 <busses>
@@
 <net name="SHIELD" class="0">
 <segment>
-<pinref part="SENSORMCU" gate="G$1" pin="CS15/SH/!HI"/>
-<wire x1="274.32" y1="-12.7" x2="274.32" y2="-22.86" width="0.1524" layer="91"/>
-<label x="274.32" y="-22.86" size="1.016" layer="95" rot="R270" xref="yes"/>
-</segment>
-<segment>
 <pinref part="S1" gate="G$1" pin="3"/>
 <wire x1="365.76" y1="-35.56" x2="375.92" y2="-35.56" width="0.1524" layer="91"/>
 <label x="375.92" y="-35.56" size="1.27" layer="95" xref="yes"/>
 </segment>
+<segment>
+<pinref part="RS" gate="G$1" pin="1"/>
+<wire x1="274.32" y1="-35.56" x2="274.32" y2="-38.1" width="0.1524" layer="91"/>
+<label x="274.32" y="-38.1" size="1.27" layer="95" rot="R270" xref="yes"/>
+</segment>
 </net>
 <net name="USART2_TX" class="0">
@@
 </segment>
 </net>
+<net name="N$1" class="0">
+<segment>
+<pinref part="SENSORMCU" gate="G$1" pin="CS15/SH/!HI"/>
+<wire x1="274.32" y1="-12.7" x2="274.32" y2="-25.4" width="0.1524" layer="91"/>
+<pinref part="RS" gate="G$1" pin="2"/>
+</segment>
+</net>

Commit message: updates
Parts:
- renumbered SIEMENS-BCU to SAM12235-ND
Connections:
- net HOST_INT: now also MCU.PC0; no longer MCU.PC3
- net PRG: now also MCU.PB1; no longer MCU.PB2
Other:
- note added: "SAM12235-ND"
- note removed: "WM17451-ND"
Changed lines of the file:
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@@
 </classes>
 <parts>
-<part name="SIEMENS-BCU" library="pinhead" deviceset="PINHD-2X5" device="_2.54-SMD" value="SIEMENS BCU"/>
+<part name="SAM12235-ND" library="pinhead" deviceset="PINHD-2X5" device="_2.54-SMD" value="SIEMENS BCU"/>
 <part name="3V3_REGULATOR" library="MCP1703T-3302E_MB" deviceset="MCP1703T-3302E_MB" device=""/>
 <part name="+3V1" library="supply1" library_urn="urn:adsk.eagle:library:371" deviceset="+3V3" device=""/>
@@
 <text x="243.84" y="43.18" size="1.778" layer="91">I2C Adr.: 0x37</text>
 <text x="243.84" y="43.18" size="1.778" layer="91">I2C Adr.: 0x37</text>
-<text x="45.72" y="63.5" size="1.778" layer="91">WM17451-ND
-</text>
+<text x="44.704" y="67.564" size="1.778" layer="91">SAM12235-ND</text>
 <text x="162.56" y="-22.86" size="1.778" layer="91">TODO:
 * I2C Pins auf VIAS
@@
 </plain>
 <instances>
-<instance part="SIEMENS-BCU" gate="A" x="53.34" y="55.88" rot="R90"/>
+<instance part="SAM12235-ND" gate="A" x="53.34" y="55.88" rot="R90"/>
 <instance part="3V3_REGULATOR" gate="G$1" x="40.64" y="20.32"/>
 <instance part="+3V1" gate="G$1" x="22.86" y="63.5"/>
@@
 <net name="+5V" class="0">
 <segment>
-<pinref part="SIEMENS-BCU" gate="A" pin="1"/>
+<pinref part="SAM12235-ND" gate="A" pin="1"/>
 <wire x1="48.26" y1="53.34" x2="48.26" y2="43.18" width="0.1524" layer="91"/>
 <label x="48.26" y="43.18" size="1.016" layer="95" rot="R270" xref="yes"/>
@@
 <net name="GND" class="0">
 <segment>
-<pinref part="SIEMENS-BCU" gate="A" pin="9"/>
+<pinref part="SAM12235-ND" gate="A" pin="9"/>
 <wire x1="58.42" y1="53.34" x2="58.42" y2="43.18" width="0.1524" layer="91"/>
 <label x="58.42" y="43.18" size="1.016" layer="95" rot="R270" xref="yes"/>
@@
 </segment>
 <segment>
-<pinref part="MCU" gate="G$1" pin="PB2"/>
-<wire x1="182.88" y1="-129.54" x2="182.88" y2="-137.16" width="0.1524" layer="91"/>
-<label x="182.88" y="-137.16" size="1.27" layer="95" rot="R270" xref="yes"/>
+<pinref part="MCU" gate="G$1" pin="PB1"/>
+<wire x1="180.34" y1="-129.54" x2="180.34" y2="-137.16" width="0.1524" layer="91"/>
+<label x="180.34" y="-137.16" size="1.27" layer="95" rot="R270" xref="yes"/>
 </segment>
 </net>
@@
 </segment>
 <segment>
-<pinref part="MCU" gate="G$1" pin="PC3"/>
-<label x="137.16" y="-99.06" size="1.27" layer="95" rot="R180" xref="yes"/>
-<wire x1="147.32" y1="-99.06" x2="137.16" y2="-99.06" width="0.1524" layer="91"/>
+<pinref part="MCU" gate="G$1" pin="PC0"/>
+<wire x1="147.32" y1="-91.44" x2="137.16" y2="-91.44" width="0.1524" layer="91"/>
+<label x="137.16" y="-91.44" size="1.27" layer="95" rot="R180" xref="yes"/>
 </segment>
 </net>
@@
 <net name="USART1_RX" class="0">
 <segment>
-<pinref part="SIEMENS-BCU" gate="A" pin="3"/>
+<pinref part="SAM12235-ND" gate="A" pin="3"/>
 <wire x1="50.8" y1="53.34" x2="50.8" y2="43.18" width="0.1524" layer="91"/>
 <label x="50.8" y="43.18" size="1.016" layer="95" rot="R270" xref="yes"/>
@@
 <net name="USART1_TX" class="0">
 <segment>
-<pinref part="SIEMENS-BCU" gate="A" pin="7"/>
+<pinref part="SAM12235-ND" gate="A" pin="7"/>
 <wire x1="55.88" y1="53.34" x2="55.88" y2="43.18" width="0.1524" layer="91"/>
 <label x="55.88" y="43.18" size="1.016" layer="95" rot="R270" xref="yes"/>
