File: eagle/4ButtonSwitch.Rev2.2.brd (EAGLE design)
At the start: 69.8 x 69.8 mm, 46 parts

Commit message: updates
Parts:
- removed 3V3_REGULATOR: MCP1703T-3302E_MB, MCP1703T-3302E_MB:SOT-89(MB)
- added 3V3_VR: TPS70933DBVT, TPS70933DBVT:SOT95P280X145-5N
- C2: value 1uF -> 2.2uF
Connections:
- net +3V3: now also 3V3_VR.5; no longer 3V3_REGULATOR.3
- net +5V: now also 3V3_VR.1; no longer 3V3_REGULATOR.2, 3V3_REGULATOR.4
- net GND: now also 3V3_VR.2; no longer 3V3_REGULATOR.1
Routing:
- net GND: track 193.3 -> 209.0 mm, vias 19 -> 20
- net +5V: track 19.8 -> 25.2 mm, vias 0 -> 1
Other:
- board text added: "5V-30V"
