File: eagle/4ButtonSwitch.Rev2.2.sch (EAGLE design)
At the start: 44 parts

Commit message: updates
Parts:
- removed 3V3_REGULATOR: MCP1703T-3302E_MB, MCP1703T-3302E_MB:MCP1703T-3302E_MB
- added 3V3_VR: TPS70933DBVT, TPS70933DBVT:TPS70933DBVT
- C2: value 1uF -> 2.2uF
Connections:
- net +3V3: now also 3V3_VR.OUT; no longer 3V3_REGULATOR.VOUT
- net +5V: now also 3V3_VR.IN; no longer 3V3_REGULATOR.VIN1, 3V3_REGULATOR.VIN2
- net GND: now also 3V3_VR.GND; no longer 3V3_REGULATOR.GND
Other:
- moved on the sheet: C1, C11, C2, C6
Changed lines of the file:
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@@
 <parts>
 <part name="SAM12235-ND" library="pinhead" deviceset="PINHD-2X5" device="_2.54-SMD" value="SIEMENS BCU"/>
-<part name="3V3_REGULATOR" library="MCP1703T-3302E_MB" deviceset="MCP1703T-3302E_MB" device=""/>
 <part name="+3V1" library="supply1" library_urn="urn:adsk.eagle:library:371" deviceset="+3V3" device=""/>
 <part name="P+1" library="supply1" library_urn="urn:adsk.eagle:library:371" deviceset="+5V" device=""/>
 <part name="GND1" library="supply1" library_urn="urn:adsk.eagle:library:371" deviceset="GND" device=""/>
 <part name="C1" library="rcl" library_urn="urn:adsk.eagle:library:334" deviceset="C-EU" device="C0402" package3d_urn="urn:adsk.eagle:package:23626/1" value="1uF"/>
-<part name="C2" library="rcl" library_urn="urn:adsk.eagle:library:334" deviceset="C-EU" device="C0402" package3d_urn="urn:adsk.eagle:package:23626/1" value="1uF"/>
+<part name="C2" library="rcl" library_urn="urn:adsk.eagle:library:334" deviceset="C-EU" device="C0402" package3d_urn="urn:adsk.eagle:package:23626/1" value="2.2uF"/>
 <part name="OSC32" library="ABS07-32.768KHZ-7-T" deviceset="ABS07-32.768KHZ-7-T" device=""/>
 <part name="CLO1" library="rcl" library_urn="urn:adsk.eagle:library:334" deviceset="C-EU" device="C0402" package3d_urn="urn:adsk.eagle:package:23626/1" value="7pF"/>
@@
 <part name="C11" library="rcl" library_urn="urn:adsk.eagle:library:334" deviceset="C-EU" device="C0402" package3d_urn="urn:adsk.eagle:package:23626/1" value="4.7uf"/>
 <part name="RS" library="resistor" library_urn="urn:adsk.eagle:library:348" deviceset="R-EU_" device="R0402" package3d_urn="urn:adsk.eagle:package:26058/1" value="560E"/>
+<part name="3V3_VR" library="TPS70933DBVT" deviceset="TPS70933DBVT" device=""/>
 </parts>
 <sheets>
@@
 <instances>
 <instance part="SAM12235-ND" gate="A" x="53.34" y="55.88" rot="R90"/>
-<instance part="3V3_REGULATOR" gate="G$1" x="40.64" y="20.32"/>
 <instance part="+3V1" gate="G$1" x="22.86" y="63.5"/>
 <instance part="P+1" gate="1" x="30.48" y="63.5"/>
 <instance part="GND1" gate="1" x="12.7" y="48.26"/>
-<instance part="C1" gate="G$1" x="35.56" y="25.4"/>
-<instance part="C2" gate="G$1" x="73.66" y="17.78"/>
+<instance part="C1" gate="G$1" x="35.56" y="12.7" rot="R180"/>
+<instance part="C2" gate="G$1" x="73.66" y="15.24"/>
 <instance part="OSC32" gate="G$1" x="66.04" y="-15.24" rot="R270"/>
 <instance part="CLO1" gate="G$1" x="50.8" y="-15.24" rot="R90"/>
@@
 <instance part="RI2C1" gate="G$1" x="27.94" y="-96.52" rot="R90"/>
 <instance part="RI2C2" gate="G$1" x="38.1" y="-96.52" rot="R90"/>
-<instance part="C6" gate="G$1" x="81.28" y="17.78"/>
+<instance part="C6" gate="G$1" x="81.28" y="15.24"/>
 <instance part="MCU" gate="G$1" x="147.32" y="-73.66"/>
 <instance part="C7" gate="G$1" x="93.98" y="-93.98"/>
@@
 <instance part="LED3" gate="G$1" x="154.94" y="30.48" rot="R270"/>
 <instance part="LED4" gate="G$1" x="154.94" y="17.78" rot="R270"/>
-<instance part="C11" gate="G$1" x="109.22" y="17.78"/>
+<instance part="C11" gate="G$1" x="109.22" y="15.24"/>
 <instance part="RS" gate="G$1" x="274.32" y="-30.48" rot="R90"/>
+<instance part="3V3_VR" gate="G$1" x="43.18" y="20.32"/>
 </instances>
 <busses>
@@
 </segment>
 <segment>
-<pinref part="3V3_REGULATOR" gate="G$1" pin="VIN1"/>
-<wire x1="40.64" y1="17.78" x2="35.56" y2="17.78" width="0.1524" layer="91"/>
-<label x="27.94" y="17.78" size="1.016" layer="95" rot="R180" xref="yes"/>
+<label x="27.94" y="20.32" size="1.016" layer="95" rot="R180" xref="yes"/>
 <pinref part="C1" gate="G$1" pin="2"/>
-<wire x1="35.56" y1="17.78" x2="27.94" y2="17.78" width="0.1524" layer="91"/>
-<wire x1="35.56" y1="20.32" x2="35.56" y2="17.78" width="0.1524" layer="91"/>
-<junction x="35.56" y="17.78"/>
-<pinref part="3V3_REGULATOR" gate="G$1" pin="VIN2"/>
-<wire x1="68.58" y1="17.78" x2="68.58" y2="12.7" width="0.1524" layer="91"/>
-<wire x1="68.58" y1="12.7" x2="35.56" y2="12.7" width="0.1524" layer="91"/>
-<wire x1="35.56" y1="12.7" x2="35.56" y2="17.78" width="0.1524" layer="91"/>
+<wire x1="35.56" y1="20.32" x2="27.94" y2="20.32" width="0.1524" layer="91"/>
+<wire x1="35.56" y1="17.78" x2="35.56" y2="20.32" width="0.1524" layer="91"/>
+<pinref part="3V3_VR" gate="G$1" pin="IN"/>
+<wire x1="35.56" y1="20.32" x2="43.18" y2="20.32" width="0.1524" layer="91"/>
+<junction x="35.56" y="20.32"/>
 </segment>
 </net>
@@
 <segment>
 <pinref part="C1" gate="G$1" pin="1"/>
-<wire x1="35.56" y1="27.94" x2="35.56" y2="30.48" width="0.1524" layer="91"/>
-<label x="35.56" y="30.48" size="1.016" layer="95" rot="R90" xref="yes"/>
-<pinref part="3V3_REGULATOR" gate="G$1" pin="GND"/>
-<wire x1="40.64" y1="20.32" x2="40.64" y2="27.94" width="0.1524" layer="91"/>
-<wire x1="40.64" y1="27.94" x2="35.56" y2="27.94" width="0.1524" layer="91"/>
-<junction x="35.56" y="27.94"/>
+<wire x1="35.56" y1="10.16" x2="35.56" y2="7.62" width="0.1524" layer="91"/>
+<label x="35.56" y="5.08" size="1.016" layer="95" rot="R270" xref="yes"/>
+<wire x1="35.56" y1="7.62" x2="35.56" y2="5.08" width="0.1524" layer="91"/>
+<wire x1="35.56" y1="7.62" x2="40.64" y2="7.62" width="0.1524" layer="91"/>
+<wire x1="40.64" y1="7.62" x2="40.64" y2="17.78" width="0.1524" layer="91"/>
+<junction x="35.56" y="7.62"/>
+<pinref part="3V3_VR" gate="G$1" pin="GND"/>
+<wire x1="40.64" y1="17.78" x2="43.18" y2="17.78" width="0.1524" layer="91"/>
 </segment>
 <segment>
 <pinref part="C2" gate="G$1" pin="2"/>
-<wire x1="73.66" y1="12.7" x2="73.66" y2="10.16" width="0.1524" layer="91"/>
-<label x="73.66" y="10.16" size="1.016" layer="95" rot="R270" xref="yes"/>
+<wire x1="73.66" y1="10.16" x2="73.66" y2="7.62" width="0.1524" layer="91"/>
+<label x="73.66" y="7.62" size="1.016" layer="95" rot="R270" xref="yes"/>
 <pinref part="C6" gate="G$1" pin="2"/>
-<wire x1="81.28" y1="12.7" x2="73.66" y2="12.7" width="0.1524" layer="91"/>
-<junction x="73.66" y="12.7"/>
+<wire x1="81.28" y1="10.16" x2="73.66" y2="10.16" width="0.1524" layer="91"/>
+<junction x="73.66" y="10.16"/>
 <pinref part="C11" gate="G$1" pin="2"/>
-<wire x1="81.28" y1="12.7" x2="109.22" y2="12.7" width="0.1524" layer="91"/>
-<junction x="81.28" y="12.7"/>
+<wire x1="81.28" y1="10.16" x2="109.22" y2="10.16" width="0.1524" layer="91"/>
+<junction x="81.28" y="10.16"/>
 </segment>
 <segment>
@@
 </segment>
 <segment>
-<pinref part="3V3_REGULATOR" gate="G$1" pin="VOUT"/>
-<wire x1="68.58" y1="20.32" x2="73.66" y2="20.32" width="0.1524" layer="91"/>
-<label x="114.3" y="20.32" size="1.016" layer="95" xref="yes"/>
+<label x="114.3" y="17.78" size="1.016" layer="95" xref="yes"/>
 <pinref part="C2" gate="G$1" pin="1"/>
-<junction x="73.66" y="20.32"/>
-<wire x1="73.66" y1="20.32" x2="81.28" y2="20.32" width="0.1524" layer="91"/>
+<wire x1="73.66" y1="17.78" x2="81.28" y2="17.78" width="0.1524" layer="91"/>
 <pinref part="C6" gate="G$1" pin="1"/>
-<junction x="81.28" y="20.32"/>
-<wire x1="81.28" y1="20.32" x2="109.22" y2="20.32" width="0.1524" layer="91"/>
+<junction x="81.28" y="17.78"/>
+<wire x1="81.28" y1="17.78" x2="109.22" y2="17.78" width="0.1524" layer="91"/>
 <pinref part="C11" gate="G$1" pin="1"/>
-<wire x1="109.22" y1="20.32" x2="114.3" y2="20.32" width="0.1524" layer="91"/>
-<junction x="109.22" y="20.32"/>
-</segment>
-<segment>
+<wire x1="109.22" y1="17.78" x2="114.3" y2="17.78" width="0.1524" layer="91"/>
+<junction x="109.22" y="17.78"/>
+<pinref part="3V3_VR" gate="G$1" pin="OUT"/>
+<wire x1="68.58" y1="17.78" x2="73.66" y2="17.78" width="0.1524" layer="91"/>
+<junction x="73.66" y="17.78"/>
+</segment>
+<segment>
