File: eagle/4ButtonSwitch.Rev3.0.sch (EAGLE design)
At the start: 35 parts, among them U1 ADP2108AUJZ-3.3-R7

Commit message: updates
Parts:
- added CLO1, CLO2: 15pF, rcl:C-EUC1206
- added OSC32: ABS07-32.768KHZ-7-T, ABS07-32.768KHZ-7-T:ABS07-32.768KHZ-7-T
- added U$3, U$4: SAMTEC-TSM-104-01-X-SHJ, SAMTEC-TSM-104-01-X-SH:SAMTEC-TSM-104-01-X-SHJ
Connections:
- new net N$3: PAD_PRG.P
- net GND: now also CLO1.1, CLO2.1, GND_NRST.P, GND_PRG.P
- net RESET: now also PAD_NRST.P
- net X32IN: now also CLO1.2, OSC32.1
- net X32OUT: now also CLO2.2, OSC32.2
Changed lines of the file:
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@@
 <part name="CB2" library="rcl" library_urn="urn:adsk.eagle:library:334" deviceset="C-EU" device="C1206" package3d_urn="urn:adsk.eagle:package:23618/2" value="10uF"/>
 <part name="L1" library="LQM31PN1R0M00L" deviceset="LQM31PN1R0M00L" device=""/>
+<part name="OSC32" library="ABS07-32.768KHZ-7-T" deviceset="ABS07-32.768KHZ-7-T" device=""/>
+<part name="CLO1" library="rcl" library_urn="urn:adsk.eagle:library:334" deviceset="C-EU" device="C1206" package3d_urn="urn:adsk.eagle:package:23618/2" value="15pF"/>
+<part name="CLO2" library="rcl" library_urn="urn:adsk.eagle:library:334" deviceset="C-EU" device="C1206" package3d_urn="urn:adsk.eagle:package:23618/2" value="15pF"/>
+<part name="U$3" library="SAMTEC-TSM-104-01-X-SH" deviceset="SAMTEC-TSM-104-01-X-SH" device="J"/>
+<part name="U$4" library="SAMTEC-TSM-104-01-X-SH" deviceset="SAMTEC-TSM-104-01-X-SH" device="J"/>
 </parts>
 <sheets>
@@
 <instance part="CB2" gate="G$1" x="116.84" y="-45.72" rot="R180"/>
 <instance part="L1" gate="G$1" x="91.44" y="-35.56"/>
+<instance part="OSC32" gate="G$1" x="58.42" y="-81.28" rot="R270"/>
+<instance part="CLO1" gate="G$1" x="43.18" y="-81.28" rot="R90"/>
+<instance part="CLO2" gate="G$1" x="43.18" y="-101.6" rot="R90"/>
+<instance part="U$3" gate="A" x="335.28" y="-73.66" rot="R90"/>
+<instance part="U$4" gate="A" x="386.08" y="-73.66" rot="R90"/>
 </instances>
 <busses>
@@
 <junction x="27.94" y="-53.34"/>
 </segment>
+<segment>
+<pinref part="GND_NRST" gate="1" pin="P"/>
+<wire x1="238.76" y1="-114.3" x2="238.76" y2="-127" width="0.1524" layer="91"/>
+<label x="238.76" y="-127" size="1.27" layer="95" rot="R270" xref="yes"/>
+</segment>
+<segment>
+<pinref part="GND_PRG" gate="1" pin="P"/>
+<wire x1="254" y1="-114.3" x2="254" y2="-127" width="0.1524" layer="91"/>
+<label x="254" y="-127" size="1.27" layer="95" rot="R270" xref="yes"/>
+</segment>
+<segment>
+<wire x1="33.02" y1="-91.44" x2="27.94" y2="-91.44" width="0.1524" layer="91"/>
+<label x="27.94" y="-91.44" size="1.016" layer="95" rot="R180" xref="yes"/>
+<pinref part="CLO1" gate="G$1" pin="1"/>
+<wire x1="40.64" y1="-81.28" x2="33.02" y2="-81.28" width="0.1524" layer="91"/>
+<wire x1="33.02" y1="-81.28" x2="33.02" y2="-91.44" width="0.1524" layer="91"/>
+<wire x1="33.02" y1="-91.44" x2="33.02" y2="-101.6" width="0.1524" layer="91"/>
+<junction x="33.02" y="-91.44"/>
+<pinref part="CLO2" gate="G$1" pin="1"/>
+<wire x1="33.02" y1="-101.6" x2="40.64" y2="-101.6" width="0.1524" layer="91"/>
+</segment>
 </net>
 <net name="+3V3" class="0">
@@
 <label x="226.06" y="15.24" size="1.27" layer="95" rot="R180" xref="yes"/>
 </segment>
+<segment>
+<pinref part="CLO1" gate="G$1" pin="2"/>
+<pinref part="OSC32" gate="G$1" pin="1"/>
+<wire x1="48.26" y1="-81.28" x2="58.42" y2="-81.28" width="0.1524" layer="91"/>
+<wire x1="58.42" y1="-81.28" x2="81.28" y2="-81.28" width="0.1524" layer="91"/>
+<junction x="58.42" y="-81.28"/>
+<label x="81.28" y="-81.28" size="1.016" layer="95" xref="yes"/>
+</segment>
 </net>
 <net name="X32OUT" class="0">
@@
 <wire x1="233.68" y1="12.7" x2="226.06" y2="12.7" width="0.1524" layer="91"/>
 <label x="226.06" y="12.7" size="1.27" layer="95" rot="R180" xref="yes"/>
+</segment>
+<segment>
+<pinref part="CLO2" gate="G$1" pin="2"/>
+<pinref part="OSC32" gate="G$1" pin="2"/>
+<wire x1="48.26" y1="-101.6" x2="58.42" y2="-101.6" width="0.1524" layer="91"/>
+<wire x1="58.42" y1="-101.6" x2="81.28" y2="-101.6" width="0.1524" layer="91"/>
+<junction x="58.42" y="-101.6"/>
+<label x="81.28" y="-101.6" size="1.016" layer="95" xref="yes"/>
 </segment>
 </net>
@@
 <wire x1="261.62" y1="66.04" x2="261.62" y2="68.58" width="0.1524" layer="91"/>
 <label x="261.62" y="68.58" size="1.27" layer="95" rot="R90" xref="yes"/>
+</segment>
+<segment>
+<pinref part="PAD_NRST" gate="1" pin="P"/>
+<wire x1="238.76" y1="-104.14" x2="238.76" y2="-91.44" width="0.1524" layer="91"/>
+<label x="238.76" y="-91.44" size="1.27" layer="95" rot="R90" xref="yes"/>
 </segment>
 </net>
@@
 </segment>
 </net>
+<net name="N$3" class="0">
+<segment>
+<pinref part="PAD_PRG" gate="1" pin="P"/>
+<wire x1="254" y1="-104.14" x2="254" y2="-91.44" width="0.1524" layer="91"/>
+<label x="254" y="-91.44" size="1.27" layer="95" rot="R90" xref="yes"/>
+</segment>
+</net>

Commit message: updates
Connections:
- new net USBVCC: U$3.4
- net GND: now also U$3.1, U$4.4
- net PA02: now also RS4.2
- net PA04: now also RS3.2
- net PA06: now also RP2.2
- net PA07: now also RP1.2
- net PB08: now also RS2.2
- net PB09: now also RS1.2
- net RESET: now also U$4.3
- net SWCLK: now also U$4.2
- net SWDIO: now also U$4.1
- net USB+: now also U$3.2
- net USB-: now also U$3.3
