File: eagle/4ButtonSwitch.Rev3.0.brd (EAGLE design)
At the start: 69.8 x 69.8 mm, 37 parts, among them U1 ADP2108AUJZ-3.3-R7

Commit message: updates
Parts:
- added CLO1, CLO2: 15pF, rcl:C1206
- added OSC32: ABS07-32.768KHZ-7-T, ABS07-32.768KHZ-7-T:ABS-07
- added U$3, U$4: SAMTEC-TSM-104-01-X-SHJ, SAMTEC-TSM-104-01-X-SH:SAMTEC-TSM-104-01-X-SH
- moved CR1 19.8 mm to (12.7, 24.1), turned to 180 degrees
- moved R1 18.3 mm to (25.4, 36.2), turned to 180 degrees
- moved RR1 15.7 mm to (12.7, 26.7), turned to 0 degrees
- moved RI2 14.4 mm to (44.5, 41.9), turned to 180 degrees
- moved RI1 13.9 mm to (44.5, 39.4), turned to 0 degrees
- moved RL2 12.7 mm to (12.7, 50.2), turned to 0 degrees
- moved RL1 12.7 mm to (57.1, 50.2)
- moved RL3 11.7 mm to (47.0, 14.0), turned to 0 degrees
- moved RL4 11.7 mm to (22.9, 14.0), turned to 180 degrees
- moved GND_NRST 10.2 mm to (6.99, 40.0)
- moved PAD_NRST 10.2 mm to (6.99, 29.8)
- moved CS1 9.71 mm to (25.4, 43.8)
- moved CC1 9.71 mm to (25.4, 41.3), turned to 180 degrees
- moved RR2 8.03 mm to (12.7, 29.2), turned to 180 degrees
- moved RP2 7.41 mm to (55.9, 27.9), turned to 180 degrees
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Connections:
- new net N$3: PAD_PRG.1
- net GND: now also CLO1.1, CLO2.1, GND_NRST.1, GND_PRG.1
- net RESET: now also PAD_NRST.1
- net X32IN: now also CLO1.2, OSC32.1
- net X32OUT: now also CLO2.2, OSC32.2
Routing:
- net SENS_4: track 0.00 -> 2.52 mm, vias 0 -> 1
- net SENS_3: track 0.00 -> 2.52 mm, vias 0 -> 1
- net SENS_2: track 0.00 -> 2.39 mm, vias 0 -> 1
- net SENS_1: track 0.00 -> 2.39 mm, vias 0 -> 1

Commit message: updates
Parts:
- moved RP2 1.27 mm to (55.9, 29.2)
- moved RP1 1.27 mm to (55.9, 40.6)
- turned CS1 to 180 degrees
- turned CS4 to 0 degrees
- turned R1 to 0 degrees
Connections:
- new net USBVCC: U$3.4
- net GND: now also U$3.1, U$4.4
- net PA02: now also RS4.2
- net PA04: now also RS3.2
- net PA06: now also RP2.2
- net PA07: now also RP1.2
- net PB08: now also RS2.2
- net PB09: now also RS1.2
- net RESET: now also U$4.3
- net SWCLK: now also U$4.2
- net SWDIO: now also U$4.1
- net USB+: now also U$3.2
- net USB-: now also U$3.3
Routing:
- net +3V3: track 0.00 -> 70.2 mm, vias 0 -> 2
- net SWCLK: track 0.00 -> 25.0 mm, vias 0 -> 4
- net +5V: track 7.15 -> 27.9 mm
- net SWDIO: track 0.00 -> 15.4 mm, vias 0 -> 2
- net USB+: track 0.00 -> 11.5 mm
- net USB-: track 0.00 -> 9.43 mm
- net VDDCORE: track 0.00 -> 5.60 mm
- net GND: track 7.53 -> 11.2 mm
- net N$2: track 0.00 -> 3.56 mm
- added copper zone on layer 1, net +3V3

Commit message: updates
Parts:
- removed RI1, RI2: 4k7, resistor:R1206
- moved R1 20.5 mm to (44.5, 43.8)
- moved RS2 7.24 mm to (25.4, 36.2), turned to 0 degrees
- moved RS1 5.71 mm to (44.5, 40.6), turned to 180 degrees
- moved U$3 0.64 mm to (27.9, 54.0)
Connections:
- net +3V3: no longer RI1.2, RI2.1
- net PA04: now also RP2.2; no longer RS3.2
- net PA05: now also RP1.2
- net PA06: no longer RP2.2
- net PA07: now also RS1.2; no longer RP1.2
- net PA22: no longer RI2.2
- net PA23: no longer RI1.1
- net PB02: now also RS2.2
- net PB08: now also RS3.2; no longer RS2.2
- net PB09: no longer RS1.2
Routing:
- net GND: track 11.2 -> 40.9 mm
- net SWCLK: track 25.0 -> 11.4 mm, vias 4 -> 2
- net SENS_PROX_2: track 114.5 -> 125.4 mm, vias 2 -> 3
- net SENS_PROX_1: track 114.5 -> 125.4 mm, vias 2 -> 3
- net +3V3: track 70.2 -> 61.2 mm, vias 2 -> 3
- net X32OUT: track 0.00 -> 8.01 mm
- net +5V: track 27.9 -> 20.7 mm, vias 1 -> 0
- net NRST: track 0.00 -> 6.45 mm
- net X32IN: track 0.00 -> 5.99 mm
- net SENS_2: track 2.39 -> 0.00 mm
- net SENS_1: track 2.39 -> 0.00 mm
- net VDDCORE: track 5.60 -> 4.93 mm
- net USB-: track 9.43 -> 8.87 mm
