File: eagle/4ButtonSwitch.Rev4.0.brd (EAGLE design)
At the start: 69.8 x 69.8 mm, 40 parts, among them U1 ADP2108AUJZ-3.3-R7

Commit message: updates
Parts:
- moved RS2 15.9 mm to (25.4, 36.2), turned to 0 degrees
Connections:
- net PA04: now also RP2.2; no longer RS3.2
- net PA05: now also RP1.2
- net PA06: no longer RP2.2
- net PA07: now also RS1.2; no longer RP1.2
- net PA16: no longer RS1.2
- net PA19: no longer RS2.2
- net PB02: now also RS2.2
- net PB08: now also RS3.2
Routing:
- net PA06: track 20.4 -> 0.00 mm
- net PA07: track 19.1 -> 0.00 mm
- net PA04: track 16.7 -> 0.00 mm
- net PA02: track 15.9 -> 0.00 mm, vias 2 -> 0
Changed lines of the file:
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@@
 <setting verticaltext="up"/>
 </settings>
-<grid distance="50" unitdist="mil" unit="inch" style="lines" multiple="1" display="yes" altdistance="5" altunitdist="mil" altunit="inch"/>
+<grid distance="50" unitdist="mil" unit="inch" style="lines" multiple="1" display="yes" altdistance="0.025" altunitdist="inch" altunit="inch"/>
 <layers>
 <layer number="1" name="Top" color="4" fill="1" visible="yes" active="yes"/>
-<layer number="2" name="Route2" color="1" fill="3" visible="no" active="no"/>
+<layer number="2" name="Route2" color="1" fill="3" visible="no" active="yes"/>
 <layer number="3" name="Route3" color="4" fill="3" visible="no" active="no"/>
 <layer number="4" name="Route4" color="1" fill="4" visible="no" active="no"/>
@@
 <layer number="13" name="Route13" color="4" fill="5" visible="no" active="no"/>
 <layer number="14" name="Route14" color="1" fill="6" visible="no" active="no"/>
-<layer number="15" name="Route15" color="4" fill="6" visible="no" active="no"/>
+<layer number="15" name="Route15" color="4" fill="6" visible="no" active="yes"/>
 <layer number="16" name="Bottom" color="1" fill="1" visible="yes" active="yes"/>
 <layer number="17" name="Pads" color="2" fill="1" visible="yes" active="yes"/>
@@
 </class>
 </classes>
-<designrules name="konnektduino">
+<designrules name="konnektduino *">
 <description language="de">&lt;b&gt;EAGLE Design Rules&lt;/b&gt;
 &lt;p&gt;
@@
 necessary adjustments and save your customized
 design rules under a new name.</description>
-<param name="layerSetup" value="(1*16)"/>
+<param name="layerSetup" value="(1*2*15*16)"/>
 <param name="mtCopper" value="0.035mm 0.035mm 0.035mm 0.035mm 0.035mm 0.035mm 0.035mm 0.035mm 0.035mm 0.035mm 0.035mm 0.035mm 0.035mm 0.035mm 0.035mm 0.035mm"/>
-<param name="mtIsolate" value="1.5mm 0.15mm 0.2mm 0.15mm 0.2mm 0.15mm 0.2mm 0.15mm 0.2mm 0.15mm 0.2mm 0.15mm 0.2mm 0.15mm 0.2mm"/>
+<param name="mtIsolate" value="0.23mm 0.93mm 0.2mm 0.15mm 0.2mm 0.15mm 0.2mm 0.15mm 0.2mm 0.15mm 0.2mm 0.15mm 0.2mm 0.15mm 0.23mm"/>
 <param name="mdWireWire" value="6mil"/>
 <param name="mdWirePad" value="6mil"/>
@@
 <attribute name="VALUE" x="52.07" y="28.575" size="1.27" layer="27" rot="R90"/>
 </element>
-<element name="RS2" library="resistor" library_urn="urn:adsk.eagle:library:348" package="R1206" package3d_urn="urn:adsk.eagle:package:26062/1" value="1k" x="34.925" y="48.895" smashed="yes" rot="R270">
-<attribute name="NAME" x="34.417" y="53.467" size="1.016" layer="25" rot="R270"/>
-<attribute name="VALUE" x="33.02" y="49.53" size="1.27" layer="27" rot="R270"/>
+<element name="RS2" library="resistor" library_urn="urn:adsk.eagle:library:348" package="R1206" package3d_urn="urn:adsk.eagle:package:26062/1" value="1k" x="25.4" y="36.195" smashed="yes">
+<attribute name="NAME" x="20.828" y="35.687" size="1.016" layer="25"/>
+<attribute name="VALUE" x="24.765" y="34.29" size="1.27" layer="27"/>
 </element>
 <element name="RS1" library="resistor" library_urn="urn:adsk.eagle:library:348" package="R1206" package3d_urn="urn:adsk.eagle:package:26062/1" value="1k" x="44.45" y="40.64" smashed="yes" rot="R180">
@@
 </polygon>
 <contactref element="RS2" pad="1"/>
-<via x="29.845" y="53.34" extent="1-16" drill="0.35"/>
-<wire x1="29.845" y1="53.34" x2="34.925" y2="50.317" width="0" layer="19" extent="1-1"/>
+<via x="19.685" y="44.45" extent="1-16" drill="0.35"/>
+<wire x1="19.685" y1="44.45" x2="23.978" y2="36.195" width="0" layer="19" extent="1-1"/>
 </signal>
 <signal name="SENS_4">
@@
 <contactref element="SAMD" pad="3"/>
 <contactref element="RS4" pad="2"/>
-<wire x1="33.175" y1="35.132" x2="33.175" y2="34.191" width="0.1524" layer="1"/>
-<wire x1="29.591" y1="30.607" x2="29.083" y2="30.607" width="0.1524" layer="1"/>
-<via x="29.083" y="30.607" extent="1-16" drill="0.35"/>
-<wire x1="29.083" y1="30.607" x2="21.209" y2="30.607" width="0.1524" layer="16"/>
-<via x="21.209" y="30.607" extent="1-16" drill="0.35"/>
-<wire x1="21.209" y1="30.607" x2="19.71" y2="30.607" width="0.1524" layer="1"/>
-<wire x1="19.71" y1="30.607" x2="19.685" y2="30.632" width="0.1524" layer="1"/>
-<wire x1="33.175" y1="34.191" x2="29.591" y2="30.607" width="0.1524" layer="1"/>
+<wire x1="19.685" y1="30.632" x2="33.175" y2="35.132" width="0" layer="19" extent="1-1"/>
 </signal>
 <signal name="PA03">
@@
 <signal name="PB08">
 <contactref element="SAMD" pad="7"/>
+<contactref element="RS3" pad="2"/>
+<wire x1="35.175" y1="35.132" x2="50.165" y2="30.632" width="0" layer="19" extent="1-1"/>
 </signal>
 <signal name="PB09">
@@
 <signal name="PA04">
 <contactref element="SAMD" pad="9"/>
-<contactref element="RS3" pad="2"/>
-<wire x1="36.175" y1="35.132" x2="36.175" y2="33.675" width="0.1524" layer="1"/>
-<wire x1="40.132" y1="33.147" x2="42.672" y2="30.607" width="0.1524" layer="1"/>
-<wire x1="42.672" y1="30.607" x2="50.14" y2="30.607" width="0.1524" layer="1"/>
-<wire x1="50.14" y1="30.607" x2="50.165" y2="30.632" width="0.1524" layer="1"/>
-<wire x1="36.175" y1="33.675" x2="36.703" y2="33.147" width="0.1524" layer="1"/>
-<wire x1="36.703" y1="33.147" x2="40.132" y2="33.147" width="0.1524" layer="1"/>
+<contactref element="RP2" pad="2"/>
+<wire x1="36.175" y1="35.132" x2="54.458" y2="29.21" width="0" layer="19" extent="1-1"/>
 </signal>
 <signal name="PA05">
 <contactref element="SAMD" pad="10"/>
+<contactref element="RP1" pad="2"/>
+<wire x1="36.675" y1="35.132" x2="54.458" y2="40.64" width="0" layer="19" extent="1-1"/>
 </signal>
 <signal name="PA06">
 <contactref element="SAMD" pad="11"/>
-<contactref element="RP2" pad="2"/>
-<wire x1="37.175" y1="35.132" x2="37.175" y2="34.072" width="0.1524" layer="1"/>
-<wire x1="49.759" y1="33.909" x2="54.458" y2="29.21" width="0.1524" layer="1"/>
-<wire x1="37.175" y1="34.072" x2="37.338" y2="33.909" width="0.1524" layer="1"/>
-<wire x1="37.338" y1="33.909" x2="49.759" y2="33.909" width="0.1524" layer="1"/>
 </signal>
 <signal name="PA07">
 <contactref element="SAMD" pad="12"/>
-<contactref element="RP1" pad="2"/>
-<wire x1="37.675" y1="35.132" x2="48.95" y2="35.132" width="0.1524" layer="1"/>
-<wire x1="48.95" y1="35.132" x2="54.458" y2="40.64" width="0.1524" layer="1"/>
+<contactref element="RS1" pad="2"/>
+<wire x1="37.675" y1="35.132" x2="43.028" y2="40.64" width="0" layer="19" extent="1-1"/>
 </signal>
 <signal name="PA08">
@@
 <signal name="PA19">
 <contactref element="SAMD" pad="28"/>
-<contactref element="RS2" pad="2"/>
-<wire x1="34.925" y1="47.473" x2="36.175" y2="43.608" width="0" layer="19" extent="1-1"/>
 </signal>
 <signal name="PA18">
@@
 <signal name="PA16">
 <contactref element="SAMD" pad="25"/>
-<contactref element="RS1" pad="2"/>
-<wire x1="37.675" y1="43.608" x2="43.028" y2="40.64" width="0" layer="19" extent="1-1"/>
 </signal>
 <signal name="PB03">
@@
 <signal name="PB02">
 <contactref element="SAMD" pad="47"/>
+<contactref element="RS2" pad="2"/>
+<wire x1="26.822" y1="36.195" x2="30.687" y2="37.12" width="0" layer="19" extent="1-1"/>
 </signal>
 <signal name="PA28">
