File: eagle/4ButtonSwitch.ItsyBitsyM0.Rev1.0.brd (EAGLE design)
At the start: 69.8 x 69.8 mm, 40 parts, among them U1 ADP2108AUJZ-3.3-R7

Commit message: updates
Parts:
- removed CB1: 4.7uF, rcl:C1206
- removed CB2: 10uF, rcl:C1206
- removed CC1: 1uF, rcl:C1206
- removed CLO1, CLO2: 15pF, rcl:C1206
- removed CR1: 100pF, rcl:C1206
- removed CS1, CS2, CS3, CS4: 100nf, rcl:C1206
- removed L1: LQM31PN1R0M00L, LQM31PN1R0M00L:INDC3216X95N
- removed OSC32: ABS07-32.768KHZ-7-T, ABS07-32.768KHZ-7-T:ABS-07
- removed R1: 1k, resistor:R1206
- removed RR1: 2.2k, resistor:R1206
- removed RR2: 330E, resistor:R1206
- removed SAMD: ATSAMD21G18A-AU, ATSAMD21G18A-AU:QFP50P900X900X120-48N
- removed U$3, U$4: SAMTEC-TSM-104-01-X-SHJ, SAMTEC-TSM-104-01-X-SH:SAMTEC-TSM-104-01-X-SH
- removed U1: ADP2108AUJZ-3.3-R7, ADP2108AUJZ-3.3-R7CT-ND:UJ_5
- added JP1, JP2: (no value), pinhead+:1X14_SMT
- moved PAD_NRST 56.8 mm to (62.9, 40.0)
- moved PAD_PRG 56.8 mm to (6.99, 29.8)
- moved RS2 17.3 mm to (19.7, 40.6)
- moved RL3 15.3 mm to (47.6, 29.2), turned to 270 degrees
- moved RL4 15.3 mm to (22.2, 29.2), turned to 270 degrees
- moved RL2 13.5 mm to (22.2, 40.6), turned to 90 degrees
- moved RL1 13.5 mm to (47.6, 40.6), turned to 90 degrees
- moved RS1 5.71 mm to (50.2, 40.6), turned to 270 degrees
Connections:
- removed net NRST: CR1.2, RR1.1, RR2.1, SAMD.40
- removed net PA03: SAMD.4
- removed net PA06: RP2.2, SAMD.11
- removed net PA08: SAMD.13
- removed net PA09: SAMD.14
- removed net PA10: SAMD.15
- removed net PA11: SAMD.16
- removed net PA12: SAMD.21
- removed net PA13: SAMD.22
- removed net PA14: SAMD.23
- removed net PA15: SAMD.24
- removed net PA16: RS1.2, SAMD.25
- removed net PA17: SAMD.26
- removed net PA18: SAMD.27
- removed net PA19: RS2.2, SAMD.28
- removed net PA20: SAMD.29
- removed net PA21: SAMD.30
- removed net PA22: SAMD.31
- removed net PA23: SAMD.32
- removed net PA27: SAMD.39
- removed net PA28: SAMD.41
- removed net PB03: SAMD.48
- removed net PB09: SAMD.8
- removed net PB10: SAMD.19
- removed net PB11: SAMD.20
- removed net PB22: SAMD.37
- removed net PB23: SAMD.38
- removed net SWCLK: R1.1, SAMD.45, U$4.2
- removed net SWDIO: SAMD.46, U$4.1
- removed net USB+: SAMD.34, U$3.2
- removed net USB-: SAMD.33, U$3.3
- removed net USBVCC: U$3.4
- removed net VDDCORE: CC1.1, SAMD.43
- removed net X32IN: CLO1.2, OSC32.1, SAMD.1
- removed net X32OUT: CLO2.2, OSC32.2, SAMD.2
- new net A0: JP2.10
- new net A1: JP2.9
- new net A2: JP2.8
- new net A3: JP2.7
- new net A4: JP2.6
- new net A5: JP2.5
- new net N$1: JP1.11
- new net N$4: JP1.9
- new net N$5: JP1.8
- new net N$6: JP1.7
- new net N$7: JP1.6
- new net RX: JP1.1
- new net SCL: JP1.4
- new net SDA: JP1.3
- new net TX: JP1.2
- net +3V3: now also JP2.13; no longer CB2.2, CR1.1, CS1.1, CS2.1, CS3.1, CS4.1, L1.2, R1.2, RR1.2, SAMD.17, SAMD.36, SAMD.44, SAMD.6, U1.4
- net +5V: now also JP1.14; no longer CB1.2, U1.1, U1.3
- net GND: now also JP1.13; no longer CB1.1, CB2.1, CC1.2, CLO1.1, CLO2.1, CS1.2, CS2.2, CS3.2, CS4.2, SAMD.18, SAMD.35, SAMD.42, SAMD.5, U$3.1, U$4.4, U1.2
- net N$2: now also JP1.10; no longer L1.1, U1.5
- net PA02: no longer SAMD.3
- net PA04: now also RP2.2; no longer RS3.2, SAMD.9
- net PA05: now also RP1.2; no longer SAMD.10
- net PA07: now also RS1.2; no longer RP1.2, SAMD.12
- net PB02: now also RS2.2; no longer SAMD.47
- net PB08: now also RS3.2; no longer SAMD.7
- net RESET: now also JP2.14; no longer RR2.2, U$4.3
Routing:
- net +3V3: track 61.2 -> 0.00 mm, vias 3 -> 1
- net GND: track 40.9 -> 0.00 mm
- net +5V: track 20.7 -> 0.00 mm
- net PA06: track 20.4 -> 0.00 mm
- net PA07: track 19.1 -> 0.00 mm
- net PA04: track 16.7 -> 0.00 mm
- net PA02: track 15.9 -> 0.00 mm, vias 2 -> 0
- net SWDIO: track 15.4 -> 0.00 mm, vias 2 -> 0
- net SWCLK: track 11.4 -> 0.00 mm, vias 2 -> 0
- net USB+: track 11.1 -> 0.00 mm
- net SENS_PROX_2: track 125.4 -> 115.4 mm, vias 3 -> 2
- net SENS_PROX_1: track 125.4 -> 115.4 mm, vias 3 -> 2
- net USB-: track 8.87 -> 0.00 mm
- net X32OUT: track 8.01 -> 0.00 mm
- net NRST: track 6.45 -> 0.00 mm
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- removed copper zone on layer 1, net +3V3
Other:
- board text added: "4xTouch Button | Itsy Bitsy M0 | Rev 1.0"
- board text added: "Konnekting | 0XCDDC | 2019 by ChriD"
- board text removed: "4xTouch Button Rev 3.0"
- board text removed: "5V-30V"
- board text removed: "Konnekting | 0XCDDC | 2018 by ChriD"

Commit message: update
Parts:
- moved RL1 6.63 mm to (49.5, 47.0), turned to 0 degrees
- moved RL2 6.63 mm to (20.3, 47.0), turned to 180 degrees
- moved RL3 6.63 mm to (49.5, 22.9), turned to 0 degrees
- moved RL4 6.63 mm to (20.3, 22.9), turned to 180 degrees
- moved RS2 0.64 mm to (20.3, 40.6), turned to 0 degrees
- moved RS4 0.64 mm to (20.3, 29.2), turned to 0 degrees
- moved RS1 0.63 mm to (49.5, 40.6), turned to 180 degrees
- moved RS3 0.63 mm to (49.5, 29.2), turned to 180 degrees
Connections:
- net N$4 renamed D11
- removed net LED1: RL1.1
- removed net LED2: RL2.1
- removed net LED3: RL3.1
- removed net LED4: RL4.1
- removed net N$1: JP1.11
- removed net N$2: JP1.10
- removed net N$3: PAD_PRG.1
- removed net N$5: JP1.8
- removed net N$6: JP1.7
- removed net N$7: JP1.6
- removed net PA02: RS4.2
- removed net PA04: RP2.2
- removed net PA05: RP1.2
- removed net PA07: RS1.2
- removed net PB02: RS2.2
- removed net PB08: RS3.2
- removed net RX: JP1.1
- removed net TX: JP1.2
- new net D10: JP1.8, PAD_PRG.1
- new net D12: JP1.10, RL1.1
- new net D13: JP1.11, RL2.1
- new net D7: JP1.6, RL3.1
- new net D9: JP1.7, RL4.1
- net A0: now also RS2.2
- net A1: now also RS1.2
- net A2: now also RP1.2
- net A3: now also RS4.2
- net A4: now also RP2.2
- net A5: now also RS3.2
- net USART1_RX: now also JP1.1
- net USART1_TX: now also JP1.2
Routing:
- net +5V: track 0.00 -> 57.0 mm, vias 0 -> 1
- net RESET: track 0.00 -> 34.8 mm
- net D10: track 0.00 -> 28.0 mm
- net D7: track 0.00 -> 27.9 mm, vias 0 -> 2
- net GND: track 0.00 -> 27.6 mm, vias 1 -> 4
- net A0: track 0.00 -> 25.0 mm, vias 0 -> 2
- net A3: track 0.00 -> 23.5 mm, vias 0 -> 2
- net USART1_TX: track 0.00 -> 20.9 mm, vias 0 -> 2
- net USART1_RX: track 0.00 -> 20.6 mm, vias 0 -> 2
- net D12: track 0.00 -> 20.3 mm, vias 0 -> 2
- net D9: track 0.00 -> 19.4 mm
- net A4: track 0.00 -> 13.5 mm
- net A2: track 0.00 -> 13.5 mm
- net A5: track 0.00 -> 10.8 mm
- net SENS_PROX_2: track 115.4 -> 125.4 mm, vias 2 -> 3
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Other:
- board text added: "SH"
