File: eagle/4ButtonSwitch.ItsyBitsyM0.Rev1.0.sch (EAGLE design)
At the start: 21 parts

Commit message: update
Connections:
- net N$4 renamed D11
- removed net LED1: RL1.1
- removed net LED2: RL2.1
- removed net LED3: RL3.1
- removed net LED4: RL4.1
- removed net N$1: JP1.11
- removed net N$2: JP1.10
- removed net N$3: PAD_PRG.P
- removed net N$5: JP1.8
- removed net N$6: JP1.7
- removed net N$7: JP1.6
- removed net PA02: RS4.2
- removed net PA04: RP2.2
- removed net PA05: RP1.2
- removed net PA07: RS1.2
- removed net PB02: RS2.2
- removed net PB08: RS3.2
- removed net RX: JP1.1
- removed net TX: JP1.2
- new net D10: JP1.8, PAD_PRG.P
- new net D12: JP1.10, RL1.1
- new net D13: JP1.11, RL2.1
- new net D7: JP1.6, RL3.1
- new net D9: JP1.7, RL4.1
- net A0: now also RS2.2
- net A1: now also RS1.2
- net A2: now also RP1.2
- net A3: now also RS4.2
- net A4: now also RP2.2
- net A5: now also RS3.2
- net USART1_RX: now also JP1.1
- net USART1_TX: now also JP1.2
