File: eagle/4ButtonSwitch.ItsyBitsyM0.Rev1.1.brd (EAGLE design)
At the start: 69.8 x 69.8 mm, 23 parts

Commit message: updates
Connections:
- net D11: now also RL3.1
- net D7: no longer RL3.1
Routing:
- net D11: track 0.00 -> 38.7 mm, vias 0 -> 2
- net D7: track 26.9 -> 0.00 mm, vias 2 -> 0
Changed lines of the file:
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@@
 <signal name="D11">
 <contactref element="JP1" pad="9"/>
+<contactref element="RL3" pad="1"/>
+<wire x1="48.108" y1="22.86" x2="48.108" y2="25.552" width="0.3048" layer="1"/>
+<wire x1="43.18" y1="30.48" x2="39.37" y2="30.48" width="0.3048" layer="1"/>
+<wire x1="39.37" y1="30.48" x2="36.83" y2="33.02" width="0.3048" layer="1"/>
+<via x="36.83" y="33.02" extent="1-16" drill="0.35"/>
+<wire x1="36.83" y1="33.02" x2="36.83" y2="43.053" width="0.3048" layer="16"/>
+<wire x1="36.83" y1="43.053" x2="35.433" y2="44.45" width="0.3048" layer="16"/>
+<via x="35.433" y="44.45" extent="1-16" drill="0.35"/>
+<wire x1="35.433" y1="44.45" x2="25.785" y2="44.45" width="0.3048" layer="1"/>
+<wire x1="48.108" y1="25.552" x2="43.18" y2="30.48" width="0.3048" layer="1"/>
 </signal>
 <signal name="D10">
@@
 <signal name="D7">
 <contactref element="JP1" pad="6"/>
-<contactref element="RL3" pad="1"/>
-<wire x1="48.108" y1="22.86" x2="46.355" y2="24.613" width="0.1524" layer="1"/>
-<wire x1="46.355" y1="24.613" x2="46.355" y2="27.813" width="0.1524" layer="1"/>
-<wire x1="46.355" y1="27.813" x2="43.815" y2="30.353" width="0.1524" layer="1"/>
-<wire x1="43.815" y1="30.353" x2="42.037" y2="30.353" width="0.1524" layer="1"/>
-<wire x1="42.037" y1="30.353" x2="38.608" y2="33.782" width="0.1524" layer="1"/>
-<via x="38.608" y="33.782" extent="1-16" drill="0.35"/>
-<wire x1="38.608" y1="33.782" x2="35.56" y2="36.83" width="0.1524" layer="16"/>
-<via x="35.56" y="36.83" extent="1-16" drill="0.35"/>
-<wire x1="35.56" y1="36.83" x2="28.825" y2="36.83" width="0.1524" layer="1"/>
 </signal>
 </signals>

Commit message: updates
Parts:
- added CRST: 100nF, rcl:C1206
- added RRST1: 10k, resistor:R1206
- added RRST2: 330, resistor:R1206
Connections:
- new net RST: CRST.1, JP2.14, RRST1.1, RRST2.1
- net +3V3: now also RRST1.2
- net GND: now also CRST.2
- net RESET: now also RRST2.2; no longer JP2.14
Routing:
- net RESET: track 34.8 -> 17.0 mm
- net RST: track 0.00 -> 16.3 mm
- net +3V3: track 0.00 -> 7.70 mm
Changed lines of the file:
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@@
 <drawing>
 <settings>
-<setting alwaysvectorfont="no"/>
+<setting alwaysvectorfont="yes"/>
 <setting verticaltext="up"/>
 </settings>
@@
 <element name="JP1" library="pinhead+" package="1X14_SMT" value="" x="27.305" y="40.64" rot="R90"/>
 <element name="JP2" library="pinhead+" package="1X14_SMT" value="" x="42.545" y="40.64" rot="R90"/>
+<element name="RRST1" library="resistor" library_urn="urn:adsk.eagle:library:348" package="R1206" package3d_urn="urn:adsk.eagle:package:26062/1" value="10k" x="48.26" y="57.15" rot="R270"/>
+<element name="CRST" library="rcl" library_urn="urn:adsk.eagle:library:334" package="C1206" package3d_urn="urn:adsk.eagle:package:23618/2" value="100nF" x="55.88" y="57.28" rot="R270">
+<attribute name="SPICEPREFIX" value="C" x="55.88" y="57.28" size="1.778" layer="27" rot="R270" display="off"/>
+</element>
+<element name="RRST2" library="resistor" library_urn="urn:adsk.eagle:library:348" package="R1206" package3d_urn="urn:adsk.eagle:package:26062/1" value="330" x="59.69" y="57.15" rot="R270"/>
 </elements>
 <signals>
@@
 <via x="36.195" y="5.08" extent="1-16" drill="1"/>
 <wire x1="25.785" y1="54.61" x2="38.1" y2="54.61" width="0.3048" layer="1"/>
+<contactref element="CRST" pad="2"/>
 </signal>
 <signal name="+3V3">
 <contactref element="JP2" pad="13"/>
+<contactref element="RRST1" pad="2"/>
+<wire x1="41.025" y1="54.61" x2="47.142" y2="54.61" width="0.1524" layer="1"/>
+<wire x1="47.142" y1="54.61" x2="48.26" y2="55.728" width="0.1524" layer="1"/>
 </signal>
 <signal name="SENS_PROX_1">
@@
 <signal name="RESET">
 <contactref element="PAD_NRST" pad="1"/>
-<contactref element="JP2" pad="14"/>
-<wire x1="62.865" y1="40.005" x2="62.865" y2="55.245" width="0.1524" layer="1"/>
-<wire x1="62.865" y1="55.245" x2="60.96" y2="57.15" width="0.1524" layer="1"/>
-<wire x1="60.96" y1="57.15" x2="44.065" y2="57.15" width="0.1524" layer="1"/>
+<contactref element="RRST2" pad="2"/>
+<wire x1="62.865" y1="40.005" x2="62.865" y2="52.553" width="0.1524" layer="1"/>
+<wire x1="62.865" y1="52.553" x2="59.69" y2="55.728" width="0.1524" layer="1"/>
 </signal>
 <signal name="A0">
@@
 <contactref element="JP1" pad="6"/>
 </signal>
+<signal name="RST">
+<contactref element="JP2" pad="14"/>
+<contactref element="RRST1" pad="1"/>
+<contactref element="CRST" pad="1"/>
+<contactref element="RRST2" pad="1"/>
+<wire x1="59.69" y1="58.572" x2="55.988" y2="58.572" width="0.1524" layer="1"/>
+<wire x1="55.988" y1="58.572" x2="55.88" y2="58.68" width="0.1524" layer="1"/>
+<wire x1="55.88" y1="58.68" x2="48.368" y2="58.68" width="0.1524" layer="1"/>
+<wire x1="48.368" y1="58.68" x2="48.26" y2="58.572" width="0.1524" layer="1"/>
+<wire x1="44.065" y1="57.15" x2="46.838" y2="57.15" width="0.1524" layer="1"/>
+<wire x1="46.838" y1="57.15" x2="48.26" y2="58.572" width="0.1524" layer="1"/>
+</signal>
 </signals>
