File: eagle/4ButtonSwitch.ItsyBitsyM0.Rev1.1.brd (EAGLE design)
At the start: 69.8 x 69.8 mm, 26 parts

Commit message: updates
Parts:
- added CPRG: 100nF, rcl:C1206
- added RPRG1: 10k, resistor:R1206
- added RPRG2: 330E, resistor:R1206
- added U1: MAX31723MUA+T, MAX31723MUA_T (1):SOP65P490X110-8N
- RRST2: value 330 -> 330E
- moved GND_NRST 10.2 mm to (6.99, 29.8)
- moved PAD_PRG 10.2 mm to (6.99, 40.0)
Connections:
- new net MISO: JP2.2, U1.5
- new net MOSI: JP2.3, U1.6
- new net PRG: PAD_PRG.1, RPRG2.2
- new net SCK: JP2.4, U1.3
- net +3V3: now also RPRG1.2, U1.2, U1.7, U1.8
- net D10: now also CPRG.1, RPRG1.1, RPRG2.1; no longer PAD_PRG.1
- net GND: now also CPRG.2, U1.4
Routing:
- net +3V3: track 7.70 -> 28.8 mm
- net PRG: track 0.00 -> 17.0 mm
- net D10: track 28.0 -> 40.8 mm, vias 0 -> 2
Changed lines of the file:
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@@
 <drawing>
 <settings>
-<setting alwaysvectorfont="no"/>
+<setting alwaysvectorfont="yes"/>
 <setting verticaltext="up"/>
 </settings>
@@
 <attribute name="VALUE" x="56.515" y="31.115" size="1.27" layer="27" rot="R180"/>
 </element>
-<element name="PAD_PRG" library="wirepad" library_urn="urn:adsk.eagle:library:412" package="SMD2,54-5,08" package3d_urn="urn:adsk.eagle:package:30841/1" value="0" x="6.985" y="29.845" smashed="yes">
+<element name="PAD_PRG" library="wirepad" library_urn="urn:adsk.eagle:library:412" package="SMD2,54-5,08" package3d_urn="urn:adsk.eagle:package:30841/1" value="0" x="6.985" y="40.005" smashed="yes">
+<attribute name="VALUE" x="6.985" y="40.005" size="0.0254" layer="27"/>
+</element>
+<element name="GND_NRST" library="wirepad" library_urn="urn:adsk.eagle:library:412" package="SMD2,54-5,08" package3d_urn="urn:adsk.eagle:package:30841/1" value="0" x="6.985" y="29.845" smashed="yes">
+<attribute name="NAME" x="5.485" y="27.345" size="1.016" layer="25" rot="R90" display="off"/>
 <attribute name="VALUE" x="6.985" y="29.845" size="0.0254" layer="27"/>
-</element>
-<element name="GND_NRST" library="wirepad" library_urn="urn:adsk.eagle:library:412" package="SMD2,54-5,08" package3d_urn="urn:adsk.eagle:package:30841/1" value="0" x="6.985" y="40.005" smashed="yes">
-<attribute name="NAME" x="5.485" y="37.505" size="1.016" layer="25" rot="R90" display="off"/>
-<attribute name="VALUE" x="6.985" y="40.005" size="0.0254" layer="27"/>
 </element>
 <element name="LED1" library="led" library_urn="urn:adsk.eagle:library:259" package="P47F-BOTTOM" package3d_urn="urn:adsk.eagle:package:15878/1" value="LWP4-BOTTOM" x="52.07" y="52.705" smashed="yes" rot="R90">
@@
 <attribute name="VALUE" x="53.34" y="58.55" size="1.27" layer="27" rot="R270"/>
 </element>
-<element name="RRST2" library="resistor" library_urn="urn:adsk.eagle:library:348" package="R1206" package3d_urn="urn:adsk.eagle:package:26062/1" value="330" x="59.69" y="57.15" smashed="yes" rot="R270">
+<element name="RRST2" library="resistor" library_urn="urn:adsk.eagle:library:348" package="R1206" package3d_urn="urn:adsk.eagle:package:26062/1" value="330E" x="59.69" y="57.15" smashed="yes" rot="R270">
 <attribute name="NAME" x="60.96" y="59.944" size="1.27" layer="25" rot="R270"/>
 <attribute name="VALUE" x="57.15" y="58.42" size="1.27" layer="27" rot="R270"/>
+</element>
+<element name="RPRG1" library="resistor" library_urn="urn:adsk.eagle:library:348" package="R1206" package3d_urn="urn:adsk.eagle:package:26062/1" value="10k" x="21.59" y="57.15" smashed="yes" rot="R90">
+<attribute name="NAME" x="24.13" y="54.229" size="1.27" layer="25" rot="R90"/>
+<attribute name="VALUE" x="24.13" y="55.88" size="1.27" layer="27" rot="R90"/>
+</element>
+<element name="CPRG" library="rcl" library_urn="urn:adsk.eagle:library:334" package="C1206" package3d_urn="urn:adsk.eagle:package:23618/2" value="100nF" x="13.97" y="57.15" smashed="yes" rot="R270">
+<attribute name="NAME" x="11.43" y="59.69" size="1.27" layer="25" rot="R270"/>
+<attribute name="SPICEPREFIX" value="C" x="13.97" y="57.15" size="1.778" layer="27" rot="R270" display="off"/>
+<attribute name="VALUE" x="11.43" y="58.42" size="1.27" layer="27" rot="R270"/>
+</element>
+<element name="RPRG2" library="resistor" library_urn="urn:adsk.eagle:library:348" package="R1206" package3d_urn="urn:adsk.eagle:package:26062/1" value="330E" x="10.16" y="57.15" smashed="yes" rot="R270">
+<attribute name="NAME" x="7.493" y="60.198" size="1.27" layer="25" rot="R270"/>
+<attribute name="VALUE" x="7.62" y="58.42" size="1.27" layer="27" rot="R270"/>
+</element>
+<element name="U1" library="MAX31723MUA_T (1)" package="SOP65P490X110-8N" value="MAX31723MUA+T" x="45.72" y="16.51" rot="R180">
+<attribute name="AVAILABILITY" value="Unavailable" x="45.72" y="16.51" size="1.778" layer="27" rot="R180" display="off"/>
+<attribute name="DESCRIPTION" value=" Thermostat Â±2Â°C Digital SMD 8-Pin uMAX T/R " x="45.72" y="16.51" size="1.778" layer="27" rot="R180" display="off"/>
+<attribute name="MF" value="Maxim Integrated" x="45.72" y="16.51" size="1.778" layer="27" rot="R180" display="off"/>
+<attribute name="MP" value="MAX31723MUA+T" x="45.72" y="16.51" size="1.778" layer="27" rot="R180" display="off"/>
+<attribute name="PACKAGE" value="MSOP-8 Maxim Integrated" x="45.72" y="16.51" size="1.778" layer="27" rot="R180" display="off"/>
+<attribute name="PRICE" value="None" x="45.72" y="16.51" size="1.778" layer="27" rot="R180" display="off"/>
 </element>
 </elements>
@@
 <wire x1="25.785" y1="54.61" x2="38.1" y2="54.61" width="0.3048" layer="1"/>
 <contactref element="CRST" pad="2"/>
+<contactref element="CPRG" pad="2"/>
+<contactref element="U1" pad="4"/>
+<wire x1="52.07" y1="14.695" x2="47.8536" y2="17.4752" width="0" layer="19" extent="1-1"/>
 </signal>
 <signal name="+3V3">
 <contactref element="JP2" pad="13"/>
 <contactref element="RRST1" pad="2"/>
-<wire x1="41.025" y1="54.61" x2="47.142" y2="54.61" width="0.1524" layer="1"/>
-<wire x1="47.142" y1="54.61" x2="48.26" y2="55.728" width="0.1524" layer="1"/>
+<contactref element="RPRG1" pad="2"/>
+<wire x1="41.025" y1="54.61" x2="37.063" y2="58.572" width="0.3048" layer="1"/>
+<wire x1="37.063" y1="58.572" x2="21.59" y2="58.572" width="0.3048" layer="1"/>
+<wire x1="41.025" y1="54.61" x2="47.142" y2="54.61" width="0.3048" layer="1"/>
+<wire x1="47.142" y1="54.61" x2="48.26" y2="55.728" width="0.3048" layer="1"/>
+<contactref element="U1" pad="2"/>
+<contactref element="U1" pad="8"/>
+<contactref element="U1" pad="7"/>
+<wire x1="47.8536" y1="16.1798" x2="47.142" y2="54.61" width="0" layer="19" extent="1-1"/>
+<wire x1="43.5864" y1="16.1798" x2="47.8536" y2="16.1798" width="0" layer="19" extent="1-1"/>
+<wire x1="43.5864" y1="15.5448" x2="43.5864" y2="16.1798" width="0" layer="19" extent="1-1"/>
 </signal>
 <signal name="SENS_PROX_1">
@@
 <signal name="D10">
 <contactref element="JP1" pad="8"/>
-<contactref element="PAD_PRG" pad="1"/>
-<wire x1="28.825" y1="41.91" x2="27.555" y2="40.64" width="0.1524" layer="1"/>
-<wire x1="27.555" y1="40.64" x2="24.638" y2="40.64" width="0.1524" layer="1"/>
-<wire x1="24.638" y1="40.64" x2="23.876" y2="39.878" width="0.1524" layer="1"/>
-<wire x1="23.876" y1="39.878" x2="23.876" y2="37.973" width="0.1524" layer="1"/>
-<wire x1="23.876" y1="37.973" x2="15.748" y2="29.845" width="0.1524" layer="1"/>
-<wire x1="15.748" y1="29.845" x2="6.985" y2="29.845" width="0.1524" layer="1"/>
+<contactref element="RPRG1" pad="1"/>
+<contactref element="CPRG" pad="1"/>
+<contactref element="RPRG2" pad="1"/>
+<wire x1="13.97" y1="58.55" x2="10.182" y2="58.55" width="0.1524" layer="1"/>
+<wire x1="10.182" y1="58.55" x2="10.16" y2="58.572" width="0.1524" layer="1"/>
+<wire x1="13.97" y1="58.55" x2="18.768" y2="58.55" width="0.1524" layer="1"/>
+<wire x1="18.768" y1="58.55" x2="21.514" y2="55.804" width="0.1524" layer="1"/>
+<wire x1="21.565" y1="55.753" x2="21.59" y2="55.728" width="0.1524" layer="1"/>
+<wire x1="28.825" y1="41.91" x2="32.385" y2="41.91" width="0.1524" layer="1"/>
+<via x="32.385" y="41.91" extent="1-16" drill="0.35"/>
+<wire x1="32.385" y1="41.91" x2="32.385" y2="55.753" width="0.1524" layer="16"/>
+<via x="32.385" y="55.753" extent="1-16" drill="0.35"/>
+<wire x1="32.385" y1="55.753" x2="21.565" y2="55.753" width="0.1524" layer="1"/>
+<wire x1="21.565" y1="55.753" x2="21.514" y2="55.804" width="0.1524" layer="1"/>
 </signal>
 <signal name="D9">
@@
 <wire x1="46.838" y1="57.15" x2="48.26" y2="58.572" width="0.1524" layer="1"/>
 </signal>
+<signal name="PRG">
+<contactref element="RPRG2" pad="2"/>
+<contactref element="PAD_PRG" pad="1"/>
+<wire x1="6.985" y1="40.005" x2="6.985" y2="52.553" width="0.1524" layer="1"/>
+<wire x1="6.985" y1="52.553" x2="10.16" y2="55.728" width="0.1524" layer="1"/>
+</signal>
+<signal name="MOSI">
+<contactref element="U1" pad="6"/>
+<contactref element="JP2" pad="3"/>
+<wire x1="43.5864" y1="16.8402" x2="41.025" y2="29.21" width="0" layer="19" extent="1-1"/>
+</signal>
+<signal name="MISO">
+<contactref element="U1" pad="5"/>
+<contactref element="JP2" pad="2"/>
+<wire x1="43.5864" y1="17.4752" x2="44.065" y2="26.67" width="0" layer="19" extent="1-1"/>
+</signal>
+<signal name="SCK">
+<contactref element="JP2" pad="4"/>
+<contactref element="U1" pad="3"/>
+<wire x1="47.8536" y1="16.8402" x2="44.065" y2="31.75" width="0" layer="19" extent="1-1"/>
+</signal>
 </signals>

Commit message: updates
Routing:
- net +3V3: track 28.8 -> 82.4 mm, vias 0 -> 2
- net SCK: track 0.00 -> 17.3 mm
- net GND: track 27.6 -> 42.4 mm, vias 2 -> 4
- net MOSI: track 0.00 -> 14.2 mm
- net MISO: track 0.00 -> 9.41 mm
- net D10: track 40.8 -> 34.0 mm, vias 2 -> 0
- net D11: track 38.7 -> 42.3 mm
- net USART1_RX: track 20.6 -> 17.7 mm, vias 2 -> 0
- net USART1_TX: track 20.9 -> 18.6 mm, vias 2 -> 0
- net A3: track 24.8 -> 24.3 mm

Commit message: updates
Parts:
- removed U1: MAX31723MUA+T, MAX31723MUA_T (1):SOP65P490X110-8N
Connections:
- net +3V3: no longer U1.2, U1.7, U1.8
- net GND: no longer U1.4
- net MISO: no longer U1.5
- net MOSI: no longer U1.6
- net SCK: no longer U1.3
Routing:
- net +3V3: track 82.4 -> 28.8 mm, vias 2 -> 0
- net SCK: track 17.3 -> 0.00 mm
- net MOSI: track 14.2 -> 0.00 mm
- net MISO: track 9.41 -> 0.00 mm
- net GND: track 42.4 -> 35.8 mm
Changed lines of the file:
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@@
 <drawing>
 <settings>
-<setting alwaysvectorfont="yes"/>
+<setting alwaysvectorfont="no"/>
 <setting verticaltext="up"/>
 </settings>
@@
 <attribute name="VALUE" x="7.62" y="58.42" size="1.27" layer="27" rot="R270"/>
 </element>
-<element name="U1" library="MAX31723MUA_T (1)" package="SOP65P490X110-8N" value="MAX31723MUA+T" x="45.72" y="16.51" rot="R180">
-<attribute name="AVAILABILITY" value="Unavailable" x="45.72" y="16.51" size="1.778" layer="27" rot="R180" display="off"/>
-<attribute name="DESCRIPTION" value=" Thermostat Â±2Â°C Digital SMD 8-Pin uMAX T/R " x="45.72" y="16.51" size="1.778" layer="27" rot="R180" display="off"/>
-<attribute name="MF" value="Maxim Integrated" x="45.72" y="16.51" size="1.778" layer="27" rot="R180" display="off"/>
-<attribute name="MP" value="MAX31723MUA+T" x="45.72" y="16.51" size="1.778" layer="27" rot="R180" display="off"/>
-<attribute name="PACKAGE" value="MSOP-8 Maxim Integrated" x="45.72" y="16.51" size="1.778" layer="27" rot="R180" display="off"/>
-<attribute name="PRICE" value="None" x="45.72" y="16.51" size="1.778" layer="27" rot="R180" display="off"/>
-</element>
 </elements>
 <signals>
@@
 <contactref element="CRST" pad="2"/>
 <contactref element="CPRG" pad="2"/>
-<contactref element="U1" pad="4"/>
-<wire x1="47.8536" y1="17.4752" x2="49.1998" y2="17.4752" width="0.3048" layer="1"/>
-<wire x1="49.1998" y1="17.4752" x2="49.403" y2="17.272" width="0.3048" layer="1"/>
-<wire x1="49.403" y1="17.272" x2="49.403" y2="15.24" width="0.3048" layer="1"/>
-<wire x1="49.948" y1="14.695" x2="52.07" y2="14.695" width="0.3048" layer="1"/>
-<wire x1="49.403" y1="15.24" x2="49.948" y2="14.695" width="0.3048" layer="1"/>
 <wire x1="38.1" y1="54.61" x2="36.83" y2="55.88" width="0.3048" layer="1"/>
 <wire x1="36.83" y1="55.88" x2="36.83" y2="57.15" width="0.3048" layer="1"/>
@@
 <contactref element="RPRG1" pad="2"/>
 <wire x1="41.025" y1="54.61" x2="37.063" y2="58.572" width="0.3048" layer="1"/>
-<wire x1="37.063" y1="58.572" x2="35.56" y2="58.572" width="0.3048" layer="1"/>
-<wire x1="35.56" y1="58.572" x2="21.59" y2="58.572" width="0.3048" layer="1"/>
+<wire x1="37.063" y1="58.572" x2="21.59" y2="58.572" width="0.3048" layer="1"/>
 <wire x1="41.025" y1="54.61" x2="47.142" y2="54.61" width="0.3048" layer="1"/>
 <wire x1="47.142" y1="54.61" x2="48.26" y2="55.728" width="0.3048" layer="1"/>
-<contactref element="U1" pad="2"/>
-<contactref element="U1" pad="8"/>
-<contactref element="U1" pad="7"/>
-<wire x1="43.5864" y1="15.5448" x2="43.5864" y2="16.1798" width="0.3048" layer="1"/>
-<wire x1="43.5864" y1="16.1798" x2="47.8536" y2="16.1798" width="0.3048" layer="1"/>
-<wire x1="35.56" y1="58.572" x2="35.56" y2="56.007" width="0.3048" layer="1"/>
-<via x="35.56" y="56.007" extent="1-16" drill="0.35"/>
-<wire x1="35.56" y1="56.007" x2="35.56" y2="46.99" width="0.3048" layer="16"/>
-<wire x1="35.56" y1="46.99" x2="34.417" y2="45.847" width="0.3048" layer="16"/>
-<via x="37.846" y="21.971" extent="1-16" drill="0.35"/>
-<wire x1="37.846" y1="21.971" x2="38.481" y2="21.336" width="0.3048" layer="1"/>
-<wire x1="38.481" y1="21.336" x2="40.64" y2="21.336" width="0.3048" layer="1"/>
-<wire x1="40.64" y1="21.336" x2="41.529" y2="20.447" width="0.3048" layer="1"/>
-<wire x1="42.2402" y1="16.1798" x2="43.5864" y2="16.1798" width="0.3048" layer="1"/>
-<wire x1="41.529" y1="20.447" x2="41.529" y2="16.891" width="0.3048" layer="1"/>
-<wire x1="41.529" y1="16.891" x2="42.2402" y2="16.1798" width="0.3048" layer="1"/>
-<wire x1="34.417" y1="25.4" x2="37.846" y2="21.971" width="0.3048" layer="16"/>
-<wire x1="34.417" y1="45.847" x2="34.417" y2="25.4" width="0.3048" layer="16"/>
 </signal>
 <signal name="SENS_PROX_1">
@@
 </signal>
 <signal name="MOSI">
-<contactref element="U1" pad="6"/>
 <contactref element="JP2" pad="3"/>
-<wire x1="41.025" y1="29.21" x2="41.025" y2="26.92" width="0.1524" layer="1"/>
-<wire x1="41.025" y1="26.92" x2="42.926" y2="25.019" width="0.1524" layer="1"/>
-<wire x1="42.926" y1="25.019" x2="42.926" y2="19.304" width="0.1524" layer="1"/>
-<wire x1="42.926" y1="19.304" x2="42.545" y2="18.923" width="0.1524" layer="1"/>
-<wire x1="42.545" y1="18.923" x2="42.545" y2="17.145" width="0.1524" layer="1"/>
-<wire x1="42.8498" y1="16.8402" x2="43.5864" y2="16.8402" width="0.1524" layer="1"/>
-<wire x1="42.545" y1="17.145" x2="42.8498" y2="16.8402" width="0.1524" layer="1"/>
 </signal>
 <signal name="MISO">
-<contactref element="U1" pad="5"/>
 <contactref element="JP2" pad="2"/>
-<wire x1="44.065" y1="26.67" x2="44.065" y2="19.173" width="0.1524" layer="1"/>
-<wire x1="44.065" y1="19.173" x2="43.561" y2="18.669" width="0.1524" layer="1"/>
-<wire x1="43.561" y1="18.669" x2="43.561" y2="17.5006" width="0.1524" layer="1"/>
-<wire x1="43.561" y1="17.5006" x2="43.5864" y2="17.4752" width="0.1524" layer="1"/>
 </signal>
 <signal name="SCK">
 <contactref element="JP2" pad="4"/>
-<contactref element="U1" pad="3"/>
-<wire x1="44.065" y1="31.75" x2="45.72" y2="30.095" width="0.1524" layer="1"/>
-<wire x1="45.72" y1="30.095" x2="45.72" y2="17.526" width="0.1524" layer="1"/>
-<wire x1="45.72" y1="17.526" x2="46.355" y2="16.891" width="0.1524" layer="1"/>
-<wire x1="46.355" y1="16.891" x2="47.8028" y2="16.891" width="0.1524" layer="1"/>
-<wire x1="47.8028" y1="16.891" x2="47.8536" y2="16.8402" width="0.1524" layer="1"/>
 </signal>
 </signals>
