File: eagle/1ButtonSwitch.ItsyBitsyM0.Rev1.0.brd (EAGLE design)
At the start: 69.8 x 69.8 mm, 30 parts, among them U1 MAX31723MUA+T

Commit message: updates
Parts:
- removed LED2, LED3, LED4: LWP4-BOTTOM, led:P47F-BOTTOM
- removed RL2, RL3, RL4: 330E, resistor:R1206
- removed RS2, RS3, RS4: 1k, resistor:R1206
- moved LED1 24.7 mm to (34.9, 34.9), turned to 270 degrees
- moved RL1 15.5 mm to (34.9, 41.9), turned to 270 degrees
Connections:
- removed net N$20: LED2.A, RL2.2
- removed net N$21: LED3.A, RL3.2
- removed net N$22: LED4.A, RL4.2
- removed net SENS_2: RS2.1
- removed net SENS_3: RS3.1
- removed net SENS_4: RS4.1
- net A0: no longer RS2.2
- net A3: no longer RS4.2
- net A5: no longer RS3.2
- net D11: no longer RL3.1
- net D13: no longer RL2.1
- net D9: no longer RL4.1
- net GND: no longer LED2.C, LED3.C, LED4.C
Routing:
- net D11: track 41.5 -> 0.00 mm, vias 2 -> 0
- net A0: track 25.0 -> 0.00 mm
- net A3: track 24.8 -> 0.00 mm
- net D9: track 19.4 -> 0.00 mm
- net GND: track 34.1 -> 20.8 mm, vias 2 -> 8
- net D12: track 20.3 -> 8.64 mm
- net A5: track 10.8 -> 0.00 mm
- net +3V3: track 82.4 -> 74.4 mm
- net D10: track 40.8 -> 32.9 mm, vias 2 -> 0
- net SHIELD_OR_GND: track 0.00 -> 7.51 mm, vias 1 -> 2
- net D13: track 5.99 -> 0.00 mm
- net SENS_3: track 4.14 -> 0.00 mm, vias 2 -> 1
- net SENS_4: track 4.14 -> 0.00 mm, vias 2 -> 1
- net SENS_2: track 4.01 -> 0.00 mm, vias 2 -> 1
- net N$21: track 3.73 -> 0.00 mm
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- removed copper zone on layer 16, net SENS_2
- removed copper zone on layer 16, net SENS_3
- removed copper zone on layer 16, net SENS_4
