File: eagle/1ButtonSwitch.ItsyBitsyM0.Rev1.0.brd (EAGLE design)
At the start: 69.8 x 69.8 mm, 21 parts, among them U1 MAX31723MUA+T

Commit message: updates
Parts:
- removed U1: MAX31723MUA+T, MAX31723MUA_T (1):SOP65P490X110-8N
Connections:
- net +3V3: no longer U1.2, U1.7, U1.8
- net GND: no longer U1.4
- net MISO: no longer U1.5
- net MOSI: no longer U1.6
- net SCK: no longer U1.3
Routing:
- net +3V3: track 74.4 -> 28.8 mm, vias 2 -> 0
- net SCK: track 17.3 -> 0.00 mm
- net MOSI: track 14.2 -> 0.00 mm
- net MISO: track 9.41 -> 0.00 mm
- net GND: track 20.8 -> 13.6 mm, vias 8 -> 6
Changed lines of the file:
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@@
 <attribute name="VALUE" x="7.62" y="58.42" size="1.27" layer="27" rot="R270"/>
-</element>
-<element name="U1" library="MAX31723MUA_T (1)" package="SOP65P490X110-8N" value="MAX31723MUA+T" x="45.72" y="16.51" rot="R180">
-<attribute name="AVAILABILITY" value="Unavailable" x="45.72" y="16.51" size="1.778" layer="27" rot="R180" display="off"/>
-<attribute name="DESCRIPTION" value=" Thermostat Â±2Â°C Digital SMD 8-Pin uMAX T/R " x="45.72" y="16.51" size="1.778" layer="27" rot="R180" display="off"/>
-<attribute name="MF" value="Maxim Integrated" x="45.72" y="16.51" size="1.778" layer="27" rot="R180" display="off"/>
-<attribute name="MP" value="MAX31723MUA+T" x="45.72" y="16.51" size="1.778" layer="27" rot="R180" display="off"/>
-<attribute name="PACKAGE" value="MSOP-8 Maxim Integrated" x="45.72" y="16.51" size="1.778" layer="27" rot="R180" display="off"/>
-<attribute name="PRICE" value="None" x="45.72" y="16.51" size="1.778" layer="27" rot="R180" display="off"/>
 </element>
 </elements>
@@
 <contactref element="CRST" pad="2"/>
 <contactref element="CPRG" pad="2"/>
-<contactref element="U1" pad="4"/>
 <wire x1="25.785" y1="54.61" x2="24.13" y2="54.61" width="0.3048" layer="1"/>
 <wire x1="24.13" y1="54.61" x2="22.86" y2="53.34" width="0.3048" layer="1"/>
@@
 <wire x1="52.07" y1="57.15" x2="52.07" y2="60.452" width="0.3048" layer="16"/>
 <via x="52.07" y="60.452" extent="1-16" drill="0.35"/>
-<wire x1="47.8536" y1="17.4752" x2="47.8536" y2="18.8976" width="0.3048" layer="1"/>
-<wire x1="47.8536" y1="18.8976" x2="47.879" y2="18.923" width="0.3048" layer="1"/>
-<via x="47.879" y="18.923" extent="1-16" drill="0.35"/>
-<wire x1="47.879" y1="18.923" x2="52.705" y2="18.923" width="0.3048" layer="16"/>
-<wire x1="52.705" y1="18.923" x2="53.34" y2="19.558" width="0.3048" layer="16"/>
-<via x="53.34" y="19.558" extent="1-16" drill="0.35"/>
 </signal>
 <signal name="+3V3">
@@
 <wire x1="41.025" y1="54.61" x2="47.142" y2="54.61" width="0.3048" layer="1"/>
 <wire x1="47.142" y1="54.61" x2="48.26" y2="55.728" width="0.3048" layer="1"/>
-<contactref element="U1" pad="2"/>
-<contactref element="U1" pad="8"/>
-<contactref element="U1" pad="7"/>
-<wire x1="43.5864" y1="15.5448" x2="43.5864" y2="16.1798" width="0.3048" layer="1"/>
-<wire x1="43.5864" y1="16.1798" x2="47.8536" y2="16.1798" width="0.3048" layer="1"/>
 <wire x1="21.59" y1="58.572" x2="31.598" y2="58.572" width="0.3048" layer="1"/>
 <wire x1="31.598" y1="58.572" x2="35.56" y2="54.61" width="0.3048" layer="1"/>
 <wire x1="35.56" y1="54.61" x2="41.025" y2="54.61" width="0.3048" layer="1"/>
-<wire x1="47.142" y1="54.61" x2="47.142" y2="44.475" width="0.3048" layer="1"/>
-<wire x1="47.142" y1="44.475" x2="47.117" y2="44.45" width="0.3048" layer="1"/>
-<via x="47.117" y="44.45" extent="1-16" drill="0.35"/>
-<wire x1="47.117" y1="44.45" x2="47.117" y2="25.273" width="0.3048" layer="16"/>
-<via x="47.117" y="25.273" extent="1-16" drill="0.35"/>
-<wire x1="47.117" y1="25.273" x2="47.117" y2="21.844" width="0.3048" layer="1"/>
-<wire x1="47.117" y1="21.844" x2="49.403" y2="19.558" width="0.3048" layer="1"/>
-<wire x1="49.403" y1="16.51" x2="49.0728" y2="16.1798" width="0.3048" layer="1"/>
-<wire x1="49.0728" y1="16.1798" x2="47.8536" y2="16.1798" width="0.3048" layer="1"/>
-<wire x1="49.403" y1="19.558" x2="49.403" y2="16.51" width="0.3048" layer="1"/>
 </signal>
 <signal name="SENS_PROX_1">
@@
 </signal>
 <signal name="MOSI">
-<contactref element="U1" pad="6"/>
 <contactref element="JP2" pad="3"/>
-<wire x1="41.025" y1="29.21" x2="41.025" y2="26.92" width="0.1524" layer="1"/>
-<wire x1="41.025" y1="26.92" x2="42.926" y2="25.019" width="0.1524" layer="1"/>
-<wire x1="42.926" y1="25.019" x2="42.926" y2="19.304" width="0.1524" layer="1"/>
-<wire x1="42.926" y1="19.304" x2="42.545" y2="18.923" width="0.1524" layer="1"/>
-<wire x1="42.545" y1="18.923" x2="42.545" y2="17.145" width="0.1524" layer="1"/>
-<wire x1="42.8498" y1="16.8402" x2="43.5864" y2="16.8402" width="0.1524" layer="1"/>
-<wire x1="42.545" y1="17.145" x2="42.8498" y2="16.8402" width="0.1524" layer="1"/>
 </signal>
 <signal name="MISO">
-<contactref element="U1" pad="5"/>
 <contactref element="JP2" pad="2"/>
-<wire x1="44.065" y1="26.67" x2="44.065" y2="19.173" width="0.1524" layer="1"/>
-<wire x1="44.065" y1="19.173" x2="43.561" y2="18.669" width="0.1524" layer="1"/>
-<wire x1="43.561" y1="18.669" x2="43.561" y2="17.5006" width="0.1524" layer="1"/>
-<wire x1="43.561" y1="17.5006" x2="43.5864" y2="17.4752" width="0.1524" layer="1"/>
 </signal>
 <signal name="SCK">
 <contactref element="JP2" pad="4"/>
-<contactref element="U1" pad="3"/>
-<wire x1="44.065" y1="31.75" x2="45.72" y2="30.095" width="0.1524" layer="1"/>
-<wire x1="45.72" y1="30.095" x2="45.72" y2="17.526" width="0.1524" layer="1"/>
-<wire x1="45.72" y1="17.526" x2="46.355" y2="16.891" width="0.1524" layer="1"/>
-<wire x1="46.355" y1="16.891" x2="47.8028" y2="16.891" width="0.1524" layer="1"/>
-<wire x1="47.8028" y1="16.891" x2="47.8536" y2="16.8402" width="0.1524" layer="1"/>
 </signal>
 </signals>
