File: eagle/5ButtonSwitch.ItsyBitsyM0.Rev1.0.sch (EAGLE design)
At the start: 25 parts, among them U1 MAX31723MUA+T

Commit message: updates
Parts:
- removed GND_NRST, GND_PRG, PAD_NRST: 0, wirepad:SMD5
- removed RSP1, RSP2: 1k, resistor:R-EU_R1206
- added +3V3, GND, PAD_GND1, PAD_GND2, PAD_RST, SCL, SDA: WIREPADSMD1,27-254, wirepad:WIREPADSMD1,27-254
- added RI2C1, RI2C2: 10k, resistor:R-EU_R1206
- PAD_PRG: value 0 -> WIREPADSMD1,27-254; device wirepad:SMD5 -> wirepad:WIREPADSMD1,27-254
- renumbered JP2 to ITSYBITSYM0
Connections:
- removed net SENS_PROX_1: RSP1.1
- removed net SENS_PROX_2: RSP2.1
- new net SENSPAD_1: RS1.1
- new net SENSPAD_2: RS2.1
- new net SENSPAD_3: RS3.1
- new net SENSPAD_4: RS4.1
- new net SENSPAD_MAIN: RSM.1
- net +3V3: now also +3V3.P, RI2C1.2, RI2C2.2
- net A1: now also RS1.2
- net A2: now also RSM.2
- net A3: now also RS2.2
- net A4: now also RS3.2
- net A5: now also RS4.2
- net D11: now also RR.1
- net D12: now also RG.1
- net D13: now also RB.1
- net GND: now also GND.P, PAD_GND1.P, PAD_GND2.P; no longer GND_NRST.P, GND_PRG.P, RB.1, RG.1, RR.1
- net RESET: now also PAD_RST.P; no longer PAD_NRST.P
- net SCL: now also RI2C2.1, SCL.P
- net SDA: now also RI2C1.1, SDA.P
Other:
- note added: "BCU PINHEADER https://www.digikey.com/product-detail/en/molex-llc/0015911282/0015911282-ND/3123842"
- note added: "LED: https://www.digikey.com/product-detail/en/qt-brightek-qtb/QBLP677R-RGB/1516-1282-1-ND/7567403"
- note added: "SI7021-A20 BME280 .. needs breakout 1528-2564-ND AM2320 KY-052 https://www.reichelt.at/entwicklerboards-temperatur-und-feuchtigkeitssensor-debo-temp-hum2-p235487.html?PROVID=2788&gclid=EAIaIQobChMI09qm7oXD4AIVQqMYCh3gOg6PEAkYAiABEgKSsPD_BwE&&r=1"
- note added: "SOUND: PAM8301"
- note removed: "LEDS: https://www.digikey.com/product-detail/en/wurth-electronics-inc/156125M173000/732-11426-1-ND/7316162 https://www.digikey.com/product-detail/en/qt-brightek-qtb/QBLP677R-RGB/1516-1282-1-ND/7567403"
- note removed: "https://www.digikey.com/product-detail/en/molex-llc/0015911282/0015911282-ND/3123842"

Commit message: updates
Parts:
- added LS1: CSS-0575B-SMT, CSS-0575B-SMT:CSS-0575B-SMT
- added RLS: 0, resistor:R-EU_R1206
Connections:
- new net N$4: LS1.P, RLS.1
- net A0: now also RLS.2
- net GND: now also LS1.N
Other:
- note added: "SOUND: PAM8301 CSS-0575B-SMT or speakers: https://www.reichelt.at/kleinlautsprecher-lsf-15m-s-0-5w-8ohm-lsf-15m-s-p145875.html?&trstct=lsbght_sldr::145881"
- note removed: "SOUND: PAM8301"
Changed lines of the file:
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@@
 <part name="PAD_GND1" library="wirepad" library_urn="urn:adsk.eagle:library:412" deviceset="WIREPAD" device="SMD1,27-254" package3d_urn="urn:adsk.eagle:package:30839/1"/>
 <part name="PAD_GND2" library="wirepad" library_urn="urn:adsk.eagle:library:412" deviceset="WIREPAD" device="SMD1,27-254" package3d_urn="urn:adsk.eagle:package:30839/1"/>
+<part name="LS1" library="CSS-0575B-SMT" deviceset="CSS-0575B-SMT" device=""/>
+<part name="RLS" library="resistor" library_urn="urn:adsk.eagle:library:348" deviceset="R-EU_" device="R1206" package3d_urn="urn:adsk.eagle:package:26062/1" value="0"/>
 </parts>
 <sheets>
@@
 KY-052
 https://www.reichelt.at/entwicklerboards-temperatur-und-feuchtigkeitssensor-debo-temp-hum2-p235487.html?PROVID=2788&amp;gclid=EAIaIQobChMI09qm7oXD4AIVQqMYCh3gOg6PEAkYAiABEgKSsPD_BwE&amp;&amp;r=1</text>
-<text x="88.9" y="-45.72" size="1.778" layer="91">SOUND: PAM8301</text>
+<text x="88.9" y="-45.72" size="1.778" layer="91">SOUND: PAM8301
+CSS-0575B-SMT
+or speakers:
+https://www.reichelt.at/kleinlautsprecher-lsf-15m-s-0-5w-8ohm-lsf-15m-s-p145875.html?&amp;trstct=lsbght_sldr::145881
+</text>
 </plain>
 <instances>
@@
 <instance part="PAD_GND1" gate="G$1" x="15.24" y="-12.7" rot="R270"/>
 <instance part="PAD_GND2" gate="G$1" x="30.48" y="-12.7" rot="R270"/>
+<instance part="LS1" gate="G$1" x="154.94" y="-88.9"/>
+<instance part="RLS" gate="G$1" x="139.7" y="-83.82" rot="R180"/>
 </instances>
 <busses>
@@
 <wire x1="7.62" y1="-88.9" x2="7.62" y2="-63.5" width="0.1524" layer="91"/>
 <label x="7.62" y="-63.5" size="1.27" layer="95" rot="R90" xref="yes"/>
+</segment>
+<segment>
+<pinref part="LS1" gate="G$1" pin="N"/>
+<wire x1="154.94" y1="-93.98" x2="129.54" y2="-93.98" width="0.1524" layer="91"/>
+<label x="129.54" y="-93.98" size="1.27" layer="95" rot="R180" xref="yes"/>
 </segment>
 </net>
@@
 <label x="101.6" y="48.26" size="1.27" layer="95" rot="R180" xref="yes"/>
 </segment>
+<segment>
+<pinref part="RLS" gate="G$1" pin="2"/>
+<label x="129.54" y="-83.82" size="1.27" layer="95" rot="R180" xref="yes"/>
+<wire x1="129.54" y1="-83.82" x2="134.62" y2="-83.82" width="0.1524" layer="91"/>
+</segment>
 </net>
 <net name="A1" class="0">
@@
 </segment>
 </net>
+<net name="N$4" class="0">
+<segment>
+<pinref part="LS1" gate="G$1" pin="P"/>
+<wire x1="154.94" y1="-83.82" x2="144.78" y2="-83.82" width="0.1524" layer="91"/>
+<pinref part="RLS" gate="G$1" pin="1"/>
+</segment>
+</net>

Commit message: updates
Parts:
- removed U1: MAX31723MUA+T, MAX31723MUA_T (1):MAX31723MUA+T
Connections:
- net +3V3: no longer U1.CE, U1.SERMODE, U1.VDD
- net GND: no longer U1.GND
- net MISO: no longer U1.SDO
- net MOSI: no longer U1.SDI
- net SCK: no longer U1.SCLK
Changed lines of the file:
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@@
 <part name="CPRG" library="rcl" library_urn="urn:adsk.eagle:library:334" deviceset="C-EU" device="C1206" package3d_urn="urn:adsk.eagle:package:23618/2" value="100nF"/>
 <part name="RPRG2" library="resistor" library_urn="urn:adsk.eagle:library:348" deviceset="R-EU_" device="R1206" package3d_urn="urn:adsk.eagle:package:26062/1" value="330E"/>
-<part name="U1" library="MAX31723MUA_T (1)" deviceset="MAX31723MUA+T" device=""/>
 <part name="RS3" library="resistor" library_urn="urn:adsk.eagle:library:348" deviceset="R-EU_" device="R1206" package3d_urn="urn:adsk.eagle:package:26062/1" value="1k"/>
 <part name="RS2" library="resistor" library_urn="urn:adsk.eagle:library:348" deviceset="R-EU_" device="R1206" package3d_urn="urn:adsk.eagle:package:26062/1" value="1k"/>
@@
 <instance part="CPRG" gate="G$1" x="203.2" y="-27.94"/>
 <instance part="RPRG2" gate="G$1" x="190.5" y="-22.86" rot="R180"/>
-<instance part="U1" gate="A" x="83.82" y="-78.74"/>
 <instance part="RS3" gate="G$1" x="96.52" y="-10.16" rot="R90"/>
 <instance part="RS2" gate="G$1" x="88.9" y="-10.16" rot="R90"/>
@@
 </segment>
 <segment>
-<pinref part="U1" gate="A" pin="GND"/>
-<wire x1="66.04" y1="-93.98" x2="55.88" y2="-93.98" width="0.1524" layer="91"/>
-<label x="55.88" y="-93.98" size="1.016" layer="95" rot="R180" xref="yes"/>
-</segment>
-<segment>
 <pinref part="GND" gate="G$1" pin="P"/>
 <wire x1="7.62" y1="-88.9" x2="7.62" y2="-63.5" width="0.1524" layer="91"/>
@@
 <wire x1="203.2" y1="-7.62" x2="203.2" y2="-2.54" width="0.1524" layer="91"/>
 <label x="203.2" y="-2.54" size="1.016" layer="95" rot="R90" xref="yes"/>
-</segment>
-<segment>
-<pinref part="U1" gate="A" pin="CE"/>
-<wire x1="66.04" y1="-81.28" x2="55.88" y2="-81.28" width="0.1524" layer="91"/>
-<pinref part="U1" gate="A" pin="VDD"/>
-<wire x1="66.04" y1="-71.12" x2="55.88" y2="-71.12" width="0.1524" layer="91"/>
-<wire x1="55.88" y1="-71.12" x2="55.88" y2="-81.28" width="0.1524" layer="91"/>
-<wire x1="55.88" y1="-71.12" x2="55.88" y2="-55.88" width="0.1524" layer="91"/>
-<junction x="55.88" y="-71.12"/>
-<pinref part="U1" gate="A" pin="SERMODE"/>
-<wire x1="55.88" y1="-81.28" x2="55.88" y2="-88.9" width="0.1524" layer="91"/>
-<wire x1="55.88" y1="-88.9" x2="66.04" y2="-88.9" width="0.1524" layer="91"/>
-<junction x="55.88" y="-81.28"/>
-<label x="55.88" y="-55.88" size="1.016" layer="95" rot="R90" xref="yes"/>
 </segment>
 <segment>
@@
 <net name="MOSI" class="0">
 <segment>
-<pinref part="U1" gate="A" pin="SDI"/>
-<wire x1="66.04" y1="-86.36" x2="48.26" y2="-86.36" width="0.1524" layer="91"/>
-<label x="48.26" y="-86.36" size="1.016" layer="95" rot="R180" xref="yes"/>
-</segment>
-<segment>
 <pinref part="ITSYBITSYM0" gate="A" pin="3"/>
 <wire x1="109.22" y1="66.04" x2="101.6" y2="66.04" width="0.1524" layer="91"/>
@@
 <net name="MISO" class="0">
 <segment>
-<pinref part="U1" gate="A" pin="SDO"/>
-<wire x1="101.6" y1="-71.12" x2="116.84" y2="-71.12" width="0.1524" layer="91"/>
-<label x="116.84" y="-71.12" size="1.016" layer="95" xref="yes"/>
-</segment>
-<segment>
 <pinref part="ITSYBITSYM0" gate="A" pin="2"/>
 <wire x1="109.22" y1="68.58" x2="101.6" y2="68.58" width="0.1524" layer="91"/>
@@
 <label x="101.6" y="63.5" size="1.016" layer="95" rot="R180" xref="yes"/>
 </segment>
-<segment>
-<pinref part="U1" gate="A" pin="SCLK"/>
-<wire x1="66.04" y1="-76.2" x2="48.26" y2="-76.2" width="0.1524" layer="91"/>
-<label x="48.26" y="-76.2" size="1.016" layer="95" rot="R180" xref="yes"/>
-</segment>
-</net>
+</net>
