File: eagle/1ButtonSwitch.ItsyBitsyM0.Rev1.0.sch (EAGLE design)
At the start: 28 parts, among them U1 MAX31723MUA+T

Commit message: updates
Parts:
- removed LED2, LED3, LED4: LWP4-BOTTOM, led:LWP4-BOTTOM
- removed RL2, RL3, RL4: 330E, resistor:R-EU_R1206
- removed RS2, RS3, RS4: 1k, resistor:R-EU_R1206
Connections:
- removed net N$20: LED2.A, RL2.2
- removed net N$21: LED3.A, RL3.2
- removed net N$22: LED4.A, RL4.2
- removed net SCLK: U1.SCLK
- removed net SDI: U1.SDI
- removed net SDO: U1.SDO
- removed net SENS_2: RS2.1
- removed net SENS_3: RS3.1
- removed net SENS_4: RS4.1
- new net MISO: JP2.2, U1.SDO
- new net MOSI: JP2.3, U1.SDI
- new net SCK: JP2.4, U1.SCLK
- net A0: no longer RS2.2
- net A3: no longer RS4.2
- net A5: no longer RS3.2
- net D11: no longer RL3.1
- net D13: no longer RL2.1
- net D9: no longer RL4.1
- net GND: no longer LED2.C, LED3.C, LED4.C
Other:
- note added: "LEDS Everlight 23-11/T7D-CQ2R2QY/2A"
- note removed: "LEDS OSRAM LW P473"

Commit message: updates
Parts:
- removed U1: MAX31723MUA+T, MAX31723MUA_T (1):MAX31723MUA+T
Connections:
- net +3V3: no longer U1.CE, U1.SERMODE, U1.VDD
- net GND: no longer U1.GND
- net MISO: no longer U1.SDO
- net MOSI: no longer U1.SDI
- net SCK: no longer U1.SCLK
Changed lines of the file:
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@@
 <part name="CPRG" library="rcl" library_urn="urn:adsk.eagle:library:334" deviceset="C-EU" device="C1206" package3d_urn="urn:adsk.eagle:package:23618/2" value="100nF"/>
 <part name="RPRG2" library="resistor" library_urn="urn:adsk.eagle:library:348" deviceset="R-EU_" device="R1206" package3d_urn="urn:adsk.eagle:package:26062/1" value="330E"/>
-<part name="U1" library="MAX31723MUA_T (1)" deviceset="MAX31723MUA+T" device=""/>
 </parts>
 <sheets>
@@
 <instance part="CPRG" gate="G$1" x="203.2" y="-27.94"/>
 <instance part="RPRG2" gate="G$1" x="190.5" y="-22.86" rot="R180"/>
-<instance part="U1" gate="A" x="83.82" y="-78.74"/>
 </instances>
 <busses>
@@
 <label x="203.2" y="-38.1" size="1.016" layer="95" rot="R270" xref="yes"/>
 </segment>
-<segment>
-<pinref part="U1" gate="A" pin="GND"/>
-<wire x1="66.04" y1="-93.98" x2="55.88" y2="-93.98" width="0.1524" layer="91"/>
-<label x="55.88" y="-93.98" size="1.016" layer="95" rot="R180" xref="yes"/>
-</segment>
 </net>
 <net name="+3V3" class="0">
@@
 <wire x1="203.2" y1="-7.62" x2="203.2" y2="-2.54" width="0.1524" layer="91"/>
 <label x="203.2" y="-2.54" size="1.016" layer="95" rot="R90" xref="yes"/>
-</segment>
-<segment>
-<pinref part="U1" gate="A" pin="CE"/>
-<wire x1="66.04" y1="-81.28" x2="55.88" y2="-81.28" width="0.1524" layer="91"/>
-<pinref part="U1" gate="A" pin="VDD"/>
-<wire x1="66.04" y1="-71.12" x2="55.88" y2="-71.12" width="0.1524" layer="91"/>
-<wire x1="55.88" y1="-71.12" x2="55.88" y2="-81.28" width="0.1524" layer="91"/>
-<wire x1="55.88" y1="-71.12" x2="55.88" y2="-55.88" width="0.1524" layer="91"/>
-<junction x="55.88" y="-71.12"/>
-<pinref part="U1" gate="A" pin="SERMODE"/>
-<wire x1="55.88" y1="-81.28" x2="55.88" y2="-88.9" width="0.1524" layer="91"/>
-<wire x1="55.88" y1="-88.9" x2="66.04" y2="-88.9" width="0.1524" layer="91"/>
-<junction x="55.88" y="-81.28"/>
-<label x="55.88" y="-55.88" size="1.016" layer="95" rot="R90" xref="yes"/>
 </segment>
 </net>
@@
 <net name="MOSI" class="0">
 <segment>
-<pinref part="U1" gate="A" pin="SDI"/>
-<wire x1="66.04" y1="-86.36" x2="48.26" y2="-86.36" width="0.1524" layer="91"/>
-<label x="48.26" y="-86.36" size="1.016" layer="95" rot="R180" xref="yes"/>
-</segment>
-<segment>
 <pinref part="JP2" gate="A" pin="3"/>
 <wire x1="109.22" y1="66.04" x2="101.6" y2="66.04" width="0.1524" layer="91"/>
@@
 <net name="MISO" class="0">
 <segment>
-<pinref part="U1" gate="A" pin="SDO"/>
-<wire x1="101.6" y1="-71.12" x2="116.84" y2="-71.12" width="0.1524" layer="91"/>
-<label x="116.84" y="-71.12" size="1.016" layer="95" xref="yes"/>
-</segment>
-<segment>
 <pinref part="JP2" gate="A" pin="2"/>
 <wire x1="109.22" y1="68.58" x2="101.6" y2="68.58" width="0.1524" layer="91"/>
@@
 <label x="101.6" y="63.5" size="1.016" layer="95" rot="R180" xref="yes"/>
 </segment>
-<segment>
-<pinref part="U1" gate="A" pin="SCLK"/>
-<wire x1="66.04" y1="-76.2" x2="48.26" y2="-76.2" width="0.1524" layer="91"/>
-<label x="48.26" y="-76.2" size="1.016" layer="95" rot="R180" xref="yes"/>
-</segment>
-</net>
+</net>
