File: eagle/5ButtonSwitch.ItsyBitsyM0.Rev1.0.brd (EAGLE design)
At the start: 69.8 x 69.8 mm, 21 parts, among them U1 MAX31723MUA+T

Commit message: updates
Parts:
- removed LED1: LWP4-BOTTOM, led:P47F-BOTTOM
- removed RL1: 330E, resistor:R1206
- removed RP1, RP2: 1k, resistor:R1206
- added RB, RG, RR: 330, resistor:R1206
- added RS2, RS3, RS4, RSM, RSP1, RSP2: 1k, resistor:R1206
- added U$4: QBLP677R-RGB-EX, ChriD_TouchSwitch:PLCC4R_EX
- moved GND_NRST 29.6 mm to (-14.6, 50.2)
- moved PAD_PRG 28.0 mm to (-14.6, 57.8)
- moved GND_PRG 27.9 mm to (83.2, 48.9)
- moved PAD_NRST 25.4 mm to (83.2, 55.2)
- moved U1 10.2 mm to (55.9, 15.2)
- moved RPRG2 5.24 mm to (15.2, 55.9)
- moved RRST2 5.24 mm to (54.6, 55.9)
- moved CRST 4.66 mm to (51.4, 55.9)
- moved CPRG 4.62 mm to (18.4, 55.9)
- moved RPRG1 1.27 mm to (21.6, 55.9)
- moved RRST1 1.27 mm to (48.3, 55.9)
- moved JP1 0.63 mm to (27.3, 40.0)
- moved JP2 0.63 mm to (42.5, 40.0)
- turned RS1 to 0 degrees
Connections:
- removed net N$19: LED1.A, RL1.2
- removed net SENS_1: RS1.1
- new net N$1: RB.2, U$4.1
- new net N$2: RG.2, U$4.2
- new net N$3: RR.2, U$4.3
- net +3V3: now also U$4.4
- net A1: no longer RS1.2
- net A2: no longer RP1.2
- net A4: no longer RP2.2
- net D12: no longer RL1.1
- net GND: now also RB.1, RG.1, RR.1; no longer LED1.C
- net SENS_PROX_1: now also RSP1.1; no longer RP1.1
- net SENS_PROX_2: now also RSP2.1; no longer RP2.1
Routing:
- net +3V3: track 74.4 -> 0.63 mm, vias 2 -> 0
- net +5V: track 60.3 -> 0.00 mm, vias 3 -> 1
- net D10: track 32.9 -> 0.00 mm
- net GND: track 20.8 -> 0.00 mm, vias 8 -> 2
- net USART1_TX: track 18.6 -> 0.00 mm
- net USART1_RX: track 17.7 -> 0.00 mm
- net SCK: track 17.3 -> 0.00 mm
- net RESET: track 17.0 -> 0.00 mm
- net PRG: track 17.0 -> 0.00 mm
- net RST: track 16.3 -> 0.00 mm
- net MOSI: track 14.2 -> 0.00 mm
- net A4: track 13.5 -> 0.00 mm
- net A2: track 13.5 -> 0.00 mm
- net SENS_PROX_2: track 125.4 -> 114.5 mm, vias 3 -> 0
- net SENS_PROX_1: track 125.4 -> 114.5 mm, vias 3 -> 0
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- added copper zone on layer 16, net SENSPAD_1
- added copper zone on layer 16, net SENSPAD_2
- added copper zone on layer 16, net SENSPAD_3
- added copper zone on layer 16, net SENSPAD_4
- added copper zone on layer 16, net SENSPAD_MAIN
- removed copper zone on layer 16, net SENS_1
- removed copper zone on layer 16, net SHIELD_OR_GND
Other:
- outline, holes or cut-outs redrawn
- board text added: "5xTouch Button | Itsy Bitsy M0 | Rev 1.0"
- board text added: "GND (max 20mA)"
- board text added: "SWCLK"
- board text added: "SWDIO"
- board text removed: "+"
- board text removed: "4xTouch Button | Itsy Bitsy M0 | Rev 1.1"
- board text removed: "PRG"
- board text removed: "RST"

Commit message: updates
Parts:
- removed GND_NRST, GND_PRG, PAD_NRST: 0, wirepad:SMD2,54-5,08
- removed RSP2: 1k, resistor:R1206
- removed U$1, U$2: (no value), holes:3,0
- added +3V3, GND, PAD_GND1, PAD_GND2, PAD_RST, SCL, SDA: WIREPADSMD1,27-254, wirepad:SMD1,27-2,54
- added RI2C1: 10k, resistor:R1206
- PAD_PRG: value 0 -> WIREPADSMD1,27-254; device wirepad:SMD2,54-5,08 -> wirepad:SMD1,27-2,54
- RI2C2: value 1k -> 10k
- moved PAD_PRG 35.2 mm to (18.4, 45.7), flipped to the bottom, turned to 90 degrees
- moved RB 24.1 mm to (34.9, 54.0), turned to 0 degrees
- moved RSM 17.4 mm to (49.5, 36.8), turned to 180 degrees
- moved RS2 14.6 mm to (34.9, 41.3)
- moved RS4 14.6 mm to (34.9, 28.6)
- moved RG 10.2 mm to (34.9, 50.2), turned to 0 degrees
- moved RS3 3.81 mm to (49.5, 33.0), turned to 180 degrees
- moved RR 3.17 mm to (34.9, 46.4), turned to 0 degrees
- moved RPRG2 2.54 mm to (12.7, 55.9)
- moved CPRG 2.54 mm to (15.9, 55.9)
- moved CRST 2.54 mm to (54.0, 55.9)
- moved RPRG1 2.54 mm to (19.1, 55.9)
- moved RRST1 2.54 mm to (50.8, 55.9)
- moved RRST2 2.54 mm to (57.1, 55.9)
- moved U1 2.01 mm to (54.0, 15.9)
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- renumbered JP2 to ITSYBITSYM0, RSP1 to RI2C2
Connections:
- removed net SENS_PROX_1: RI2C2.1
- removed net SENS_PROX_2: RSP2.1
- new net SENSPAD_1: RS1.1
- new net SENSPAD_2: RS2.1
- new net SENSPAD_3: RS3.1
- new net SENSPAD_4: RS4.1
- new net SENSPAD_MAIN: RSM.1
- net +3V3: now also +3V3.1, RI2C1.2, RI2C2.2
- net A1: now also RS1.2
- net A2: now also RSM.2
- net A3: now also RS2.2
- net A4: now also RS3.2
- net A5: now also RS4.2
- net D11: now also RR.1
- net D12: now also RG.1
- net D13: now also RB.1
- net GND: now also GND.1, PAD_GND1.1, PAD_GND2.1; no longer GND_NRST.1, GND_PRG.1, RB.1, RG.1, RR.1
- net RESET: now also PAD_RST.1; no longer PAD_NRST.1
- net SCL: now also RI2C2.1, SCL.1
- net SDA: now also RI2C1.1, SDA.1
Routing:
- net +3V3: track 0.63 -> 148.6 mm, vias 0 -> 1
- net +5V: track 0.00 -> 126.3 mm
- net SENS_PROX_2: track 114.5 -> 0.00 mm
- net SENS_PROX_1: track 114.5 -> 0.00 mm
- net GND: track 0.00 -> 41.7 mm, vias 2 -> 9
- net SENSPAD_4: track 0.00 -> 28.9 mm, vias 0 -> 1
- net D10: track 0.00 -> 27.4 mm
- net N$1: track 0.00 -> 27.3 mm
- net SENSPAD_2: track 0.00 -> 25.2 mm, vias 0 -> 1
- net SCL: track 0.00 -> 22.5 mm
- net SCK: track 0.00 -> 21.9 mm
- net USART1_TX: track 0.00 -> 19.0 mm
- net MOSI: track 0.00 -> 17.2 mm
- net N$2: track 0.00 -> 14.1 mm
- net USART1_RX: track 0.00 -> 13.9 mm
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- added copper zone on layer 16, net GND
Other:
- outline, holes or cut-outs redrawn
- board text added: "+3V3"
- board text added: "0XCDDC | 2019 by ChriD"
- board text added: "5xTouch Button | Konnekting | Rev 1.0"
- board text added: "BME/BMP280"
- board text added: "Breakout Board"
- board text added: "GND (SWD)"
- board text added: "I2C Pullup"
- board text added: "LED"
- board text added: "MAX31723"
- board text added: "PRG"
- board text added: "PRG BUTTON"
- board text added: "RESET BUTTON"
- board text added: "RGB LED"
- board text added: "RST"
- board text added: "Resistors"
- board text added: "SPEAKER"
- board text removed: "5xTouch Button | Itsy Bitsy M0 | Rev 1.0"
- board text removed: "GND (max 20mA)"
- board text removed: "Konnekting | 0XCDDC | 2019 by ChriD"
- board text removed: "SH"

Commit message: updates
Parts:
- added LS1: CSS-0575B-SMT, CSS-0575B-SMT:CUI_CSS-0575B-SMT
- added RLS: 0, resistor:R1206
Connections:
- new net N$4: LS1.1, RLS.1
- net A0: now also RLS.2
- net GND: now also LS1.2
Routing:
- net A0: track 0.00 -> 21.9 mm
- net GND: track 41.7 -> 57.4 mm
- net N$4: track 0.00 -> 4.59 mm
Changed lines of the file:
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@@
 <wire x1="59.69" y1="10.16" x2="48.26" y2="10.16" width="0.1524" layer="21"/>
 <wire x1="48.26" y1="13.208" x2="59.69" y2="13.208" width="0.1524" layer="25"/>
-<text x="50.419" y="11.43" size="1.016" layer="21">MAX31723</text>
-<wire x1="48.26" y1="29.845" x2="59.69" y2="29.845" width="0.1524" layer="21"/>
-<wire x1="48.26" y1="29.845" x2="48.26" y2="20.955" width="0.1524" layer="21"/>
+<text x="50.419" y="11.176" size="1.016" layer="21">MAX31723</text>
+<wire x1="46.99" y1="29.845" x2="59.69" y2="29.845" width="0.1524" layer="21"/>
+<wire x1="46.99" y1="29.845" x2="46.99" y2="20.955" width="0.1524" layer="21"/>
 <wire x1="59.69" y1="29.845" x2="59.69" y2="20.955" width="0.1524" layer="21"/>
-<wire x1="59.69" y1="20.955" x2="48.26" y2="20.955" width="0.1524" layer="21"/>
+<wire x1="59.69" y1="20.955" x2="46.99" y2="20.955" width="0.1524" layer="21"/>
 <wire x1="48.26" y1="23.368" x2="59.69" y2="23.368" width="0.1524" layer="25"/>
-<text x="51.054" y="21.463" size="1.016" layer="21">SPEAKER</text>
+<text x="51.054" y="21.59" size="1.016" layer="21">SPEAKER</text>
 <wire x1="31.75" y1="43.18" x2="38.1" y2="43.18" width="0.1524" layer="25"/>
 <wire x1="38.1" y1="43.18" x2="38.1" y2="55.88" width="0.1524" layer="25"/>
@@
 <attribute name="VALUE" x="51.435" y="48.26" size="0.0254" layer="28" rot="MR90"/>
 </element>
+<element name="LS1" library="CSS-0575B-SMT" package="CUI_CSS-0575B-SMT" value="CSS-0575B-SMT" x="55.245" y="26.67" smashed="yes">
+<attribute name="CUI_PURCHASE_URL" value="https://www.cui.com/product/audio/buzzers/audio-transducers/css-0575b-smt?utm_source=snapeda.com&amp;utm_medium=referral&amp;utm_campaign=snapedaBOM" x="55.245" y="26.67" size="1.778" layer="27" display="off"/>
+<attribute name="DESCRIPTION" value=" AUDIO MAGNETIC XDCR 2-4V SMD " x="55.245" y="26.67" size="1.778" layer="27" display="off"/>
+<attribute name="DIGI-KEY_PART_NUMBER" value="102-2202-1-ND" x="55.245" y="26.67" size="1.778" layer="27" display="off"/>
+<attribute name="DIGI-KEY_PURCHASE_URL" value="https://www.digikey.com/product-detail/en/cui-inc/CSS-0575B-SMT-TR/102-2202-1-ND/2364651?utm_source=snapeda&amp;utm_medium=aggregator&amp;utm_campaign=symbol" x="55.245" y="26.67" size="1.778" layer="27" display="off"/>
+<attribute name="MF" value="CUI Inc." x="55.245" y="26.67" size="1.778" layer="27" display="off"/>
+<attribute name="MP" value="CSS-0575B-SMT-TR" x="55.245" y="26.67" size="1.778" layer="27" display="off"/>
+<attribute name="PACKAGE" value=" CUI Inc." x="55.245" y="26.67" size="1.778" layer="27" display="off"/>
+<attribute name="VALUE" x="50.41291875" y="21.661509375" size="1.782090625" layer="27"/>
+</element>
+<element name="RLS" library="resistor" library_urn="urn:adsk.eagle:library:348" package="R1206" package3d_urn="urn:adsk.eagle:package:26062/1" value="0" x="48.895" y="26.67" smashed="yes" rot="R90">
+<attribute name="NAME" x="51.054" y="25.527" size="1.016" layer="25" rot="R90"/>
+<attribute name="VALUE" x="51.435" y="25.4" size="1.27" layer="27" rot="R90"/>
+</element>
 </elements>
 <signals>
@@
 <wire x1="40.132" y1="10.668" x2="40.894" y2="11.43" width="0.3048" layer="16"/>
 <wire x1="40.894" y1="11.43" x2="43.815" y2="11.43" width="0.3048" layer="16"/>
-<wire x1="56.1086" y1="16.8402" x2="56.896" y2="17.6276" width="0.3048" layer="1"/>
-<wire x1="56.896" y1="17.6276" x2="56.896" y2="17.78" width="0.3048" layer="1"/>
-<via x="56.896" y="17.78" extent="1-16" drill="0.35"/>
+<contactref element="LS1" pad="2"/>
+<wire x1="57.145" y1="24.92" x2="59.591" y2="24.92" width="0.3048" layer="1"/>
+<via x="59.817" y="30.353" extent="1-16" drill="0.35"/>
+<wire x1="60.373" y1="25.702" x2="60.373" y2="29.797" width="0.3048" layer="1"/>
+<wire x1="60.373" y1="29.797" x2="59.817" y2="30.353" width="0.3048" layer="1"/>
+<wire x1="59.591" y1="24.92" x2="60.373" y2="25.702" width="0.3048" layer="1"/>
+<wire x1="56.1086" y1="16.8402" x2="57.145" y2="17.8766" width="0.3048" layer="1"/>
+<wire x1="57.145" y1="17.8766" x2="57.145" y2="24.92" width="0.3048" layer="1"/>
 </signal>
 <signal name="+3V3">
@@
 <signal name="A0">
 <contactref element="ITSYBITSYM0" pad="10"/>
+<contactref element="RLS" pad="2"/>
+<wire x1="44.065" y1="46.355" x2="45.974" y2="46.355" width="0.3048" layer="1"/>
+<wire x1="45.974" y1="46.355" x2="49.53" y2="42.799" width="0.3048" layer="1"/>
+<wire x1="49.53" y1="28.727" x2="48.895" y2="28.092" width="0.3048" layer="1"/>
+<wire x1="49.53" y1="42.799" x2="49.53" y2="28.727" width="0.3048" layer="1"/>
 </signal>
 <signal name="A1">
@@
 <wire x1="35.306" y1="38.862" x2="35.306" y2="46.101" width="0.1524" layer="1"/>
 </signal>
+<signal name="N$4">
+<contactref element="LS1" pad="1"/>
+<contactref element="RLS" pad="1"/>
+<wire x1="53.345" y1="24.92" x2="49.223" y2="24.92" width="0.3048" layer="1"/>
+<wire x1="49.223" y1="24.92" x2="48.895" y2="25.248" width="0.3048" layer="1"/>
+</signal>
 </signals>

Commit message: updates
Parts:
- removed U1: MAX31723MUA+T, MAX31723MUA_T (1):SOP65P490X110-8N
Connections:
- net +3V3: no longer U1.2, U1.7, U1.8
- net GND: no longer U1.4
- net MISO: no longer U1.5
- net MOSI: no longer U1.6
- net SCK: no longer U1.3
Routing:
- net SCK: track 21.9 -> 0.00 mm
- net MOSI: track 17.2 -> 0.00 mm
- net +3V3: track 148.6 -> 135.8 mm
- net MISO: track 12.8 -> 0.00 mm
- net GND: track 57.4 -> 48.9 mm
Other:
- board text removed: "MAX31723"
Changed lines of the file:
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@@
 <wire x1="17.145" y1="38.608" x2="23.495" y2="38.608" width="0.1524" layer="25"/>
 <wire x1="10.16" y1="14.478" x2="21.59" y2="14.478" width="0.1524" layer="25"/>
-<wire x1="48.26" y1="18.415" x2="59.69" y2="18.415" width="0.1524" layer="21"/>
-<wire x1="48.26" y1="18.415" x2="48.26" y2="10.16" width="0.1524" layer="21"/>
-<wire x1="59.69" y1="18.415" x2="59.69" y2="10.16" width="0.1524" layer="21"/>
-<wire x1="59.69" y1="10.16" x2="48.26" y2="10.16" width="0.1524" layer="21"/>
-<wire x1="48.26" y1="13.208" x2="59.69" y2="13.208" width="0.1524" layer="25"/>
-<text x="50.419" y="11.176" size="1.016" layer="21">MAX31723</text>
 <wire x1="46.99" y1="29.845" x2="59.69" y2="29.845" width="0.1524" layer="21"/>
 <wire x1="46.99" y1="29.845" x2="46.99" y2="20.955" width="0.1524" layer="21"/>
@@
 <attribute name="VALUE" x="10.16" y="57.15" size="1.27" layer="27" rot="R270"/>
 </element>
-<element name="U1" library="MAX31723MUA_T (1)" package="SOP65P490X110-8N" value="MAX31723MUA+T" x="53.975" y="15.875" smashed="yes" rot="R180">
-<attribute name="AVAILABILITY" value="Unavailable" x="53.975" y="15.875" size="1.778" layer="27" rot="R180" display="off"/>
-<attribute name="DESCRIPTION" value=" Thermostat Â±2Â°C Digital SMD 8-Pin uMAX T/R " x="53.975" y="15.875" size="1.778" layer="27" rot="R180" display="off"/>
-<attribute name="MF" value="Maxim Integrated" x="53.975" y="15.875" size="1.778" layer="27" rot="R180" display="off"/>
-<attribute name="MP" value="MAX31723MUA+T" x="53.975" y="15.875" size="1.778" layer="27" rot="R180" display="off"/>
-<attribute name="PACKAGE" value="MSOP-8 Maxim Integrated" x="53.975" y="15.875" size="1.778" layer="27" rot="R180" display="off"/>
-<attribute name="PRICE" value="None" x="53.975" y="15.875" size="1.778" layer="27" rot="R180" display="off"/>
-<attribute name="VALUE" x="57.435990625" y="20.328490625" size="2.08678125" layer="27" ratio="10" rot="SR180"/>
-</element>
 <element name="RS3" library="resistor" library_urn="urn:adsk.eagle:library:348" package="R1206" package3d_urn="urn:adsk.eagle:package:26062/1" value="1k" x="49.53" y="33.02" smashed="yes" rot="R180">
 <attribute name="NAME" x="50.673" y="31.75" size="1.016" layer="25" rot="R180"/>
@@
 <contactref element="CRST" pad="2"/>
 <contactref element="CPRG" pad="2"/>
-<contactref element="U1" pad="4"/>
 <contactref element="GND" pad="1"/>
 <contactref element="PAD_GND1" pad="1"/>
@@
 <wire x1="60.373" y1="29.797" x2="59.817" y2="30.353" width="0.3048" layer="1"/>
 <wire x1="59.591" y1="24.92" x2="60.373" y2="25.702" width="0.3048" layer="1"/>
-<wire x1="56.1086" y1="16.8402" x2="57.145" y2="17.8766" width="0.3048" layer="1"/>
-<wire x1="57.145" y1="17.8766" x2="57.145" y2="24.92" width="0.3048" layer="1"/>
+<wire x1="57.145" y1="17.8766" x2="57.145" y2="24.92" width="0" layer="19" extent="1-16"/>
 </signal>
 <signal name="+3V3">
@@
 <contactref element="RRST1" pad="2"/>
 <contactref element="RPRG1" pad="2"/>
-<contactref element="U1" pad="2"/>
-<contactref element="U1" pad="8"/>
-<contactref element="U1" pad="7"/>
-<wire x1="51.8414" y1="14.9098" x2="51.8414" y2="15.5448" width="0.3048" layer="1"/>
 <contactref element="U$4" pad="4"/>
 <contactref element="+3V3" pad="1"/>
@@
 <wire x1="39.497" y1="53.975" x2="41.025" y2="53.975" width="0.3048" layer="1"/>
 <wire x1="21.107" y1="55.245" x2="38.227" y2="55.245" width="0.3048" layer="1"/>
-<wire x1="56.1086" y1="15.5448" x2="51.8414" y2="15.5448" width="0.1524" layer="1"/>
 <via x="43.815" y="13.97" extent="1-16" drill="1"/>
 <wire x1="42.40125" y1="24.2998" x2="42.3752" y2="24.2998" width="0.3048" layer="1"/>
@@
 <wire x1="35.687" y1="26.035" x2="35.052" y2="26.67" width="0.3048" layer="1"/>
 <wire x1="35.052" y1="26.67" x2="35.052" y2="31.115" width="0.3048" layer="1"/>
-<wire x1="51.8414" y1="15.5448" x2="43.8658" y2="15.5448" width="0.3048" layer="1"/>
 <wire x1="43.8658" y1="15.5448" x2="43.815" y2="15.494" width="0.3048" layer="1"/>
 </signal>
@@
 </signal>
 <signal name="MOSI">
-<contactref element="U1" pad="6"/>
 <contactref element="ITSYBITSYM0" pad="3"/>
-<wire x1="41.025" y1="28.575" x2="41.025" y2="26.412" width="0.1524" layer="1"/>
-<wire x1="51.2318" y1="16.2052" x2="51.8414" y2="16.2052" width="0.1524" layer="1"/>
-<wire x1="41.025" y1="26.412" x2="51.2318" y2="16.2052" width="0.1524" layer="1"/>
 </signal>
 <signal name="MISO">
-<contactref element="U1" pad="5"/>
 <contactref element="ITSYBITSYM0" pad="2"/>
-<wire x1="44.065" y1="26.035" x2="44.323" y2="25.777" width="0.1524" layer="1"/>
-<wire x1="44.323" y1="25.777" x2="44.323" y2="23.622" width="0.1524" layer="1"/>
-<wire x1="44.323" y1="23.622" x2="51.1048" y2="16.8402" width="0.1524" layer="1"/>
-<wire x1="51.1048" y1="16.8402" x2="51.8414" y2="16.8402" width="0.1524" layer="1"/>
 </signal>
 <signal name="SCK">
 <contactref element="ITSYBITSYM0" pad="4"/>
-<contactref element="U1" pad="3"/>
-<wire x1="44.065" y1="31.115" x2="45.847" y2="29.333" width="0.1524" layer="1"/>
-<wire x1="45.847" y1="29.333" x2="45.847" y2="22.987" width="0.1524" layer="1"/>
-<wire x1="45.847" y1="22.987" x2="51.435" y2="17.399" width="0.1524" layer="1"/>
-<wire x1="51.435" y1="17.399" x2="53.721" y2="17.399" width="0.1524" layer="1"/>
-<wire x1="53.721" y1="17.399" x2="54.9148" y2="16.2052" width="0.1524" layer="1"/>
-<wire x1="54.9148" y1="16.2052" x2="56.1086" y2="16.2052" width="0.1524" layer="1"/>
 </signal>
 <signal name="SENSPAD_2">

Commit message: updates
Other:
- board text added: "GND (IO)"
- board text removed: "GND (SWD)"
Changed lines of the file:
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@@
 <text x="32.893" y="8.89" size="1.016" layer="25" rot="R90">RXD</text>
 <text x="24.765" y="13.716" size="0.762" layer="25" align="bottom-right">+5V</text>
-<text x="25.019" y="11.049" size="0.762" layer="25" rot="R180" align="top-left">GND</text>
+<text x="24.765" y="11.049" size="0.762" layer="25" rot="R180" align="top-left">GND</text>
 <text x="45.085" y="13.589" size="0.762" layer="25" rot="R180" align="top-right">+3V3</text>
 <text x="45.339" y="11.049" size="0.762" layer="25" rot="R180" align="top-right">GND</text>
@@
 <text x="37.084" y="24.511" size="0.762" layer="26" rot="MR90">SWDIO</text>
 <text x="34.544" y="24.511" size="0.762" layer="26" rot="MR90">SWCLK</text>
-<text x="32.004" y="24.511" size="0.762" layer="26" rot="MR90">GND (SWD)</text>
+<text x="32.004" y="24.511" size="0.762" layer="26" rot="MR90">GND (IO)</text>
 <wire x1="10.16" y1="26.67" x2="21.59" y2="26.67" width="0.1524" layer="21"/>
 <wire x1="10.16" y1="26.67" x2="10.16" y2="10.16" width="0.1524" layer="21"/>
@@
 <wire x1="59.69" y1="29.845" x2="59.69" y2="20.955" width="0.1524" layer="21"/>
 <wire x1="59.69" y1="20.955" x2="46.99" y2="20.955" width="0.1524" layer="21"/>
-<wire x1="48.26" y1="23.368" x2="59.69" y2="23.368" width="0.1524" layer="25"/>
-<text x="51.054" y="21.59" size="1.016" layer="21">SPEAKER</text>
+<wire x1="46.99" y1="23.368" x2="59.69" y2="23.368" width="0.1524" layer="25"/>
+<text x="50.292" y="21.59" size="1.016" layer="21">SPEAKER</text>
 <wire x1="31.75" y1="43.18" x2="38.1" y2="43.18" width="0.1524" layer="25"/>
 <wire x1="38.1" y1="43.18" x2="38.1" y2="55.88" width="0.1524" layer="25"/>
@@
 <wire x1="60.373" y1="29.797" x2="59.817" y2="30.353" width="0.3048" layer="1"/>
 <wire x1="59.591" y1="24.92" x2="60.373" y2="25.702" width="0.3048" layer="1"/>
-<wire x1="57.145" y1="17.8766" x2="57.145" y2="24.92" width="0" layer="19" extent="1-16"/>
 </signal>
 <signal name="+3V3">
