File: eagle/5ButtonSwitch.ItsyBitsyM0.Rev1.1.sch (EAGLE design)
At the start: 30 parts

Commit message: updates
Parts:
- added U1: SN74LV1T34DBVR, SN74LV1T34DBVR:SN74LV1T34DBVR
Connections:
- new net N$5: U1.VCC
- new net N$6: U1.GND
- new net N$7: U1.A
- new net N$8: U1.Y
Changed lines of the file:
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@@
 <part name="LS1" library="CSS-0575B-SMT" deviceset="CSS-0575B-SMT" device=""/>
 <part name="RLS" library="resistor" library_urn="urn:adsk.eagle:library:348" deviceset="R-EU_" device="R1206" package3d_urn="urn:adsk.eagle:package:26062/1" value="0"/>
+<part name="U1" library="SN74LV1T34DBVR" deviceset="SN74LV1T34DBVR" device=""/>
 </parts>
 <sheets>
@@
 <instance part="LS1" gate="G$1" x="154.94" y="-88.9"/>
 <instance part="RLS" gate="G$1" x="139.7" y="-83.82" rot="R180"/>
+<instance part="U1" gate="A" x="50.8" y="-68.58"/>
 </instances>
 <busses>
@@
 </segment>
 </net>
+<net name="N$5" class="0">
+<segment>
+<pinref part="U1" gate="A" pin="VCC"/>
+<wire x1="104.14" y1="-68.58" x2="109.22" y2="-68.58" width="0.1524" layer="91"/>
+<label x="109.22" y="-68.58" size="1.27" layer="95" xref="yes"/>
+</segment>
+</net>
+<net name="N$6" class="0">
+<segment>
+<pinref part="U1" gate="A" pin="GND"/>
+<wire x1="104.14" y1="-73.66" x2="109.22" y2="-73.66" width="0.1524" layer="91"/>
+<label x="109.22" y="-73.66" size="1.27" layer="95" xref="yes"/>
+</segment>
+</net>
+<net name="N$7" class="0">
+<segment>
+<pinref part="U1" gate="A" pin="A"/>
+<wire x1="53.34" y1="-71.12" x2="45.72" y2="-71.12" width="0.1524" layer="91"/>
+<label x="45.72" y="-71.12" size="1.27" layer="95" rot="R180" xref="yes"/>
+</segment>
+</net>
+<net name="N$8" class="0">
+<segment>
+<pinref part="U1" gate="A" pin="Y"/>
+<wire x1="104.14" y1="-71.12" x2="109.22" y2="-71.12" width="0.1524" layer="91"/>
+<label x="109.22" y="-71.12" size="1.27" layer="95" xref="yes"/>
+</segment>
+</net>
