File: eagle/5ButtonSwitch.ItsyBitsyM0.Rev1.2.brd (EAGLE design)
At the start: 69.8 x 69.8 mm, 31 parts, among them U1 SN74LV1T34DBVR

Commit message: updates
Parts:
- moved U1 41.8 mm to (25.4, 18.4), turned to 90 degrees
Connections:
- removed net N$5: U1.5
- removed net N$6: U1.3
- removed net N$7: U1.2
- removed net N$8: U1.4
- new net LS_USART1_RX: SAM12235-ND.3, U1.2
- net +3V3: now also U1.5
- net GND: now also U1.3
- net USART1_RX: now also U1.4; no longer SAM12235-ND.3
Routing:
- net +3V3: track 134.8 -> 159.4 mm
- net LS_USART1_RX: track 0.00 -> 11.9 mm
- net USART1_RX: track 13.9 -> 4.20 mm
- net GND: track 48.9 -> 56.6 mm
Other:
- outline, holes or cut-outs redrawn
- board text added: "5xTouch Button | Konnekting | Rev 1.2"
- board text removed: "5xTouch Button | Konnekting | Rev 1.1"
Changed lines of the file:
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@@
 <drawing>
 <settings>
-<setting alwaysvectorfont="no"/>
+<setting alwaysvectorfont="yes"/>
 <setting verticaltext="up"/>
 </settings>
-<grid distance="50" unitdist="mil" unit="inch" style="lines" multiple="1" display="yes" altdistance="0.025" altunitdist="inch" altunit="inch"/>
+<grid distance="50" unitdist="mil" unit="inch" style="lines" multiple="1" display="yes" altdistance="5" altunitdist="mil" altunit="inch"/>
 <layers>
 <layer number="1" name="Top" color="4" fill="1" visible="yes" active="yes"/>
@@
 <wire x1="-2.54" y1="17.145" x2="73.025" y2="17.145" width="0.1524" layer="51"/>
 <wire x1="73.025" y1="17.145" x2="73.66" y2="17.78" width="0.1524" layer="51"/>
-<text x="22.098" y="60.96" size="1.016" layer="25">5xTouch Button | Konnekting | Rev 1.1</text>
+<text x="22.098" y="60.96" size="1.016" layer="25">5xTouch Button | Konnekting | Rev 1.2</text>
 <text x="26.924" y="59.182" size="1.016" layer="25">0XCDDC | 2019 by ChriD</text>
 <text x="30.353" y="8.89" size="1.016" layer="25" rot="R90">+5V</text>
@@
 <wire x1="40.64" y1="7.366" x2="46.99" y2="7.366" width="0.1524" layer="46"/>
 <wire x1="46.99" y1="7.366" x2="46.99" y2="6.477" width="0.1524" layer="46"/>
-<wire x1="39.37" y1="6.477" x2="30.48" y2="6.477" width="0.1524" layer="46"/>
+<wire x1="33.02" y1="6.477" x2="30.48" y2="6.477" width="0.1524" layer="46"/>
 <wire x1="30.48" y1="6.477" x2="30.48" y2="7.366" width="0.1524" layer="46"/>
-<wire x1="30.48" y1="7.366" x2="39.37" y2="7.366" width="0.1524" layer="46"/>
-<wire x1="39.37" y1="7.366" x2="39.37" y2="6.477" width="0.1524" layer="46"/>
+<wire x1="30.48" y1="7.366" x2="33.02" y2="7.366" width="0.1524" layer="46"/>
+<wire x1="33.02" y1="7.366" x2="33.02" y2="6.477" width="0.1524" layer="46"/>
 <wire x1="63.5" y1="62.611" x2="63.5" y2="46.99" width="0.1524" layer="46"/>
 <wire x1="63.5" y1="46.99" x2="62.611" y2="46.99" width="0.1524" layer="46"/>
@@
 <text x="33.02" y="30.353" size="0.762" layer="25">RGB LED</text>
 <wire x1="38.1" y1="29.972" x2="38.1" y2="31.496" width="0.1524" layer="25"/>
+<wire x1="36.83" y1="7.366" x2="36.83" y2="6.477" width="0.1524" layer="46"/>
+<wire x1="36.83" y1="7.366" x2="39.37" y2="7.366" width="0.1524" layer="46"/>
+<wire x1="39.37" y1="6.477" x2="36.83" y2="6.477" width="0.1524" layer="46"/>
+<wire x1="39.37" y1="6.477" x2="39.37" y2="7.366" width="0.1524" layer="46"/>
 </plain>
 <attributes>
@@
 <attribute name="VALUE" x="51.435" y="25.4" size="1.27" layer="27" rot="R90"/>
 </element>
-<element name="U1" library="SN74LV1T34DBVR" package="DBV5" value="SN74LV1T34DBVR" x="-3.81" y="-11.43">
-<attribute name="MANUFACTURER_PART_NUMBER" value="SN74LV1T34DBVR" x="-3.81" y="-11.43" size="1.778" layer="27" display="off"/>
-<attribute name="VENDOR" value="Texas Instruments" x="-3.81" y="-11.43" size="1.778" layer="27" display="off"/>
+<element name="U1" library="SN74LV1T34DBVR" package="DBV5" value="SN74LV1T34DBVR" x="25.4" y="18.415" rot="R90">
+<attribute name="MANUFACTURER_PART_NUMBER" value="SN74LV1T34DBVR" x="25.4" y="18.415" size="1.778" layer="27" rot="R90" display="off"/>
+<attribute name="VENDOR" value="Texas Instruments" x="25.4" y="18.415" size="1.778" layer="27" rot="R90" display="off"/>
 </element>
 </elements>
@@
 <wire x1="60.373" y1="29.797" x2="59.817" y2="30.353" width="0.3048" layer="1"/>
 <wire x1="59.591" y1="24.92" x2="60.373" y2="25.702" width="0.3048" layer="1"/>
-<wire x1="59.817" y1="30.353" x2="53.34" y2="48.26" width="0" layer="19" extent="1-1"/>
-<wire x1="43.815" y1="11.43" x2="57.145" y2="24.92" width="0" layer="19" extent="1-1"/>
-<wire x1="40.005" y1="13.716" x2="40.894" y2="11.43" width="0" layer="19" extent="1-16"/>
-<wire x1="14.224" y1="24.892" x2="26.035" y2="11.43" width="0" layer="19" extent="1-1"/>
-<wire x1="16.51" y1="48.26" x2="14.605" y2="27.305" width="0" layer="19" extent="1-1"/>
-<wire x1="23.114" y1="53.975" x2="15.875" y2="54.48" width="0" layer="19" extent="1-1"/>
+<contactref element="U1" pad="3"/>
+<wire x1="26.35" y1="17.2974" x2="26.35" y2="15.682" width="0.3048" layer="1"/>
+<wire x1="26.35" y1="15.682" x2="25.908" y2="15.24" width="0.3048" layer="1"/>
+<wire x1="25.908" y1="15.24" x2="25.273" y2="15.24" width="0.3048" layer="1"/>
+<wire x1="25.273" y1="15.24" x2="24.638" y2="14.605" width="0.3048" layer="1"/>
+<wire x1="24.638" y1="12.446" x2="25.654" y2="11.43" width="0.3048" layer="1"/>
+<wire x1="25.654" y1="11.43" x2="26.035" y2="11.43" width="0.3048" layer="1"/>
+<wire x1="24.638" y1="14.605" x2="24.638" y2="12.446" width="0.3048" layer="1"/>
 </signal>
 <signal name="+3V3">
@@
 <wire x1="18.898" y1="36.83" x2="18.898" y2="36.576" width="0.3048" layer="1"/>
 <wire x1="18.898" y1="36.576" x2="18.898" y2="33.02" width="0.3048" layer="1"/>
-<wire x1="12.065" y1="27.305" x2="12.065" y2="29.337" width="0.3048" layer="1"/>
+<wire x1="12.065" y1="27.305" x2="12.065" y2="27.94" width="0.3048" layer="1"/>
+<wire x1="12.065" y1="27.94" x2="12.065" y2="29.337" width="0.3048" layer="1"/>
 <wire x1="12.065" y1="29.337" x2="13.335" y2="30.607" width="0.3048" layer="1"/>
 <wire x1="18.161" y1="30.607" x2="18.923" y2="31.369" width="0.3048" layer="1"/>
@@
 <wire x1="42.40125" y1="24.2998" x2="42.3752" y2="24.2998" width="0.3048" layer="1"/>
 <wire x1="42.3752" y1="24.2998" x2="40.64" y2="26.035" width="0.3048" layer="1"/>
-<wire x1="43.815" y1="13.97" x2="43.815" y2="15.494" width="0.3048" layer="1"/>
-<wire x1="43.815" y1="15.494" x2="43.815" y2="22.88605" width="0.3048" layer="1"/>
+<wire x1="43.815" y1="13.97" x2="43.815" y2="22.88605" width="0.3048" layer="1"/>
 <wire x1="43.815" y1="22.88605" x2="42.40125" y2="24.2998" width="0.3048" layer="1"/>
 <wire x1="40.64" y1="26.035" x2="35.687" y2="26.035" width="0.3048" layer="1"/>
 <wire x1="35.687" y1="26.035" x2="34.925" y2="26.797" width="0.3048" layer="1"/>
-<wire x1="43.8658" y1="15.5448" x2="43.815" y2="15.494" width="0.3048" layer="1"/>
 <wire x1="34.925" y1="30.099" x2="34.163" y2="30.861" width="0.3048" layer="1"/>
 <wire x1="34.163" y1="31.8876" x2="34.163" y2="30.861" width="0.3048" layer="1"/>
@@
 <wire x1="32.639" y1="30.861" x2="28.575" y2="34.925" width="0.3048" layer="1"/>
 <wire x1="34.163" y1="32.258" x2="34.163" y2="31.8876" width="0.1524" layer="1"/>
+<contactref element="U1" pad="5"/>
+<wire x1="24.45" y1="19.5326" x2="12.2174" y2="19.5326" width="0.3048" layer="1"/>
+<wire x1="12.2174" y1="19.5326" x2="8.89" y2="22.86" width="0.3048" layer="1"/>
+<wire x1="8.89" y1="22.86" x2="8.89" y2="27.051" width="0.3048" layer="1"/>
+<wire x1="8.89" y1="27.051" x2="9.779" y2="27.94" width="0.3048" layer="1"/>
+<wire x1="9.779" y1="27.94" x2="12.065" y2="27.94" width="0.3048" layer="1"/>
 </signal>
 <signal name="USART1_RX">
-<contactref element="SAM12235-ND" pad="3"/>
 <contactref element="JP1" pad="1"/>
-<wire x1="25.785" y1="23.495" x2="28.702" y2="20.578" width="0.1524" layer="1"/>
-<wire x1="28.702" y1="20.578" x2="28.702" y2="16.891" width="0.1524" layer="1"/>
-<wire x1="28.702" y1="16.891" x2="29.591" y2="16.002" width="0.1524" layer="1"/>
-<wire x1="29.591" y1="16.002" x2="30.988" y2="16.002" width="0.1524" layer="1"/>
-<wire x1="30.988" y1="16.002" x2="31.242" y2="15.748" width="0.1524" layer="1"/>
-<wire x1="31.242" y1="13.97" x2="31.496" y2="13.716" width="0.1524" layer="1"/>
-<wire x1="31.496" y1="13.716" x2="32.385" y2="13.716" width="0.1524" layer="1"/>
-<wire x1="31.242" y1="15.748" x2="31.242" y2="13.97" width="0.1524" layer="1"/>
+<contactref element="U1" pad="4"/>
+<wire x1="26.35" y1="19.5326" x2="26.35" y2="22.93" width="0.1524" layer="1"/>
+<wire x1="26.35" y1="22.93" x2="25.785" y2="23.495" width="0.1524" layer="1"/>
 </signal>
 <signal name="USART1_TX">
@@
 <via x="66.04" y="31.115" extent="1-16" drill="1"/>
 </signal>
-<signal name="N$5">
-<contactref element="U1" pad="5"/>
-</signal>
-<signal name="N$6">
-<contactref element="U1" pad="3"/>
-</signal>
-<signal name="N$7">
+<signal name="LS_USART1_RX">
+<contactref element="SAM12235-ND" pad="3"/>
 <contactref element="U1" pad="2"/>
-</signal>
-<signal name="N$8">
-<contactref element="U1" pad="4"/>
+<wire x1="25.4" y1="17.2974" x2="25.4" y2="17.78" width="0.1524" layer="1"/>
+<wire x1="25.4" y1="17.2974" x2="25.4" y2="18.288" width="0.1524" layer="1"/>
+<wire x1="25.4" y1="18.288" x2="25.527" y2="18.415" width="0.1524" layer="1"/>
+<wire x1="27.305" y1="17.78" x2="27.305" y2="17.018" width="0.1524" layer="1"/>
+<wire x1="27.305" y1="17.018" x2="28.321" y2="16.002" width="0.1524" layer="1"/>
+<wire x1="31.877" y1="16.002" x2="32.385" y2="15.494" width="0.1524" layer="1"/>
+<wire x1="25.527" y1="18.415" x2="26.67" y2="18.415" width="0.1524" layer="1"/>
+<wire x1="26.67" y1="18.415" x2="27.305" y2="17.78" width="0.1524" layer="1"/>
+<wire x1="28.321" y1="16.002" x2="31.877" y2="16.002" width="0.1524" layer="1"/>
+<wire x1="32.385" y1="15.494" x2="32.385" y2="13.716" width="0.1524" layer="1"/>
 </signal>
 </signals>
