File: eagle/5ButtonSwitch.ItsyBitsyM0.Rev1.2.sch (EAGLE design)
At the start: 30 parts

Commit message: updates
Parts:
- added U1: SN74LV1T34DBVR, SN74LV1T34DBVR:SN74LV1T34DBVR
Connections:
- new net LS_USART1_RX: SAM12235-ND.3, U1.A
- net +3V3: now also U1.VCC
- net D11: now also RB.1; no longer RR.1
- net D13: now also RR.1; no longer RB.1
- net GND: now also U1.GND
- net USART1_RX: now also U1.Y; no longer SAM12235-ND.3
